File: kicad/haathi.sch (KiCad schematic (older format))
At the start: 1 part

Commit message: added BGA routing guides
Parts:
- U1: renamed from U?; footprint BGA196C65P14X14_1000X1000X152N -> footprint_lib:BGA196C65P14X14_1000X1000X152N_v2
Changed lines of the file:
@@
 $EndDescr
 $Comp
-L MIMXRT1052DVL6A:MIMXRT1052DVL6A U?
+L MIMXRT1052DVL6A:MIMXRT1052DVL6A U1
 U 1 1 5A4E4F98
 P 4475 5275
-F 0 "U?" H 4500 10025 50  0000 C CNN
+F 0 "U1" H 4500 10025 50  0000 C CNN
 F 1 "MIMXRT1052DVL6A" H 4500 9925 50  0000 C CNN
-F 2 "BGA196C65P14X14_1000X1000X152N" H 4475 5275 50  0001 L BNN
+F 2 "footprint_lib:BGA196C65P14X14_1000X1000X152N_v2" H 4475 5275 50  0001 L BNN
 F 3 "LFBGA-196 NXP Semiconductors" H 4475 5275 50  0001 L BNN
 F 4 "NXP Semiconductors" H 4475 5275 50  0001 L BNN "Field4"

Commit message: added some schematic symbols to lib
Parts:
- removed U1: MIMXRT1052DVL6A, footprint_lib:BGA196C65P14X14_1000X1000X152N_v2, symbol MIMXRT1052DVL6A:MIMXRT1052DVL6A
Other:
- note added: "1. Block Diagram\n2. Schematic\n a. Main Power\n b. Power Domain\n c. i.MXRT1052\n d. USB\n e. Audio\n f. SD Card\n g. JTAG\n h. SDRAM\n i. CSI (Camera)\n j. Misc."
- note added: ":: INDEX ::"
Changed lines of the file:
@@
 EELAYER 26 0
 EELAYER END
-$Descr A3 16535 11693
+$Descr A4 11693 8268
 encoding utf-8
-Sheet 1 1
+Sheet 1 2
 Title ""
 Date "2018-01-04"
@@
 Comment4 ""
 $EndDescr
-$Comp
-L MIMXRT1052DVL6A:MIMXRT1052DVL6A U1
-U 1 1 5A4E4F98
-P 4475 5275
-F 0 "U1" H 4500 10025 50  0000 C CNN
-F 1 "MIMXRT1052DVL6A" H 4500 9925 50  0000 C CNN
-F 2 "footprint_lib:BGA196C65P14X14_1000X1000X152N_v2" H 4475 5275 50  0001 L BNN
-F 3 "LFBGA-196 NXP Semiconductors" H 4475 5275 50  0001 L BNN
-F 4 "NXP Semiconductors" H 4475 5275 50  0001 L BNN "Field4"
-F 5 "https://www.digikey.in/product-detail/en/nxp-usa-inc/MIMXRT1052DVL6A/568-13515-ND/7646297?WT.z_cid=ref_snapeda&utm_source=snapeda&utm_medium=aggregator&utm_campaign=buynow" H 4475 5275 50  0001 L BNN "Field5"
-F 6 "568-13515-ND" H 4475 5275 50  0001 L BNN "Field6"
-F 7 "MIMXRT1052DVL6A" H 4475 5275 50  0001 L BNN "Field7"
-F 8 "I.MXRT1050" H 4475 5275 50  0001 L BNN "Field8"
-	1    4475 5275
-	1    0    0    -1
-$EndComp
+Text Notes 1400 1150 0    150  ~ 30
+:: INDEX ::
+Wire Notes Line
+	1400 1200 2575 1200
+Text Notes 1400 3700 0    120  ~ 24
+1. Block Diagram\n2. Schematic\n     a. Main Power\n     b. Power Domain\n     c. i.MXRT1052\n     d. USB\n     e. Audio\n     f. SD Card\n     g. JTAG\n     h. SDRAM\n     i. CSI (Camera)\n     j. Misc.
+$Sheet
+S 5000 1500 2500 1250
+U 5A56B6F6
+F0 "Block Diagram" 120
+F1 "block.sch" 120
+$EndSheet
+$Sheet
+S 5000 4000 2500 1250
+U 5A56B6FF
+F0 "Schematic" 120
+F1 "schematic.sch" 120
+$EndSheet
 $EndSCHEMATC
