File: kicad/_saved_haathi_power.sch (KiCad schematic (older format))
At the start: 12 parts

Commit message: Added power circuits for buck converter and snvs
Parts:
- added R? (x3): 0, symbol haathi_mayank:R
Connections:
- net labels added: DCDC_IN, NVCC_EMC, NVCC_GPIO, NVCC_SD0, NVCC_SD1, VDDA_ADC_3P3, VDD_HIGH_IN
- wire segments 50 -> 72
Changed lines of the file:
@@
 L haathi_mayank:R R?
 U 1 1 5A6ED3C7
-P 7300 1700
-F 0 "R?" H 7370 1746 50  0000 L CNN
-F 1 "0" H 7370 1655 50  0000 L CNN
-F 2 "" V 7230 1700 30  0000 C CNN
-F 3 "" H 7300 1700 30  0000 C CNN
-	1    7300 1700
-	1    0    0    -1
+P 8450 1250
+F 0 "R?" H 8520 1296 50  0000 L CNN
+F 1 "0" H 8520 1205 50  0000 L CNN
+F 2 "" V 8380 1250 30  0000 C CNN
+F 3 "" H 8450 1250 30  0000 C CNN
+	1    8450 1250
+	0    1    1    0
 $EndComp
 $Comp
 L haathi_mayank:R R?
 U 1 1 5A6ED45D
-P 7650 1700
-F 0 "R?" H 7720 1746 50  0000 L CNN
-F 1 "0" H 7720 1655 50  0000 L CNN
-F 2 "" V 7580 1700 30  0000 C CNN
-F 3 "" H 7650 1700 30  0000 C CNN
-	1    7650 1700
-	1    0    0    -1
+P 8450 1600
+F 0 "R?" H 8520 1646 50  0000 L CNN
+F 1 "0" H 8520 1555 50  0000 L CNN
+F 2 "" V 8380 1600 30  0000 C CNN
+F 3 "" H 8450 1600 30  0000 C CNN
+	1    8450 1600
+	0    1    1    0
 $EndComp
 $Comp
 L haathi_mayank:R R?
 U 1 1 5A6ED497
-P 7950 1700
-F 0 "R?" H 8020 1746 50  0000 L CNN
-F 1 "0" H 8020 1655 50  0000 L CNN
-F 2 "" V 7880 1700 30  0000 C CNN
-F 3 "" H 7950 1700 30  0000 C CNN
-	1    7950 1700
-	1    0    0    -1
+P 8450 1900
+F 0 "R?" H 8520 1946 50  0000 L CNN
+F 1 "0" H 8520 1855 50  0000 L CNN
+F 2 "" V 8380 1900 30  0000 C CNN
+F 3 "" H 8450 1900 30  0000 C CNN
+	1    8450 1900
+	0    1    1    0
 $EndComp
 $Comp
 L haathi_mayank:R R?
 U 1 1 5A6ED4CD
-P 8250 1700
-F 0 "R?" H 8320 1746 50  0000 L CNN
-F 1 "0" H 8320 1655 50  0000 L CNN
-F 2 "" V 8180 1700 30  0000 C CNN
-F 3 "" H 8250 1700 30  0000 C CNN
-	1    8250 1700
+P 8450 2200
+F 0 "R?" H 8520 2246 50  0000 L CNN
+F 1 "0" H 8520 2155 50  0000 L CNN
+F 2 "" V 8380 2200 30  0000 C CNN
+F 3 "" H 8450 2200 30  0000 C CNN
+	1    8450 2200
+	0    1    1    0
+$EndComp
+$Comp
+L haathi_mayank:R R?
+U 1 1 5A6ED6D7
+P 8450 2500
+F 0 "R?" H 8520 2546 50  0000 L CNN
+F 1 "0" H 8520 2455 50  0000 L CNN
+F 2 "" V 8380 2500 30  0000 C CNN
+F 3 "" H 8450 2500 30  0000 C CNN
+	1    8450 2500
+	0    1    1    0
+$EndComp
+$Comp
+L haathi_mayank:R R?
+U 1 1 5A6ED735
+P 8450 2800
+F 0 "R?" H 8520 2846 50  0000 L CNN
+F 1 "0" H 8520 2755 50  0000 L CNN
+F 2 "" V 8380 2800 30  0000 C CNN
+F 3 "" H 8450 2800 30  0000 C CNN
+	1    8450 2800
+	0    1    1    0
+$EndComp
+$Comp
+L haathi_mayank:R R?
+U 1 1 5A6ED769
+P 8450 3050
+F 0 "R?" H 8520 3096 50  0000 L CNN
+F 1 "0" H 8520 3005 50  0000 L CNN
+F 2 "" V 8380 3050 30  0000 C CNN
+F 3 "" H 8450 3050 30  0000 C CNN
+	1    8450 3050
+	0    1    1    0
+$EndComp
+Wire Wire Line
+	8300 1250 8150 1250
+Wire Wire Line
+	8300 1600 8150 1600
+Wire Wire Line
+	8150 1600 8150 1250
+Connection ~ 8150 1250
+Wire Wire Line
+	8150 1250 8000 1250
+Wire Wire Line
+	8300 1900 8150 1900
+Wire Wire Line
+	8150 1900 8150 1600
+Connection ~ 8150 1600
+Wire Wire Line
+	8300 2200 8150 2200
+Wire Wire Line
+	8150 2200 8150 1900
+Connection ~ 8150 1900
+Wire Wire Line
+	8300 2500 8150 2500
+Wire Wire Line
+	8150 2500 8150 2200
+Connection ~ 8150 2200
+Wire Wire Line
+	8300 2800 8150 2800
+Wire Wire Line
+	8150 2800 8150 2500
+Connection ~ 8150 2500
+Wire Wire Line
+	8300 3050 8150 3050
+Wire Wire Line
+	8150 3050 8150 2800
+Connection ~ 8150 2800
+Wire Wire Line
+	8600 1250 8750 1250
+Wire Wire Line
+	8600 1600 8750 1600
+Wire Wire Line
+	8600 1900 8750 1900
+Wire Wire Line
+	8600 2200 8750 2200
+Wire Wire Line
+	8600 2500 8750 2500
+Wire Wire Line
+	8600 2800 8750 2800
+Wire Wire Line
+	8600 3050 8750 3050
+$Comp
+L power:VCC #PWR?
+U 1 1 5A6FED5F
+P 7950 1250
+F 0 "#PWR?" H 7950 1100 50  0001 C CNN
+F 1 "VCC" H 7967 1423 50  0000 C CNN
+F 2 "" H 7950 1250 50  0001 C CNN
+F 3 "" H 7950 1250 50  0001 C CNN
+	1    7950 1250
 	1    0    0    -1
 $EndComp
+$Comp
+L power:PWR_FLAG #FLG?
+U 1 1 5A6FEDB5
+P 8000 1250
+F 0 "#FLG?" H 8000 1325 50  0001 C CNN
+F 1 "PWR_FLAG" H 8000 1423 50  0000 C CNN
+F 2 "" H 8000 1250 50  0001 C CNN
+F 3 "" H 8000 1250 50  0001 C CNN
+	1    8000 1250
+	-1   0    0    1
+$EndComp
+Connection ~ 8000 1250
+Wire Wire Line
+	8000 1250 7950 1250
+Text HLabel 8750 1250 2    50   Input ~ 0
+DCDC_IN
+Text HLabel 8750 1600 2    50   Input ~ 0
+NVCC_SD0
+Text HLabel 8750 1900 2    50   Input ~ 0
+NVCC_SD1
+Text HLabel 8750 2200 2    50   Input ~ 0
+NVCC_EMC
+Text HLabel 8750 2500 2    50   Input ~ 0
+NVCC_GPIO
+Text HLabel 8750 2800 2    50   Input ~ 0
+VDDA_ADC_3P3
+Text HLabel 8750 3050 2    50   Input ~ 0
+VDD_HIGH_IN
 $EndSCHEMATC
