File: kicad/haathi_schematic2.sch (KiCad schematic (older format))
At the start: 0 parts

Commit message: Anool, USB sheet
Connections:
- wire segments 5 -> 4
Changed lines of the file:
@@
 F0 "POWER" 50
 F1 "haathi_power.sch" 50
-F2 "VIN" I L 2000 1350 50
 $EndSheet
 $Sheet
@@
 claimed : Mayank
 Wire Wire Line
-	2000 1350 1700 1350
+	2000 3200 1375 3200
 Wire Wire Line
-	2000 3200 1250 3200
+	1375 3300 2000 3300
 Wire Wire Line
-	1250 3300 2000 3300
+	2000 3400 1375 3400
 Wire Wire Line
-	2000 3400 1250 3400
-Wire Wire Line
-	1250 3500 2000 3500
-Text Label 1250 3200 0    50   ~ 0
+	1375 3500 2000 3500
+Text Label 1375 3200 0    50   ~ 0
 5V_USB_OTG
-Text Label 1250 3300 0    50   ~ 0
+Text Label 1375 3300 0    50   ~ 0
 USB_OTG1_D-
-Text Label 1250 3400 0    50   ~ 0
+Text Label 1375 3400 0    50   ~ 0
 USB_OTG1_D+
-Text Label 1250 3500 0    50   ~ 0
+Text Label 1375 3500 0    50   ~ 0
 USB_OTG1_ID
 $EndSCHEMATC
