File: kicad/haathi_usb.sch (KiCad schematic (older format))
At the start: 13 parts, among them J1 USB_microAB

Commit message: Annotated schematic
Parts:
- gave numbers to parts that had none: 6
Changed lines of the file:
@@
 NoConn ~ 4500 2825
 $Comp
-L haathi:C_NP C?
+L haathi:C_NP C108
 U 1 1 5A8AEC37
 P 5450 4675
-F 0 "C?" H 5550 4725 40  0000 L CNN
+F 0 "C108" H 5550 4725 40  0000 L CNN
 F 1 "4.7uF" H 5550 4650 40  0000 L CNN
 F 2 "" H 5450 4675 60  0000 C CNN
@@
 $EndComp
 $Comp
-L haathi:IND_FERRITE_BEAD L?
+L haathi:IND_FERRITE_BEAD L6
 U 1 1 5A8AEC3E
 P 2375 5675
-F 0 "L?" H 2175 5700 40  0000 C CNN
+F 0 "L6" H 2175 5700 40  0000 C CNN
 F 1 "330E" H 2375 5550 40  0000 C CNN
 F 2 "" H 2375 5675 60  0000 C CNN
@@
 $EndComp
 $Comp
-L haathi:IND_FERRITE_BEAD L?
+L haathi:IND_FERRITE_BEAD L7
 U 1 1 5A8AEC45
 P 4875 4425
-F 0 "L?" H 4875 4550 40  0000 C CNN
+F 0 "L7" H 4875 4550 40  0000 C CNN
 F 1 "330E" H 4900 4300 40  0000 C CNN
 F 2 "" H 4875 4425 60  0000 C CNN
@@
 $EndComp
 $Comp
-L haathi:Diode_TVS D?
+L haathi:Diode_TVS D7
 U 1 1 5A8AEC4C
 P 3650 6275
-F 0 "D?" H 3900 6075 50  0000 R CNN
+F 0 "D7" H 3900 6075 50  0000 R CNN
 F 1 "RClamp0854P.TCT" H 4175 6000 50  0000 R CNN
 F 2 "" H 3650 6275 50  0001 C CNN
@@
 $EndComp
 $Comp
-L haathi:IND_CHOKE_CM L?
+L haathi:IND_CHOKE_CM L8
 U 1 1 5A8AEC53
 P 4875 5425
-F 0 "L?" H 4875 5200 40  0000 C CNN
+F 0 "L8" H 4875 5200 40  0000 C CNN
 F 1 "90E" H 4875 5275 40  0000 C CNN
 F 2 "" H 4875 5325 60  0000 C CNN
@@
 $EndComp
 $Comp
-L haathi:R R?
+L haathi:R R72
 U 1 1 5A8AEC5A
 P 4850 5800
-F 0 "R?" V 4750 5800 50  0000 C CNN
+F 0 "R72" V 4750 5800 50  0000 C CNN
 F 1 "0E" V 4850 5800 50  0000 C CNN
 F 2 "" V 4780 5800 30  0000 C CNN
@@
 	6325 5525 5075 5525
 $Comp
-L power:GND #PWR?
+L power:GND #PWR081
 U 1 1 5A8AEC88
 P 2725 7400
-F 0 "#PWR?" H 2725 7150 50  0001 C CNN
+F 0 "#PWR081" H 2725 7150 50  0001 C CNN
 F 1 "GND" H 2750 7200 50  0000 C CNN
 F 2 "" H 2725 7400 50  0001 C CNN
@@
 $EndComp
 $Comp
-L power:GND #PWR?
+L power:GND #PWR082
 U 1 1 5A8AEC8E
 P 3450 7400
-F 0 "#PWR?" H 3450 7150 50  0001 C CNN
+F 0 "#PWR082" H 3450 7150 50  0001 C CNN
 F 1 "GND" H 3500 7200 50  0000 C CNN
 F 2 "" H 3450 7400 50  0001 C CNN
@@
 $EndComp
 $Comp
-L power:GND #PWR?
+L power:GND #PWR083
 U 1 1 5A8AEC94
 P 5450 4950
-F 0 "#PWR?" H 5450 4700 50  0001 C CNN
+F 0 "#PWR083" H 5450 4700 50  0001 C CNN
 F 1 "GND" H 5500 4750 50  0000 C CNN
 F 2 "" H 5450 4950 50  0001 C CNN
