File: kicad/haathi_usb.sch (KiCad schematic (older format))
At the start: 12 parts, among them J1 USB_microAB

Commit message: Complete annotation
Signed-off-by: Kumar Abhishek <abhishek@theembeddedkitchen.net>
Parts:
- gave numbers to parts that had none: 2
Changed lines of the file:
@@
 EESchema Schematic File Version 4
+LIBS:haathi_schematic-cache
 EELAYER 26 0
 EELAYER END
 $Descr A4 11693 8268
 encoding utf-8
-Sheet 1 9
+Sheet 4 9
 Title "haathi_cam"
 Date "2018-03-11"
@@
 GPIO_AD_B0_00
 $Comp
-L haathi:TPD4S012 D?
+L haathi:TPD4S012 D3
 U 1 1 5B0B0690
 P 3650 6375
-F 0 "D?" H 3362 6396 50  0000 R CNN
+F 0 "D3" H 3362 6396 50  0000 R CNN
 F 1 "TPD4S012" H 3362 6305 50  0000 R CNN
 F 2 "" H 3650 6375 50  0001 C CNN
@@
 	3450 6775 3450 7400
 $Comp
-L haathi:TPD4S012 D?
+L haathi:TPD4S012 D4
 U 1 1 5B0B3608
 P 4150 2825
-F 0 "D?" H 3862 2846 50  0000 R CNN
+F 0 "D4" H 3862 2846 50  0000 R CNN
 F 1 "TPD4S012" H 3862 2755 50  0000 R CNN
 F 2 "" H 4150 2825 50  0001 C CNN

Commit message: USB connector changed to be compatible with 6 pin Wurth one
Parts:
- J1: symbol haathi:USB_microAB -> haathi:USB_micro
Connections:
- wire segments 72 -> 63
Changed lines of the file:
@@
 EESchema Schematic File Version 4
-LIBS:haathi_schematic-cache
+LIBS:haathi_usb-cache
 EELAYER 26 0
 EELAYER END
 $Descr A4 11693 8268
 encoding utf-8
-Sheet 4 9
+Sheet 1 1
 Title "haathi_cam"
 Date "2018-03-11"
@@
 $EndDescr
 $Comp
-L haathi:USB_microAB J1
+L haathi:USB_micro J1
 U 1 1 5A6AD825
-P 2275 1925
-F 0 "J1" H 2050 2000 50  0000 R CNN
-F 1 "USB_microAB" H 2050 1900 50  0000 R CNN
-F 2 "" H 2275 1925 50  0001 C CNN
-F 3 "" H 2275 1925 50  0001 C CNN
-	1    2275 1925
+P 2075 1925
+F 0 "J1" H 1850 2000 50  0000 R CNN
+F 1 "USB_microAB" H 1850 1900 50  0000 R CNN
+F 2 "" H 2075 1925 50  0001 C CNN
+F 3 "" H 2075 1925 50  0001 C CNN
+	1    2075 1925
 	1    0    0    -1
 $EndComp
@@
 Wire Wire Line
 	3225 2125 3225 3850
-Wire Wire Line
-	2275 1525 2275 1425
-Wire Wire Line
-	2275 1425 2175 1425
-Wire Wire Line
-	1425 1425 1425 2425
-Wire Wire Line
-	1425 2425 2175 2425
-Wire Wire Line
-	2275 2425 2275 2325
-Wire Wire Line
-	2175 2325 2175 2425
-Connection ~ 2175 2425
-Wire Wire Line
-	2175 2425 2275 2425
-Wire Wire Line
-	2175 1525 2175 1425
-Connection ~ 2175 1425
-Wire Wire Line
-	2175 1425 1425 1425
-Wire Wire Line
-	2175 2425 2175 2850
-Wire Wire Line
-	2175 2850 2450 2850
 Wire Wire Line
 	2850 2850 2975 2850
@@
 Wire Wire Line
 	3950 3225 3950 3850
+Wire Wire Line
+	2075 2325 2075 2850
+Wire Wire Line
+	2075 2850 2450 2850
 $EndSCHEMATC
