File: kicad/haathi_cpu.sch (KiCad schematic (older format))
At the start: 0 parts

Commit message: Mayank, CPU Sheet init and supervisor IC
Parts:
- added C?: 0.1uF_DNP, symbol haathi_mayank:C_POL
- added R?: 100k_DNP, symbol haathi_mayank:R
- added R?: 1k, symbol haathi_mayank:R
- added R?: 0E_DNP, symbol haathi_mayank:R
- added R?: 1.5k 1%, symbol haathi_mayank:R
- added U? (x9): MIMXRT1052DVL6A_0, BGA196C65P14X14_1000X1000X152N, symbol haathi_mayank:MIMXRT1052DVL6A_0
- added U?: APX809S-26SR, symbol haathi_mayank:APX809S-26SR
Connections:
- net labels added: GND, MCU_RESET_N, ONOFF, VCC, VDD_SNVS_IN
- wire segments 0 -> 24

Commit message: Mayank, CPU Power connections
Parts:
- removed C?: 0.1uF_DNP, symbol haathi_mayank:C_POL
- added C?: 0.1uF_DNP, symbol haathi_mayank:C_NP
- added C? (x2): 18pF, symbol haathi_mayank:C_NP
- added C? (x2): 4.7pF, symbol haathi_mayank:C_NP
- added C? (x9): 4.7uF, symbol haathi_mayank:C_NP
- added C? (x9): 0.1uF, symbol haathi_mayank:C_NP
- added C? (x20): 0.22uF, symbol haathi_mayank:C_NP
- added C? (x2): 22uF_DNP, symbol haathi_mayank:C_NP
- added C?: 10uF, symbol haathi_mayank:C_NP
- added C?: 1uF, symbol haathi_mayank:C_NP
- added C?: 33uF, symbol haathi_mayank:C_NP
- added J?: Conn_01x02, symbol haathi_mayank:Conn_01x02
- added L?: 4.7uH, symbol haathi_mayank:IND_SML
- added R?: 2.2M, symbol haathi_mayank:R
- added R?: 1M_DNP, symbol haathi_mayank:R
- added R?: 0E, symbol haathi_mayank:R
- added TP? (x2): Test_Point_Probe, symbol haathi_mayank:Test_Point_Probe
- added Y?: 32.768kHz, symbol haathi_mayank:Crystal
- added Y?: 24MHz, symbol haathi_mayank:Crystal_GND24
Connections:
- net labels added: DCDC_OUT, NVCC_GPIO_3V3, NVCC_SD0, NVCC_SD1, NVCC_SEMC_3V3, PMIC_ON_REQ, PMIC_STBY_REQ, USER_BUTTON, VDDA_ADC_3P3, VDD_HIGH_CAP, VDD_HIGH_IN, VDD_SNVS_CAP, VDD_SOC_IN, VDD_USB_CAP
- wire segments 24 -> 236
- no-connect marks 0 -> 2

Commit message: Mayank, CPU finished GPIO EMC block
Parts:
- added C?: 0.1uF, symbol haathi_mayank:C_NP
Connections:
- net labels added: ENET_MDC, ENET_MDIO, SEMC_A0, SEMC_A1, SEMC_A10, SEMC_A11, SEMC_A12, SEMC_A2, SEMC_A3, SEMC_A4, SEMC_A5, SEMC_A6, SEMC_A7, SEMC_A8, SEMC_A9, SEMC_A[12:0], SEMC_BA0, SEMC_BA1, SEMC_CAS, SEMC_CKE, SEMC_CLK, SEMC_CS0, SEMC_D0, SEMC_D1, SEMC_D10, SEMC_D11, SEMC_D12, SEMC_D13, SEMC_D14, SEMC_D15, SEMC_D2, SEMC_D3, SEMC_D4, SEMC_D5, SEMC_D6, SEMC_D7, SEMC_D8, SEMC_D9, SEMC_DM0, SEMC_DM1, SEMC_DQS, SEMC_D[15:8], SEMC_D[7:0], SEMC_RAS, SEMC_WE
- wire segments 236 -> 286
Other:
- note added: "MCU Power Circuit"

Commit message: Mayank, CPU, completed GPIO_AD_B1
Parts:
- added R? (x2): 4.7k, symbol haathi_mayank:R
- added R?: 10k, symbol haathi_mayank:R
- added TP?: Test_Point_Probe, symbol haathi_mayank:Test_Point_Probe
Connections:
- net labels added: AUD_INT, CAN2_RX, CAN2_TX, ENET_INT, ENET_RST, GPIO_AD_B0_00, GPIO_AD_B0_09, GPIO_AD_B0_1, GPIO_AD_B0_10, GPIO_AD_B0_11, GPIO_AD_B0_2, GPIO_AD_B0_3, GPIO_AD_B0_4, GPIO_AD_B0_5, GPIO_AD_B1_00, GPIO_AD_B1_1, GPIO_AD_B1_10, GPIO_AD_B1_11, GPIO_AD_B1_12, GPIO_AD_B1_13, GPIO_AD_B1_14, GPIO_AD_B1_15, GPIO_AD_B1_2, GPIO_AD_B1_3, GPIO_AD_B1_4, GPIO_AD_B1_5, GPIO_AD_B1_6, GPIO_AD_B1_7, GPIO_AD_B1_8, GPIO_AD_B1_9, I2C1_SCL, I2C1_SDA, INT1_COMBO, INT2_COMBO, JTAG_MOD, JTAG_TCK, JTAG_TDI, JTAG_TDO, JTAG_TMS, JTAG_nTRST, LCD_TOUCH_INT, SAI1_MCLK, SAI1_RXD, SAI1_RX_BCLK, SAI1_RX_SYNC, SAI1_TXD, SAI1_TX_BCLK, SAI1_TX_SYNC, SPDIF_IN, SPDIF_OUT, SWD_DIO, SWD_SCK, UART1_RXD, UART1_TXD, USER_LED
- wire segments 286 -> 347
Other:
- note added: "By Default"
- note added: "JTAG"

Commit message: Mayank, CPU added GPIO_B0 and GPIO_B1
Connections:
- net labels added: BACKLIGHT_CTL, ENET_CRS_DV, ENET_RXD0, ENET_RXD1, ENET_RXER, ENET_TXD0, ENET_TXD1, ENET_TXEN, ENET_TX_CLK, GPIO_B0_04, GPIO_B0_05, GPIO_B0_06, GPIO_B0_08, GPIO_B0_09, GPIO_B0_10, GPIO_B0_11, GPIO_B0_12, GPIO_B0_13, GPIO_B0_14, GPIO_B0_15, GPIO_B0_7, LCDIF_CLK, LCDIF_D0, LCDIF_D1, LCDIF_D10, LCDIF_D11, LCDIF_D12, LCDIF_D13, LCDIF_D14, LCDIF_D15, LCDIF_D2, LCDIF_D3, LCDIF_D4, LCDIF_D5, LCDIF_D6, LCDIF_D7, LCDIF_D8, LCDIF_D9, LCDIF_D[15:0], LCDIF_ENABLE, LCDIF_HSYNC, LCDIF_VSYNC, SD0_VSELECT, SD_CD_SW, USB_HOST_PWR, WDOG_B
- wire segments 347 -> 382

Commit message: Mayank, CPU Sheet done, added USB OTG pins
Parts:
- added C? (x2): 1uF, symbol haathi_mayank:C_NP
- added R? (x2): 10k, symbol haathi_mayank:R
- added TP? (x3): Test_Point_Probe, symbol haathi_mayank:Test_Point_Probe
Connections:
- net labels added: 5V_USB_HS, 5V_USB_OTG, FlexSPI_CLK, FlexSPI_CLK_B, FlexSPI_D0_A, FlexSPI_D0_B, FlexSPI_D1_A, FlexSPI_D1_B, FlexSPI_D2_A, FlexSPI_D2_B, FlexSPI_D3_A, FlexSPI_D3_B, FlexSPI_DQS, FlexSPI_SS0, GPIO_SD_B0_00, GPIO_SD_B0_02, GPIO_SD_B0_03, GPIO_SD_B1_01, GPIO_SD_B1_02, GPIO_SD_B1_04, GPIO_SD_B1_05, SD1_CLK, SD1_CMD, SD1_D0, SD1_D1, SD1_D2, SD1_D3, USB_OTG1_D+, USB_OTG1_D-, USB_OTG2_D+, USB_OTG2_D-
- wire segments 382 -> 424
Other:
- note added: "LCD Interface\n"
- note added: "SD Interface\n"
- note added: "USB_OTG\n"

Commit message: Mayank, added BootCFG with dipswitch to CPU sheet
Parts:
- added R? (x14): 10k, symbol haathi_mayank:R
- added R? (x3): 1k, symbol haathi_mayank:R
- added R? (x10): 1k_DNP, symbol haathi_mayank:R
- added SW?: SW_DIP_x03, symbol haathi_mayank:SW_DIP_x03
Connections:
- net labels added: BOOT_MODE[0], BOOT_MODE[1], BT_CFG[0], BT_CFG[10], BT_CFG[11], BT_CFG[1], BT_CFG[2], BT_CFG[3], BT_CFG[4], BT_CFG[5], BT_CFG[6], BT_CFG[7], BT_CFG[8], BT_CFG[9], GPIO_AD_B0_04, GPIO_AD_B0_05, GPIO_B0_07, GPIO_B0_5, GPIO_B0_6, GPIO_B0_8, GPIO_B0_9
- wire segments 424 -> 527
Other:
- note added: "Boot Configuration\n"

Commit message: Renamed USER_BUTTON to WAKEUP_BUTTON
Connections:
- net labels added: WAKEUP_BUTTON
- net labels removed: USER_BUTTON
Changed lines of the file:
@@
 	3650 3150 4350 3150
 Text HLabel 3600 3450 0    50   Input ~ 0
-USER_BUTTON
+WAKEUP_BUTTON
 Wire Wire Line
 	3600 3450 3700 3450
@@
 	3850 11300 4050 11300
 Connection ~ 4050 11300
+Text Notes 4500 10950 0    100  ~ 0
+Boot Configuration\n
 Wire Bus Line
 	21100 950  21100 1750
@@
 Wire Bus Line
 	9425 8000 9425 9800
-Text Notes 4500 10950 0    100  ~ 0
-Boot Configuration\n
 $EndSCHEMATC
