File: kicad/haathi_cpu.sch (KiCad schematic (older format))
At the start: 113 parts

Commit message: Migration to A1 needs RC delay for PSWITCH.
Change the 0E to 30k for the RC filter to delay the PSWITCH signal as compared to DCDC_IN
Parts:
- R?: value 0E -> 30k
Changed lines of the file:
@@
 $Descr A2 23386 16535
 encoding utf-8
-Sheet 1 9
+Sheet 1 1
 Title "haathi_cam"
 Date "2018-03-11"
@@
 P 7350 4450
 F 0 "R?" V 7557 4450 50  0000 C CNN
-F 1 "0E" V 7466 4450 50  0000 C CNN
+F 1 "30k" V 7466 4450 50  0000 C CNN
 F 2 "" V 7280 4450 30  0000 C CNN
 F 3 "" H 7350 4450 30  0000 C CNN
@@
 Wire Wire Line
 	13825 5225 14550 5225
-Wire Bus Line
-	21850 4000 21850 4750
-Wire Bus Line
-	21100 950  21100 1750
-Wire Bus Line
-	21900 1900 21900 3350
-Wire Bus Line
-	9425 8000 9425 9800
 Text HLabel 13825 4925 0    50   Input ~ 0
 GPIO_AD_B1_04
@@
 Text HLabel 13825 5225 0    50   Input ~ 0
 GPIO_AD_B1_07
+Wire Bus Line
+	21850 4000 21850 4750
+Wire Bus Line
+	21100 950  21100 1750
+Wire Bus Line
+	21900 1900 21900 3350
+Wire Bus Line
+	9425 8000 9425 9800
 $EndSCHEMATC

Commit message: Add the 0.1 decoupling/RC filter cap to the voltage detector. Gone are SPDIF In and Out, one of them used for SD_PWREN and other a general GPIO.
Parts:
- added C?: 0.1uF, symbol haathi_mayank:C_NP
Connections:
- net labels added: SD_PWREN
- net labels removed: SPDIF_IN, SPDIF_OUT
- wire segments 516 -> 519
Changed lines of the file:
@@
 EESchema Schematic File Version 4
+LIBS:haathi_cpu-cache
 EELAYER 26 0
 EELAYER END
@@
 L haathi_mayank:R R?
 U 1 1 5A7C3889
-P 1200 3050
-F 0 "R?" V 1407 3050 50  0000 C CNN
-F 1 "1.5k 1%" V 1316 3050 50  0000 C CNN
-F 2 "" V 1130 3050 30  0000 C CNN
-F 3 "" H 1200 3050 30  0000 C CNN
-	1    1200 3050
+P 1150 3050
+F 0 "R?" V 1357 3050 50  0000 C CNN
+F 1 "1.5k 1%" V 1266 3050 50  0000 C CNN
+F 2 "" V 1080 3050 30  0000 C CNN
+F 3 "" H 1150 3050 30  0000 C CNN
+	1    1150 3050
 	0    -1   -1   0
 $EndComp
@@
 L power:PWR_FLAG #FLG?
 U 1 1 5A7C425A
-P 950 3050
-F 0 "#FLG?" H 950 3125 50  0001 C CNN
-F 1 "PWR_FLAG" H 950 3223 50  0000 C CNN
-F 2 "" H 950 3050 50  0001 C CNN
-F 3 "" H 950 3050 50  0001 C CNN
-	1    950  3050
+P 900 3050
+F 0 "#FLG?" H 900 3125 50  0001 C CNN
+F 1 "PWR_FLAG" H 900 3223 50  0000 C CNN
+F 2 "" H 900 3050 50  0001 C CNN
+F 3 "" H 900 3050 50  0001 C CNN
+	1    900  3050
 	-1   0    0    1
 $EndComp
@@
 Wire Wire Line
 	1700 4200 1700 4300
-Connection ~ 950  3050
 Wire Wire Line
-	950  3050 1050 3050
-Wire Wire Line
-	800  3050 950  3050
+	800  3050 900  3050
 $Comp
 L power:GND #PWR?
@@
 Text HLabel 13825 4625 0    50   Input ~ 0
 I2C1_SDA
-Text HLabel 13825 4725 0    50   Input ~ 0
-SPDIF_OUT
+Text HLabel 13825 4725 0    50   Output ~ 0
+SD_PWREN
 Text HLabel 13825 4825 0    50   Input ~ 0
-SPDIF_IN
+GPIO_AD_B1_03
 Text HLabel 13825 5325 0    50   Input ~ 0
 AUD_INT
@@
 Text HLabel 13825 5225 0    50   Input ~ 0
 GPIO_AD_B1_07
+$Comp
+L haathi_mayank:C_NP C?
+U 1 1 5AC009C6
+P 1350 3250
+F 0 "C?" H 1453 3288 40  0000 L CNN
+F 1 "0.1uF" H 1453 3212 40  0000 L CNN
+F 2 "" H 1350 3250 60  0000 C CNN
+F 3 "" H 1350 3250 60  0000 C CNN
+	1    1350 3250
+	1    0    0    -1
+$EndComp
+Wire Wire Line
+	1350 3050 1350 3100
+Connection ~ 1350 3050
+Wire Wire Line
+	1350 3050 1300 3050
+$Comp
+L power:GND #PWR?
+U 1 1 5AC5894C
+P 1350 3450
+F 0 "#PWR?" H 1350 3200 50  0001 C CNN
+F 1 "GND" H 1250 3350 50  0000 C CNN
+F 2 "" H 1350 3450 50  0001 C CNN
+F 3 "" H 1350 3450 50  0001 C CNN
+	1    1350 3450
+	1    0    0    -1
+$EndComp
+Wire Wire Line
+	1350 3400 1350 3450
+Connection ~ 900  3050
+Wire Wire Line
+	900  3050 1000 3050
 Wire Bus Line
 	21850 4000 21850 4750

Commit message: Removes the redundant APX809 voltage detector and its replaced by APX811, which receives input from a reset button.
Parts:
- removed U?: APX809S-26SR, symbol haathi_mayank:APX809S-26SR
- added U?: APX811, symbol haathi_mayank:APX811
Connections:
- net labels added: POR_BUTTON
- net labels removed: MCU_RESET_N
Other:
- note added: "Power Monitoring and Reset"
- note added: "Replace by 0E if \nRC isn't needed"
Changed lines of the file:
@@
 ONOFF
 Wire Wire Line
-	4350 3050 3250 3050
+	4350 3050 3050 3050
 $Comp
 L haathi_mayank:R R?
 U 1 1 5A7C045C
-P 3250 2650
-F 0 "R?" H 3320 2696 50  0000 L CNN
-F 1 "100k_DNP" H 3320 2605 50  0000 L CNN
-F 2 "" V 3180 2650 30  0000 C CNN
-F 3 "" H 3250 2650 30  0000 C CNN
-	1    3250 2650
+P 3050 2700
+F 0 "R?" H 3120 2746 50  0000 L CNN
+F 1 "100k_DNP" H 3120 2655 50  0000 L CNN
+F 2 "" V 2980 2700 30  0000 C CNN
+F 3 "" H 3050 2700 30  0000 C CNN
+	1    3050 2700
 	1    0    0    -1
 $EndComp
@@
 	3950 2950 3950 2850
 Wire Wire Line
-	3250 2800 3250 3050
-Connection ~ 3250 3050
+	3050 2850 3050 3050
+Connection ~ 3050 3050
 Wire Wire Line
-	3250 3050 3100 3050
-Wire Wire Line
-	3250 2500 3250 2400
+	3050 2550 3050 2400
 Text HLabel 2600 2400 0    50   BiDi ~ 0
 VDD_SNVS_IN
-Text HLabel 2200 2550 0    50   BiDi ~ 0
-MCU_RESET_N
-Wire Wire Line
-	3100 2550 3100 3050
-Connection ~ 3100 3050
-Wire Wire Line
-	2800 3050 3100 3050
 $Comp
 L power:GND #PWR?
@@
 L haathi_mayank:R R?
 U 1 1 5A7C3651
-P 2050 3050
-F 0 "R?" V 2257 3050 50  0000 C CNN
-F 1 "0E_DNP" V 2166 3050 50  0000 C CNN
-F 2 "" V 1980 3050 30  0000 C CNN
-F 3 "" H 2050 3050 30  0000 C CNN
-	1    2050 3050
+P 1700 3050
+F 0 "R?" V 1907 3050 50  0000 C CNN
+F 1 "0E_DNP" V 1816 3050 50  0000 C CNN
+F 2 "" V 1630 3050 30  0000 C CNN
+F 3 "" H 1700 3050 30  0000 C CNN
+	1    1700 3050
 	0    -1   -1   0
 $EndComp
 Wire Wire Line
-	1900 3050 1700 3050
+	1550 3050 1250 3050
 $Comp
 L haathi_mayank:R R?
 U 1 1 5A7C3889
-P 1150 3050
-F 0 "R?" V 1357 3050 50  0000 C CNN
-F 1 "1.5k 1%" V 1266 3050 50  0000 C CNN
-F 2 "" V 1080 3050 30  0000 C CNN
-F 3 "" H 1150 3050 30  0000 C CNN
-	1    1150 3050
-	0    -1   -1   0
+P 900 2750
+F 0 "R?" V 1107 2750 50  0000 C CNN
+F 1 "1.5k 1%" V 1016 2750 50  0000 C CNN
+F 2 "" V 830 2750 30  0000 C CNN
+F 3 "" H 900 2750 30  0000 C CNN
+	1    900  2750
+	1    0    0    -1
 $EndComp
 $Comp
 L power:PWR_FLAG #FLG?
 U 1 1 5A7C425A
-P 900 3050
-F 0 "#FLG?" H 900 3125 50  0001 C CNN
-F 1 "PWR_FLAG" H 900 3223 50  0000 C CNN
-F 2 "" H 900 3050 50  0001 C CNN
-F 3 "" H 900 3050 50  0001 C CNN
-	1    900  3050
-	-1   0    0    1
+P 900 2400
+F 0 "#FLG?" H 900 2475 50  0001 C CNN
+F 1 "PWR_FLAG" H 900 2573 50  0000 C CNN
+F 2 "" H 900 2400 50  0001 C CNN
+F 3 "" H 900 2400 50  0001 C CNN
+	1    900  2400
+	0    -1   -1   0
 $EndComp
 Wire Wire Line
-	2300 3800 2300 3050
+	2300 3900 2300 3050
 Connection ~ 2300 3050
 Wire Wire Line
-	2300 3050 2200 3050
-$Comp
-L haathi_mayank:APX809S-26SR U?
-U 1 1 5A7C6200
-P 1700 3800
-F 0 "U?" H 1422 3846 50  0000 R CNN
-F 1 "APX809S-26SR" H 1422 3755 50  0000 R CNN
-F 2 "" H 1550 3800 50  0001 C CNN
-F 3 "" H 1550 3800 50  0001 C CNN
-	1    1700 3800
-	1    0    0    -1
-$EndComp
+	2300 3050 1850 3050
 Wire Wire Line
-	2100 3800 2300 3800
+	2100 3900 2300 3900
 Wire Wire Line
-	1700 3400 1700 3050
-Connection ~ 1700 3050
+	1250 3750 1250 3050
 Wire Wire Line
-	1700 3050 1350 3050
+	1250 3050 900  3050
 $Comp
 L power:GND #PWR?
 U 1 1 5A7C68AE
-P 1700 4300
-F 0 "#PWR?" H 1700 4050 50  0001 C CNN
-F 1 "GND" H 1705 4127 50  0000 C CNN
-F 2 "" H 1700 4300 50  0001 C CNN
-F 3 "" H 1700 4300 50  0001 C CNN
-	1    1700 4300
+P 2450 4000
+F 0 "#PWR?" H 2450 3750 50  0001 C CNN
+F 1 "GND" H 2455 3827 50  0000 C CNN
+F 2 "" H 2450 4000 50  0001 C CNN
+F 3 "" H 2450 4000 50  0001 C CNN
+	1    2450 4000
 	1    0    0    -1
 $EndComp
 Wire Wire Line
-	1700 4200 1700 4300
-Wire Wire Line
-	800  3050 900  3050
+	900  2200 900  2400
 $Comp
 L power:GND #PWR?
@@
 L power:+3V3 #PWR?
 U 1 1 5A9B420A
-P 800 3050
-F 0 "#PWR?" H 800 2900 50  0001 C CNN
-F 1 "+3V3" H 815 3223 50  0000 C CNN
-F 2 "" H 800 3050 50  0001 C CNN
-F 3 "" H 800 3050 50  0001 C CNN
-	1    800  3050
+P 900 2200
+F 0 "#PWR?" H 900 2050 50  0001 C CNN
+F 1 "+3V3" H 915 2373 50  0000 C CNN
+F 2 "" H 900 2200 50  0001 C CNN
+F 3 "" H 900 2200 50  0001 C CNN
+	1    900  2200
 	1    0    0    -1
 $EndComp
@@
 Wire Wire Line
 	10325 11050 11100 11050
-Wire Wire Line
-	2200 2550 3100 2550
-Text Label 2325 2550 0    50   ~ 0
-MCU_RESET_N
-Wire Wire Line
-	2600 2400 3250 2400
 Text Label 2700 2400 0    50   ~ 0
 VDD_SNVS_IN
@@
 L haathi_mayank:C_NP C?
 U 1 1 5AC009C6
-P 1350 3250
-F 0 "C?" H 1453 3288 40  0000 L CNN
-F 1 "0.1uF" H 1453 3212 40  0000 L CNN
-F 2 "" H 1350 3250 60  0000 C CNN
-F 3 "" H 1350 3250 60  0000 C CNN
-	1    1350 3250
+P 900 3300
+F 0 "C?" H 1003 3338 40  0000 L CNN
+F 1 "0.1uF" H 1003 3262 40  0000 L CNN
+F 2 "" H 900 3300 60  0000 C CNN
+F 3 "" H 900 3300 60  0000 C CNN
+	1    900  3300
 	1    0    0    -1
 $EndComp
 Wire Wire Line
-	1350 3050 1350 3100
-Connection ~ 1350 3050
+	900  3050 900  3150
+Connection ~ 900  3050
 Wire Wire Line
-	1350 3050 1300 3050
+	900  3050 900  2900
 $Comp
 L power:GND #PWR?
 U 1 1 5AC5894C
-P 1350 3450
-F 0 "#PWR?" H 1350 3200 50  0001 C CNN
-F 1 "GND" H 1250 3350 50  0000 C CNN
-F 2 "" H 1350 3450 50  0001 C CNN
-F 3 "" H 1350 3450 50  0001 C CNN
-	1    1350 3450
+P 900 3500
+F 0 "#PWR?" H 900 3250 50  0001 C CNN
+F 1 "GND" H 800 3400 50  0000 C CNN
+F 2 "" H 900 3500 50  0001 C CNN
+F 3 "" H 900 3500 50  0001 C CNN
+	1    900  3500
 	1    0    0    -1
 $EndComp
 Wire Wire Line
-	1350 3400 1350 3450
-Connection ~ 900  3050
+	900  3450 900  3500
+Wire Wire Line
+	2800 3050 3050 3050
+$Comp
+L haathi_mayank:APX811 U?
+U 1 1 5AC13820
+P 1700 3800
+F 0 "U?" H 1675 4122 50  0000 C CNN
+F 1 "APX811" H 1675 4031 50  0000 C CNN
+F 2 "" H 1550 3700 50  0001 C CNN
+F 3 "" H 1550 3700 50  0001 C CNN
+	1    1700 3800
+	-1   0    0    -1
+$EndComp
+Wire Wire Line
+	2100 3750 2450 3750
+Wire Wire Line
+	2450 3750 2450 4000
+Connection ~ 1250 3050
+Wire Wire Line
+	1250 3750 1350 3750
+Connection ~ 900  2400
+Wire Wire Line
+	900  2400 900  2600
+Text HLabel 1100 3900 0    50   Input ~ 0
+POR_BUTTON
+Wire Wire Line
+	1100 3900 1350 3900
 Wire Wire Line
-	900  3050 1000 3050
+	2600 2400 3050 2400
 Wire Bus Line
 	21850 4000 21850 4750
@@
 Wire Bus Line
 	9425 8000 9425 9800
+Text Notes 1200 4100 0    50   ~ 0
+Power Monitoring and Reset
+Text Notes 950  2600 0    50   ~ 0
+Replace by 0E if \nRC isn't needed
 $EndSCHEMATC

Commit message: Replaces 3V3 with DCDC_IN for the DCDC of the imxrt. Adds MCU_RESET_N for the SD card power off.
Connections:
- net labels added: DCDC_IN, MCU_RESET_N
- wire segments 519 -> 521
Changed lines of the file:
@@
 EESchema Schematic File Version 4
-LIBS:haathi_schematic-cache
+LIBS:haathi_cpu-cache
 EELAYER 26 0
 EELAYER END
 $Descr A2 23386 16535
 encoding utf-8
-Sheet 1 9
+Sheet 1 1
 Title "haathi_cam"
 Date "2018-03-11"
@@
 $EndComp
 Wire Wire Line
-	2300 3900 2300 3050
+	2300 3900 2300 3250
 Connection ~ 2300 3050
 Wire Wire Line
@@
 $Comp
 L power:+3V3 #PWR?
-U 1 1 5A9B411A
-P 10350 2550
-F 0 "#PWR?" H 10350 2400 50  0001 C CNN
-F 1 "+3V3" H 10365 2723 50  0000 C CNN
-F 2 "" H 10350 2550 50  0001 C CNN
-F 3 "" H 10350 2550 50  0001 C CNN
-	1    10350 2550
-	1    0    0    -1
-$EndComp
-$Comp
-L power:+3V3 #PWR?
 U 1 1 5A9B420A
 P 900 2200
@@
 Wire Wire Line
 	2600 2400 3050 2400
+Text Notes 1200 4100 0    50   ~ 0
+Power Monitoring and Reset
+Text Notes 950  2600 0    50   ~ 0
+Replace by 0E if \nRC isn't needed
+Text HLabel 2250 3250 0    50   Input ~ 0
+MCU_RESET_N
+Wire Wire Line
+	2250 3250 2300 3250
 Wire Bus Line
 	21850 4000 21850 4750
@@
 Wire Bus Line
 	9425 8000 9425 9800
-Text Notes 1200 4100 0    50   ~ 0
-Power Monitoring and Reset
-Text Notes 950  2600 0    50   ~ 0
-Replace by 0E if \nRC isn't needed
+Connection ~ 2300 3250
+Wire Wire Line
+	2300 3250 2300 3050
+Text HLabel 10350 2550 2    50   Input ~ 0
+DCDC_IN
 $EndSCHEMATC

Commit message: CPU, Interfaces, SDRAM top sheet wiring done, CPU bootcfg local labels fixed
Connections:
- net labels removed: GPIO_B0_5, GPIO_B0_6, GPIO_B0_7, GPIO_B0_8, GPIO_B0_9
- wire segments 521 -> 563
Changed lines of the file:
@@
 GPIO_B0_04
 Text HLabel 6550 13050 2    50   Input ~ 0
-GPIO_B0_5
+GPIO_B0_05
 Text HLabel 6550 13150 2    50   Input ~ 0
-GPIO_B0_6
+GPIO_B0_06
 Text HLabel 6550 13250 2    50   Input ~ 0
-GPIO_B0_7
+GPIO_B0_07
 Text HLabel 6550 13350 2    50   Input ~ 0
-GPIO_B0_8
+GPIO_B0_08
 Text HLabel 6550 13450 2    50   Input ~ 0
-GPIO_B0_9
+GPIO_B0_09
 Text HLabel 6550 13550 2    50   Input ~ 0
 GPIO_B0_10
@@
 	4050 13250 5050 13250
 Wire Wire Line
-	4050 13350 6550 13350
+	4050 13350 6500 13350
 Wire Wire Line
 	4050 13450 4850 13450
@@
 	4050 13650 4650 13650
 Wire Wire Line
-	6550 14000 4450 14000
-Wire Wire Line
-	6550 14100 4400 14100
-Wire Wire Line
-	6550 14200 4350 14200
-Wire Wire Line
-	6550 14300 4300 14300
+	6550 14000 6500 14000
+Wire Wire Line
+	6550 14100 6500 14100
+Wire Wire Line
+	6550 14200 6500 14200
+Wire Wire Line
+	6550 14300 6500 14300
 Text Label 5150 12950 0    50   ~ 0
 BT_CFG[0]
@@
 GPIO_AD_B0_05
 Wire Wire Line
-	6550 14800 6050 14800
+	6550 14800 6500 14800
 Text Label 5100 14700 0    50   ~ 0
 BOOT_MODE[0]
@@
 Connection ~ 6250 13550
 Wire Wire Line
-	6250 13550 6550 13550
+	6250 13550 6500 13550
 Wire Wire Line
 	6150 12600 6150 14700
 Connection ~ 6150 14700
 Wire Wire Line
-	6150 14700 6550 14700
+	6150 14700 6500 14700
 Wire Wire Line
 	6050 12600 6050 14800
@@
 Connection ~ 5650 12950
 Wire Wire Line
-	5650 12950 6550 12950
+	5650 12950 6500 12950
 Wire Wire Line
 	5450 11800 5450 13050
 Connection ~ 5450 13050
 Wire Wire Line
-	5450 13050 6550 13050
+	5450 13050 6500 13050
 Wire Wire Line
 	5250 11800 5250 13150
 Connection ~ 5250 13150
 Wire Wire Line
-	5250 13150 6550 13150
+	5250 13150 6500 13150
 Wire Wire Line
 	5050 11800 5050 13250
 Connection ~ 5050 13250
 Wire Wire Line
-	5050 13250 6550 13250
+	5050 13250 6500 13250
 Wire Wire Line
 	4850 11800 4850 13450
 Connection ~ 4850 13450
 Wire Wire Line
-	4850 13450 6550 13450
+	4850 13450 6500 13450
 Wire Wire Line
 	4650 11800 4650 13650
 Connection ~ 4650 13650
 Wire Wire Line
-	4650 13650 6550 13650
+	4650 13650 6500 13650
 Wire Wire Line
 	5650 11500 5650 11300
@@
 Text HLabel 10350 2550 2    50   Input ~ 0
 DCDC_IN
+Wire Wire Line
+	6500 12950 6500 12900
+Wire Wire Line
+	6500 12900 7200 12900
+Connection ~ 6500 12950
+Wire Wire Line
+	6500 12950 6550 12950
+Wire Wire Line
+	6500 13000 7200 13000
+Wire Wire Line
+	6500 13100 7200 13100
+Wire Wire Line
+	6500 13200 7200 13200
+Wire Wire Line
+	6500 13300 7200 13300
+Wire Wire Line
+	6500 13400 7200 13400
+Wire Wire Line
+	6500 13500 7200 13500
+Wire Wire Line
+	6500 13600 7200 13600
+Wire Wire Line
+	6500 13050 6500 13000
+Connection ~ 6500 13050
+Wire Wire Line
+	6500 13050 6550 13050
+Wire Wire Line
+	6500 13150 6500 13100
+Wire Wire Line
+	6500 13250 6500 13200
+Wire Wire Line
+	6500 13350 6500 13300
+Wire Wire Line
+	6500 13450 6500 13400
+Connection ~ 6500 13150
+Wire Wire Line
+	6500 13150 6550 13150
+Connection ~ 6500 13250
+Wire Wire Line
+	6500 13250 6550 13250
+Connection ~ 6500 13350
+Wire Wire Line
+	6500 13350 6550 13350
+Connection ~ 6500 13450
+Wire Wire Line
+	6500 13450 6550 13450
+Wire Wire Line
+	6500 13500 6500 13550
+Connection ~ 6500 13550
+Wire Wire Line
+	6500 13550 6550 13550
+Wire Wire Line
+	6500 13600 6500 13650
+Connection ~ 6500 13650
+Wire Wire Line
+	6500 13650 6550 13650
+Wire Wire Line
+	6500 14000 6500 13950
+Wire Wire Line
+	6500 13950 7200 13950
+Connection ~ 6500 14000
+Wire Wire Line
+	6500 14000 4450 14000
+Wire Wire Line
+	6500 14050 7200 14050
+Wire Wire Line
+	6500 14150 7200 14150
+Wire Wire Line
+	6500 14250 7200 14250
+Wire Wire Line
+	6500 14650 7200 14650
+Wire Wire Line
+	6500 14750 7200 14750
+Wire Wire Line
+	6500 14050 6500 14100
+Connection ~ 6500 14100
+Wire Wire Line
+	6500 14100 4400 14100
+Wire Wire Line
+	6500 14150 6500 14200
+Connection ~ 6500 14200
+Wire Wire Line
+	6500 14200 4350 14200
+Wire Wire Line
+	6500 14250 6500 14300
+Connection ~ 6500 14300
+Wire Wire Line
+	6500 14300 4300 14300
+Wire Wire Line
+	6500 14650 6500 14700
+Connection ~ 6500 14700
+Wire Wire Line
+	6500 14700 6550 14700
+Wire Wire Line
+	6500 14750 6500 14800
 Wire Bus Line
 	21850 4000 21850 4750
@@
 Wire Bus Line
 	9425 8000 9425 9800
+Connection ~ 6500 14800
+Wire Wire Line
+	6500 14800 6050 14800
+Text Label 7200 12900 0    50   ~ 0
+GPIO_B0_04
+Text Label 7200 13000 0    50   ~ 0
+GPIO_B0_05
+Text Label 7200 13100 0    50   ~ 0
+GPIO_B0_06
+Text Label 7200 13200 0    50   ~ 0
+GPIO_B0_07
+Text Label 7200 13300 0    50   ~ 0
+GPIO_B0_08
+Text Label 7200 13400 0    50   ~ 0
+GPIO_B0_09
+Text Label 7200 13500 0    50   ~ 0
+GPIO_B0_10
+Text Label 7200 13600 0    50   ~ 0
+GPIO_B0_11
+Text Label 7200 13950 0    50   ~ 0
+GPIO_B0_12
+Text Label 7200 14050 0    50   ~ 0
+GPIO_B0_13
+Text Label 7200 14150 0    50   ~ 0
+GPIO_B0_14
+Text Label 7200 14250 0    50   ~ 0
+GPIO_B0_15
+Text Label 7200 14650 0    50   ~ 0
+GPIO_AD_B0_04
+Text Label 7200 14750 0    50   ~ 0
+GPIO_AD_B0_05
 $EndSCHEMATC
