File: kicad/haathi_power.sch (KiCad schematic (older format))
At the start: 12 parts

Commit message: Anool, Memory schematic WIP
Parts:
- gave numbers to parts that had none: 12
Changed lines of the file:
@@
 $EndDescr
 $Comp
-L haathi_mayank:TPS62142 U?
+L haathi_mayank:TPS62142 U1
 U 1 1 5A6DEEB7
 P 4600 1850
-F 0 "U?" H 4575 2415 50  0000 C CNN
+F 0 "U1" H 4575 2415 50  0000 C CNN
 F 1 "TPS62142" H 4575 2324 50  0000 C CNN
 F 2 "" H 4700 1850 50  0001 C CNN
@@
 $EndComp
 $Comp
-L haathi_mayank:C_NP C?
+L haathi_mayank:C_NP C4
 U 1 1 5A6DEFBB
 P 5250 2400
-F 0 "C?" H 5353 2438 40  0000 L CNN
+F 0 "C4" H 5353 2438 40  0000 L CNN
 F 1 "3.3nF" H 5353 2362 40  0000 L CNN
 F 2 "" H 5250 2400 60  0000 C CNN
@@
 $EndComp
 $Comp
-L haathi_mayank:C_POL C?
+L haathi_mayank:C_POL C3
 U 1 1 5A6DF04E
 P 5650 2150
-F 0 "C?" H 5753 2188 40  0000 L CNN
+F 0 "C3" H 5753 2188 40  0000 L CNN
 F 1 "10uF" H 5753 2112 40  0000 L CNN
 F 2 "" H 5650 2150 60  0000 C CNN
@@
 $EndComp
 $Comp
-L haathi_mayank:IND_SML L?
+L haathi_mayank:IND_SML L4
 U 1 1 5A6DF0E7
 P 3700 1550
-F 0 "L?" H 3700 1744 40  0000 C CNN
+F 0 "L4" H 3700 1744 40  0000 C CNN
 F 1 "2.2uH" H 3700 1668 40  0000 C CNN
 F 2 "" H 3700 1550 60  0000 C CNN
@@
 	4000 2250 4000 2350
 $Comp
-L power:GND #PWR?
+L power:GND #PWR08
 U 1 1 5A6E020F
 P 3650 2050
-F 0 "#PWR?" H 3650 1800 50  0001 C CNN
+F 0 "#PWR08" H 3650 1800 50  0001 C CNN
 F 1 "GND" H 3655 1877 50  0000 C CNN
 F 2 "" H 3650 2050 50  0001 C CNN
@@
 $EndComp
 $Comp
-L power:GND #PWR?
+L power:GND #PWR06
 U 1 1 5A6E024F
 P 5500 1650
-F 0 "#PWR?" H 5500 1400 50  0001 C CNN
+F 0 "#PWR06" H 5500 1400 50  0001 C CNN
 F 1 "GND" H 5505 1477 50  0000 C CNN
 F 2 "" H 5500 1650 50  0001 C CNN
@@
 $EndComp
 $Comp
-L power:GND #PWR?
+L power:GND #PWR010
 U 1 1 5A6E0298
 P 5250 2650
-F 0 "#PWR?" H 5250 2400 50  0001 C CNN
+F 0 "#PWR010" H 5250 2400 50  0001 C CNN
 F 1 "GND" H 5255 2477 50  0000 C CNN
 F 2 "" H 5250 2650 50  0001 C CNN
@@
 $EndComp
 $Comp
-L power:GND #PWR?
+L power:GND #PWR07
 U 1 1 5A6E02C9
 P 2900 2000
-F 0 "#PWR?" H 2900 1750 50  0001 C CNN
+F 0 "#PWR07" H 2900 1750 50  0001 C CNN
 F 1 "GND" H 2905 1827 50  0000 C CNN
 F 2 "" H 2900 2000 50  0001 C CNN
@@
 	5250 2600 5250 2650
 $Comp
-L power:GND #PWR?
+L power:GND #PWR09
 U 1 1 5A6E2969
 P 4000 2350
-F 0 "#PWR?" H 4000 2100 50  0001 C CNN
+F 0 "#PWR09" H 4000 2100 50  0001 C CNN
 F 1 "GND" H 4005 2177 50  0000 C CNN
 F 2 "" H 4000 2350 50  0001 C CNN
@@
 Connection ~ 4000 1550
 $Comp
-L haathi_mayank:R R?
+L haathi_mayank:R R2
 U 1 1 5A6E447F
 P 3350 1700
-F 0 "R?" H 3420 1746 50  0000 L CNN
+F 0 "R2" H 3420 1746 50  0000 L CNN
 F 1 "100k" H 3420 1655 50  0000 L CNN
 F 2 "" V 3280 1700 30  0000 C CNN
@@
 $EndComp
 $Comp
-L haathi_mayank:C_POL C?
+L haathi_mayank:C_POL C2
 U 1 1 5A6E57C1
 P 2900 1700
-F 0 "C?" H 3003 1738 40  0000 L CNN
+F 0 "C2" H 3003 1738 40  0000 L CNN
 F 1 "22uF" H 3003 1662 40  0000 L CNN
 F 2 "" H 2900 1700 60  0000 C CNN
@@
 	5250 1750 5000 1750
 $Comp
-L power:PWR_FLAG #FLG?
+L power:PWR_FLAG #FLG02
 U 1 1 5A6E82C3
 P 5900 1950
-F 0 "#FLG?" H 5900 2025 50  0001 C CNN
+F 0 "#FLG02" H 5900 2025 50  0001 C CNN
 F 1 "PWR_FLAG" H 5900 2124 50  0000 C CNN
 F 2 "" H 5900 1950 50  0001 C CNN
@@
 Connection ~ 5900 1950
 $Comp
-L power:PWR_FLAG #FLG?
+L power:PWR_FLAG #FLG03
 U 1 1 5A6E8353
 P 5650 2600
-F 0 "#FLG?" H 5650 2675 50  0001 C CNN
+F 0 "#FLG03" H 5650 2675 50  0001 C CNN
 F 1 "PWR_FLAG" V 5650 2728 50  0000 L CNN
 F 2 "" H 5650 2600 50  0001 C CNN
@@
 Connection ~ 5650 2600
 $Comp
-L power:VCC #PWR?
+L power:VCC #PWR05
 U 1 1 5A6E83DA
 P 2400 1550
-F 0 "#PWR?" H 2400 1400 50  0001 C CNN
+F 0 "#PWR05" H 2400 1400 50  0001 C CNN
 F 1 "VCC" H 2417 1723 50  0000 C CNN
 F 2 "" H 2400 1550 50  0001 C CNN
@@
 $EndComp
 $Comp
-L power:PWR_FLAG #FLG?
+L power:PWR_FLAG #FLG01
 U 1 1 5A6E843F
 P 2800 1550
-F 0 "#FLG?" H 2800 1625 50  0001 C CNN
+F 0 "#FLG01" H 2800 1625 50  0001 C CNN
 F 1 "PWR_FLAG" H 2800 1724 50  0000 C CNN
 F 2 "" H 2800 1550 50  0001 C CNN
@@
 VIN
 $Comp
-L haathi_mayank:batt_coin_holder BT?
+L haathi_mayank:batt_coin_holder BT1
 U 1 1 5A6EAFEE
 P 2800 3450
-F 0 "BT?" H 2918 3488 40  0000 L CNN
+F 0 "BT1" H 2918 3488 40  0000 L CNN
 F 1 "batt_coin_holder" H 2918 3412 40  0000 L CNN
 F 2 "" V 2800 3425 60  0000 C CNN
@@
 	2800 3300 3300 3300
 $Comp
-L power:GND #PWR?
+L power:GND #PWR011
 U 1 1 5A6EBB3E
 P 2800 3650
-F 0 "#PWR?" H 2800 3400 50  0001 C CNN
+F 0 "#PWR011" H 2800 3400 50  0001 C CNN
 F 1 "GND" H 2805 3477 50  0000 C CNN
 F 2 "" H 2800 3650 50  0001 C CNN
@@
 VDD_SNVS_IN
 $Comp
-L haathi_mayank:C_NP C?
+L haathi_mayank:C_NP C5
 U 1 1 5A6EC61E
 P 3300 3450
-F 0 "C?" H 3403 3488 40  0000 L CNN
+F 0 "C5" H 3403 3488 40  0000 L CNN
 F 1 "3.3nF" H 3403 3412 40  0000 L CNN
 F 2 "" H 3300 3450 60  0000 C CNN
@@
 SNVS
 $Comp
-L haathi_mayank:R R?
+L haathi_mayank:R R3
 U 1 1 5A6ED3C7
 P 7300 1700
-F 0 "R?" H 7370 1746 50  0000 L CNN
+F 0 "R3" H 7370 1746 50  0000 L CNN
 F 1 "0" H 7370 1655 50  0000 L CNN
 F 2 "" V 7230 1700 30  0000 C CNN
@@
 $EndComp
 $Comp
-L haathi_mayank:R R?
+L haathi_mayank:R R4
 U 1 1 5A6ED45D
 P 7650 1700
-F 0 "R?" H 7720 1746 50  0000 L CNN
+F 0 "R4" H 7720 1746 50  0000 L CNN
 F 1 "0" H 7720 1655 50  0000 L CNN
 F 2 "" V 7580 1700 30  0000 C CNN
@@
 $EndComp
 $Comp
-L haathi_mayank:R R?
+L haathi_mayank:R R5
 U 1 1 5A6ED497
 P 7950 1700
-F 0 "R?" H 8020 1746 50  0000 L CNN
+F 0 "R5" H 8020 1746 50  0000 L CNN
 F 1 "0" H 8020 1655 50  0000 L CNN
 F 2 "" V 7880 1700 30  0000 C CNN
@@
 $EndComp
 $Comp
-L haathi_mayank:R R?
+L haathi_mayank:R R6
 U 1 1 5A6ED4CD
 P 8250 1700
-F 0 "R?" H 8320 1746 50  0000 L CNN
+F 0 "R6" H 8320 1746 50  0000 L CNN
 F 1 "0" H 8320 1655 50  0000 L CNN
 F 2 "" V 8180 1700 30  0000 C CNN

Commit message: Mayank, Power added decoupling and buttons
Parts:
- added BT?: Battery, symbol haathi_mayank:Battery
- added C? (x2): 22uF, symbol haathi_mayank:C_POL
- added C? (x9): 4.7uF, symbol haathi_mayank:C_POL
- added C? (x12): 0.22uF, symbol haathi_mayank:C_NP
- added C? (x8): 0.1uF, symbol haathi_mayank:C_NP
- added C?: 1uF, symbol haathi_mayank:C_POL
- added R? (x3): 0, symbol haathi_mayank:R
- added S? (x3): SW-SPST-M, symbol haathi_mayank:SW-SPST-M
- added SW?: SW_SPDT, symbol haathi_mayank:SW_SPDT
- C?: renamed from C5; value 3.3nF -> 0.22uF
- renumbered BT1 to BT?, C4 to C?, C3 to C?, C2 to C?, L4 to L?, R2 to R?, R3 to R?, R4 to R?, R5 to R?, R6 to R?, U1 to U?
Connections:
- net labels added: DCDC_IN, NVCC_EMC, NVCC_GPIO, NVCC_SD0, NVCC_SD1, ONOFF, POR_BUTTON, USER_BUTTON, VDDA_ADC_3P3, VDD_HIGH_CAP, VDD_HIGH_IN, VDD_SNVS_CAP, VDD_SOC_IN, V_BATT, V_USB
- wire segments 50 -> 154
Other:
- note added: "Battery"
- note added: "Buttons"
- note added: "CPU ONOFF Button"
- note added: "Decoupling Capacitors\n"
- note added: "Power Input Selection"
- note added: "Supply Nets"
- note added: "System Reset Button"
- note added: "User Button"

Commit message: Mayank, power ckt, corrections and reset ckt
Parts:
- removed BT?: Battery, symbol haathi_mayank:Battery
- removed C? (x3): 22uF, symbol haathi_mayank:C_POL
- removed C? (x9): 4.7uF, symbol haathi_mayank:C_POL
- removed C?: 1uF, symbol haathi_mayank:C_POL
- removed C?: 0.1uF, symbol haathi_mayank:C_NP
- removed SW?: SW_SPDT, symbol haathi_mayank:SW_SPDT
- added C? (x3): 0.1uF, symbol haathi_mayank:C_NP
- added C?: 1uF, symbol haathi_mayank:C_NP
- added C? (x9): 4.7uF, symbol haathi_mayank:C_NP
- added C? (x4): 22uF, symbol haathi_mayank:C_NP
- added D? (x2): D_Schottky, symbol haathi_mayank:D_Schottky
- added J?: Barrel_Jack, symbol haathi_mayank:Barrel_Jack
- added J?: Conn_01x02, symbol haathi_mayank:Conn_01x02
- added SW?: SW_SP3T, symbol haathi_mayank:SW_SP3T
- added U?: APX811, symbol haathi_mayank:APX811
Connections:
- net labels added: MCU_RESET_N
- wire segments 154 -> 183
- no-connect marks 0 -> 1
Other:
- note added: "OFF"
- note added: "Power Monitoring and Reset"

Commit message: Mayank, reverse polarity protection and test points
Parts:
- added Q?: Q_PMOS_GDS, symbol haathi_mayank:Q_PMOS_GDS
- added TP? (x3): Test_Point_Probe, symbol haathi_mayank:Test_Point_Probe
- C?: value 10uF -> 22uF
Connections:
- net labels added: V_INPUT
- wire segments 183 -> 187
Other:
- note added: "Reverse Polarity Protection"
Changed lines of the file:
@@
 EESchema Schematic File Version 4
+LIBS:haathi-cache
 EELAYER 26 0
 EELAYER END
 $Descr A4 11693 8268
 encoding utf-8
-Sheet 1 1
+Sheet 4 12
 Title ""
 Date ""
@@
 P 4200 1700
 F 0 "C?" H 4303 1738 40  0000 L CNN
-F 1 "10uF" H 4303 1662 40  0000 L CNN
+F 1 "22uF" H 4303 1662 40  0000 L CNN
 F 2 "" H 4200 1700 60  0000 C CNN
 F 3 "" H 4200 1700 60  0000 C CNN
@@
 L power:VCC #PWR?
 U 1 1 5A6FED5F
-P 7450 1250
-F 0 "#PWR?" H 7450 1100 50  0001 C CNN
-F 1 "VCC" H 7467 1423 50  0000 C CNN
-F 2 "" H 7450 1250 50  0001 C CNN
-F 3 "" H 7450 1250 50  0001 C CNN
-	1    7450 1250
+P 7100 1250
+F 0 "#PWR?" H 7100 1100 50  0001 C CNN
+F 1 "VCC" H 7117 1423 50  0000 C CNN
+F 2 "" H 7100 1250 50  0001 C CNN
+F 3 "" H 7100 1250 50  0001 C CNN
+	1    7100 1250
 	1    0    0    -1
 $EndComp
@@
 $EndComp
 Connection ~ 7500 1250
-Wire Wire Line
-	7500 1250 7450 1250
 Text HLabel 8250 1250 2    50   Input ~ 0
 DCDC_IN
@@
 Text Label 4750 1500 0    50   ~ 0
 VIN
-Text Label 5600 1300 2    50   ~ 0
-VIN
 Text Label 6400 1300 0    50   ~ 0
 V_BATT
@@
 L haathi_mayank:SW-SPST-M S?
 U 1 1 5A81CDE8
-P 6100 2100
-F 0 "S?" H 6100 2402 40  0000 C CNB
-F 1 "SW-SPST-M" H 6100 2326 40  0000 C CNB
-F 2 "" H 6100 2100 60  0000 C CNN
-F 3 "" H 6100 2100 60  0000 C CNN
-	1    6100 2100
+P 9600 4350
+F 0 "S?" H 9600 4652 40  0000 C CNB
+F 1 "SW-SPST-M" H 9600 4576 40  0000 C CNB
+F 2 "" H 9600 4350 60  0000 C CNN
+F 3 "" H 9600 4350 60  0000 C CNN
+	1    9600 4350
 	1    0    0    -1
 $EndComp
@@
 L haathi_mayank:SW-SPST-M S?
 U 1 1 5A81CEB6
-P 6100 2550
-F 0 "S?" H 6100 2852 40  0000 C CNB
-F 1 "SW-SPST-M" H 6100 2776 40  0000 C CNB
-F 2 "" H 6100 2550 60  0000 C CNN
-F 3 "" H 6100 2550 60  0000 C CNN
-	1    6100 2550
+P 9600 4800
+F 0 "S?" H 9600 5102 40  0000 C CNB
+F 1 "SW-SPST-M" H 9600 5026 40  0000 C CNB
+F 2 "" H 9600 4800 60  0000 C CNN
+F 3 "" H 9600 4800 60  0000 C CNN
+	1    9600 4800
 	1    0    0    -1
 $EndComp
@@
 L haathi_mayank:SW-SPST-M S?
 U 1 1 5A81CF46
-P 6100 3050
-F 0 "S?" H 6100 3352 40  0000 C CNB
-F 1 "SW-SPST-M" H 6100 3276 40  0000 C CNB
-F 2 "" H 6100 3050 60  0000 C CNN
-F 3 "" H 6100 3050 60  0000 C CNN
-	1    6100 3050
+P 9600 5300
+F 0 "S?" H 9600 5602 40  0000 C CNB
+F 1 "SW-SPST-M" H 9600 5526 40  0000 C CNB
+F 2 "" H 9600 5300 60  0000 C CNN
+F 3 "" H 9600 5300 60  0000 C CNN
+	1    9600 5300
 	1    0    0    -1
 $EndComp
@@
 L power:GND #PWR?
 U 1 1 5A81D0A2
-P 5650 3150
-F 0 "#PWR?" H 5650 2900 50  0001 C CNN
-F 1 "GND" H 5655 2977 50  0000 C CNN
-F 2 "" H 5650 3150 50  0001 C CNN
-F 3 "" H 5650 3150 50  0001 C CNN
-	1    5650 3150
-	1    0    0    -1
-$EndComp
-Wire Wire Line
-	5950 2100 5650 2100
-Wire Wire Line
-	5650 2100 5650 2550
-Wire Wire Line
-	5950 2550 5650 2550
-Connection ~ 5650 2550
-Wire Wire Line
-	5650 2550 5650 3050
-Wire Wire Line
-	5950 3050 5650 3050
-Connection ~ 5650 3050
-Wire Wire Line
-	5650 3050 5650 3150
-Wire Wire Line
-	6250 3050 6450 3050
-Wire Wire Line
-	6250 2550 6450 2550
-Wire Wire Line
-	6250 2100 6450 2100
-Text HLabel 6450 2100 2    50   Input ~ 0
+P 9150 5400
+F 0 "#PWR?" H 9150 5150 50  0001 C CNN
+F 1 "GND" H 9155 5227 50  0000 C CNN
+F 2 "" H 9150 5400 50  0001 C CNN
+F 3 "" H 9150 5400 50  0001 C CNN
+	1    9150 5400
+	1    0    0    -1
+$EndComp
+Wire Wire Line
+	9450 4350 9150 4350
+Wire Wire Line
+	9150 4350 9150 4800
+Wire Wire Line
+	9450 4800 9150 4800
+Connection ~ 9150 4800
+Wire Wire Line
+	9150 4800 9150 5300
+Wire Wire Line
+	9450 5300 9150 5300
+Connection ~ 9150 5300
+Wire Wire Line
+	9150 5300 9150 5400
+Wire Wire Line
+	9750 5300 9950 5300
+Wire Wire Line
+	9750 4800 9950 4800
+Wire Wire Line
+	9750 4350 9950 4350
+Text HLabel 9950 4350 2    50   Input ~ 0
 ONOFF
-Text HLabel 6450 2550 2    50   Input ~ 0
+Text HLabel 9950 4800 2    50   Input ~ 0
 POR_BUTTON
-Text HLabel 6450 3050 2    50   Input ~ 0
+Text HLabel 9950 5300 2    50   Input ~ 0
 USER_BUTTON
-Text Notes 5250 2100 0    50   ~ 0
+Text Notes 8750 4350 0    50   ~ 0
 Buttons
-Text Notes 6450 2250 0    50   ~ 0
+Text Notes 9950 4500 0    50   ~ 0
 CPU ONOFF Button
-Text Notes 6450 2700 0    50   ~ 0
+Text Notes 9950 4950 0    50   ~ 0
 System Reset Button
-Text Notes 6450 3200 0    50   ~ 0
+Text Notes 9950 5450 0    50   ~ 0
 User Button
 Wire Wire Line
@@
 Text HLabel 2950 3050 2    50   Input ~ 0
 POR_BUTTON
-Wire Wire Line
-	5950 2150 5950 2100
-Connection ~ 5950 2100
-Wire Wire Line
-	6250 2150 6250 2100
-Connection ~ 6250 2100
-Wire Wire Line
-	6250 2600 6250 2550
-Connection ~ 6250 2550
-Wire Wire Line
-	5950 2600 5950 2550
-Connection ~ 5950 2550
-Wire Wire Line
-	5950 3100 5950 3050
-Connection ~ 5950 3050
-Wire Wire Line
-	6250 3100 6250 3050
-Connection ~ 6250 3050
 $Comp
 L power:VCC #PWR?
@@
 Text Notes 2700 2550 2    50   ~ 0
 Power Monitoring and Reset
+Text Label 5600 1300 2    50   ~ 0
+V_INPUT
+$Comp
+L haathi_mayank:Q_PMOS_GDS Q?
+U 1 1 5A778B6C
+P 6100 2050
+F 0 "Q?" V 6443 2050 50  0000 C CNN
+F 1 "Q_PMOS_GDS" V 6352 2050 50  0000 C CNN
+F 2 "" H 6300 2150 50  0001 C CNN
+F 3 "~" H 6100 2050 50  0001 C CNN
+	1    6100 2050
+	0    -1   -1   0
+$EndComp
+Text Label 6450 1950 0    50   ~ 0
+VIN
+Text Label 5800 1950 2    50   ~ 0
+V_INPUT
+$Comp
+L power:GND #PWR?
+U 1 1 5A78CC9B
+P 6100 2350
+F 0 "#PWR?" H 6100 2100 50  0001 C CNN
+F 1 "GND" H 6105 2177 50  0000 C CNN
+F 2 "" H 6100 2350 50  0001 C CNN
+F 3 "" H 6100 2350 50  0001 C CNN
+	1    6100 2350
+	1    0    0    -1
+$EndComp
+Wire Wire Line
+	6100 2250 6100 2300
+Wire Wire Line
+	5800 1950 5900 1950
+Wire Wire Line
+	6300 1950 6350 1950
+Text Notes 5600 1650 0    50   ~ 0
+Reverse Polarity Protection
+Wire Wire Line
+	7100 1250 7300 1250
+$Comp
+L haathi_mayank:Test_Point_Probe TP?
+U 1 1 5A7E05E8
+P 7300 1100
+F 0 "TP?" H 7453 1202 50  0000 L CNN
+F 1 "Test_Point_Probe" H 7453 1111 50  0000 L CNN
+F 2 "" H 7500 1100 50  0001 C CNN
+F 3 "~" H 7500 1100 50  0001 C CNN
+	1    7300 1100
+	1    0    0    -1
+$EndComp
+$Comp
+L haathi_mayank:Test_Point_Probe TP?
+U 1 1 5A7E0B7A
+P 6300 2300
+F 0 "TP?" H 6453 2402 50  0000 L CNN
+F 1 "Test_Point_Probe" H 6453 2311 50  0000 L CNN
+F 2 "" H 6500 2300 50  0001 C CNN
+F 3 "~" H 6500 2300 50  0001 C CNN
+	1    6300 2300
+	1    0    0    -1
+$EndComp
+$Comp
+L haathi_mayank:Test_Point_Probe TP?
+U 1 1 5A7E0EB4
+P 6450 1850
+F 0 "TP?" H 6603 1952 50  0000 L CNN
+F 1 "Test_Point_Probe" H 6603 1861 50  0000 L CNN
+F 2 "" H 6650 1850 50  0001 C CNN
+F 3 "~" H 6650 1850 50  0001 C CNN
+	1    6450 1850
+	1    0    0    -1
+$EndComp
+Wire Wire Line
+	6450 1850 6350 1850
+Wire Wire Line
+	6350 1850 6350 1950
+Connection ~ 6350 1950
+Wire Wire Line
+	6350 1950 6450 1950
+Wire Wire Line
+	6300 2300 6100 2300
+Connection ~ 6100 2300
+Wire Wire Line
+	6100 2300 6100 2350
+Wire Wire Line
+	7300 1100 7300 1250
+Connection ~ 7300 1250
+Wire Wire Line
+	7300 1250 7500 1250
 $EndSCHEMATC

Commit message: Mayank, Added current measurement jumpers on power sheet
Parts:
- added J? (x3): Conn_01x02, symbol haathi_mayank:Conn_01x02
Connections:
- net labels added: VCC_3V3
- wire segments 187 -> 191

Commit message: Mayank, Power sheet: Added 0Ohm resistors in parallel to current measurement jumpers
Parts:
- added R? (x3): 0, symbol haathi_mayank:R
Connections:
- wire segments 191 -> 209
Changed lines of the file:
@@
 	900  1100 1200 1100
-Wire Wire Line
-	5000 1500 5300 1500
 Wire Wire Line
 	5400 1500 5500 1500
@@
 Wire Wire Line
 	10000 1100 10050 1100
+$Comp
+L haathi_mayank:R R?
+U 1 1 5A864549
+P 5400 1900
+F 0 "R?" H 5470 1946 50  0000 L CNN
+F 1 "0" H 5470 1855 50  0000 L CNN
+F 2 "" V 5330 1900 30  0000 C CNN
+F 3 "" H 5400 1900 30  0000 C CNN
+	1    5400 1900
+	0    1    1    0
+$EndComp
+Wire Wire Line
+	5400 1500 5400 1800
+Wire Wire Line
+	5400 1800 5550 1800
+Wire Wire Line
+	5550 1800 5550 1900
+Connection ~ 5400 1500
+Wire Wire Line
+	5300 1500 5300 1800
+Wire Wire Line
+	5300 1800 5250 1800
+Wire Wire Line
+	5250 1800 5250 1900
+Wire Wire Line
+	5000 1500 5300 1500
+Connection ~ 5300 1500
+$Comp
+L haathi_mayank:R R?
+U 1 1 5A8938A2
+P 9700 1550
+F 0 "R?" H 9770 1596 50  0000 L CNN
+F 1 "0" H 9770 1505 50  0000 L CNN
+F 2 "" V 9630 1550 30  0000 C CNN
+F 3 "" H 9700 1550 30  0000 C CNN
+	1    9700 1550
+	0    1    1    0
+$EndComp
+Wire Wire Line
+	9650 1100 9650 1450
+Wire Wire Line
+	9650 1450 9550 1450
+Wire Wire Line
+	9550 1450 9550 1550
+Connection ~ 9650 1100
+Wire Wire Line
+	9750 1100 9750 1450
+Wire Wire Line
+	9750 1450 9850 1450
+Wire Wire Line
+	9850 1450 9850 1550
+Connection ~ 9750 1100
+$Comp
+L haathi_mayank:R R?
+U 1 1 5A8ABC59
+P 1250 1650
+F 0 "R?" H 1320 1696 50  0000 L CNN
+F 1 "0" H 1320 1605 50  0000 L CNN
+F 2 "" V 1180 1650 30  0000 C CNN
+F 3 "" H 1250 1650 30  0000 C CNN
+	1    1250 1650
+	0    1    1    0
+$EndComp
+Wire Wire Line
+	1300 1100 1300 1550
+Wire Wire Line
+	1300 1550 1400 1550
+Wire Wire Line
+	1400 1550 1400 1650
+Connection ~ 1300 1100
+Wire Wire Line
+	1200 1100 1200 1550
+Wire Wire Line
+	1200 1550 1100 1550
+Wire Wire Line
+	1100 1550 1100 1650
+Connection ~ 1200 1100
 $EndSCHEMATC

Commit message: Mayank, Power: added TVS Diode to V_INPUT
Parts:
- added D?: D_TVS, symbol haathi_mayank:D_TVS
Connections:
- wire segments 209 -> 212
Changed lines of the file:
@@
 Text Label 7800 5250 0    50   ~ 0
 VIN
-Text Label 7150 5250 2    50   ~ 0
+Text Label 6800 5250 2    50   ~ 0
 V_INPUT
 $Comp
@@
 Wire Wire Line
 	7450 5550 7450 5600
-Wire Wire Line
-	7150 5250 7250 5250
 Wire Wire Line
 	7650 5250 7700 5250
@@
 	1100 1550 1100 1650
 Connection ~ 1200 1100
+$Comp
+L haathi_mayank:D_TVS D?
+U 1 1 5A8D6681
+P 7000 5400
+F 0 "D?" V 6954 5479 50  0000 L CNN
+F 1 "D_TVS" V 7045 5479 50  0000 L CNN
+F 2 "" H 7000 5400 50  0001 C CNN
+F 3 "~" H 7000 5400 50  0001 C CNN
+	1    7000 5400
+	0    1    1    0
+$EndComp
+Wire Wire Line
+	6800 5250 7000 5250
+Connection ~ 7000 5250
+Wire Wire Line
+	7000 5250 7250 5250
+Wire Wire Line
+	7000 5550 7000 5600
+Wire Wire Line
+	7000 5600 7450 5600
 $EndSCHEMATC

Commit message: Renamed USER_BUTTON to WAKEUP_BUTTON
Connections:
- net labels added: WAKEUP_BUTTON
- net labels removed: USER_BUTTON
Other:
- note added: "Wakeup Button"
- note removed: "User Button"
Changed lines of the file:
@@
 POR_BUTTON
 Text HLabel 10400 5300 2    50   Input ~ 0
-USER_BUTTON
+WAKEUP_BUTTON
 Text Notes 9200 4350 0    50   ~ 0
 Buttons
@@
 System Reset Button
 Text Notes 10400 5450 0    50   ~ 0
-User Button
+Wakeup Button
 Wire Wire Line
 	2250 700  2250 1100
