File: kicad/haathi_power.sch (KiCad schematic (older format))
At the start: 70 parts

Commit message: Mayank, Power sheet:Flipped Buck ckt, changed conn vals, 0Ohm to 0E on power sheet
Parts:
- J?: value Conn_01x02 -> Conn12_BAT
- J?: value Conn_01x02 -> Conn12_I_3V3
- J?: value Conn_01x02 -> Conn12_I_VIN
- J?: value Conn_01x02 -> Conn12_I_VDD_SNVS_IN
- R? (x10): value 0 -> 0E
- TP?: value Test_Point_Probe -> TP_3V3
- TP?: value Test_Point_Probe -> TP_GND
- TP?: value Test_Point_Probe -> TP_VIN
Connections:
- net labels added: +3V3
- net labels removed: VCC
- wire segments 212 -> 218

Commit message: power: Edited V_USB label to 5V_USB_OTG
Connections:
- net labels added: 5V_USB_OTG
- net labels removed: V_USB
Changed lines of the file:
@@
 EESchema Schematic File Version 4
-LIBS:haathi-cache
+LIBS:haathi_power-cache
 EELAYER 26 0
 EELAYER END
 $Descr A4 11693 8268
 encoding utf-8
-Sheet 1 11
+Sheet 1 1
 Title "haathi_cam"
 Date "2018-03-11"
@@
 Wire Wire Line
 	4000 7200 4200 7200
-Text HLabel 7750 4500 2    50   Input ~ 0
-V_USB
+Text HLabel 8050 4500 2    50   Input ~ 0
+5V_USB_OTG
 Text Label 950  1500 2    50   ~ 0
 VIN
@@
 $EndComp
 Wire Wire Line
-	7450 4500 7750 4500
-Wire Wire Line
 	7450 4600 7750 4600
 Wire Wire Line
@@
 Connection ~ 9575 5300
 Text Label 7500 4500 0    50   ~ 0
-V_USB
+5V_USB_OTG
 Text Label 4900 5450 0    50   ~ 0
 VDD_HIGH_IN
@@
 Wire Wire Line
 	2775 3425 3425 3425
+Wire Wire Line
+	7450 4500 8050 4500
 $EndSCHEMATC

Commit message: power: added note for reverse pol Coin Cell to go on silk
Other:
- note added: "Add silk note warning\nto not put coin cell other\nway around"
Changed lines of the file:
@@
 Wire Wire Line
 	7450 4500 8050 4500
+Text Notes 10050 1450 0    50   ~ 0
+Add silk note warning\nto not put coin cell other\nway around
 $EndSCHEMATC
