File: kicad/haathi_power.sch (KiCad schematic (older format))
At the start: 70 parts

Commit message: Removes the APX811 from the power sheet, as its shifted to CPU sheet
Parts:
- removed U?: APX811, symbol haathi_mayank:APX811
Connections:
- net labels removed: MCU_RESET_N
- wire segments 218 -> 213
Other:
- note removed: "Power Monitoring and Reset"
Changed lines of the file:
@@
 $Descr A4 11693 8268
 encoding utf-8
-Sheet 1 9
+Sheet 1 1
 Title "haathi_cam"
 Date "2018-03-11"
@@
 Text Notes 7550 4750 0    50   ~ 0
 OFF
-$Comp
-L haathi_mayank:APX811 U?
-U 1 1 5A8B233D
-P 2425 3325
-F 0 "U?" H 2400 3640 50  0000 C CNN
-F 1 "APX811" H 2400 3549 50  0000 C CNN
-F 2 "" H 2275 3225 50  0001 C CNN
-F 3 "" H 2275 3225 50  0001 C CNN
-	1    2425 3325
-	1    0    0    -1
-$EndComp
-Text HLabel 3425 3425 2    50   Input ~ 0
-POR_BUTTON
-Text HLabel 1275 3425 0    50   Input ~ 0
-MCU_RESET_N
-Wire Wire Line
-	2775 3275 2925 3275
-$Comp
-L power:GND #PWR?
-U 1 1 5A92FBAD
-P 1925 3525
-F 0 "#PWR?" H 1925 3275 50  0001 C CNN
-F 1 "GND" H 1930 3352 50  0000 C CNN
-F 2 "" H 1925 3525 50  0001 C CNN
-F 3 "" H 1925 3525 50  0001 C CNN
-	1    1925 3525
-	1    0    0    -1
-$EndComp
-Wire Wire Line
-	2025 3275 1925 3275
-Wire Wire Line
-	1925 3275 1925 3525
-Text Notes 2675 2925 2    50   ~ 0
-Power Monitoring and Reset
 Text Label 6950 4600 2    50   ~ 0
 V_INPUT
@@
 F 3 "" H 6250 1250 50  0001 C CNN
 	1    6250 1250
-	1    0    0    -1
-$EndComp
-$Comp
-L power:+3V3 #PWR?
-U 1 1 5A9D23A7
-P 2925 3275
-F 0 "#PWR?" H 2925 3125 50  0001 C CNN
-F 1 "+3V3" H 2940 3448 50  0000 C CNN
-F 2 "" H 2925 3275 50  0001 C CNN
-F 3 "" H 2925 3275 50  0001 C CNN
-	1    2925 3275
 	1    0    0    -1
 $EndComp
@@
 DCDC_IN
 Wire Wire Line
-	1275 3425 2025 3425
-Text Label 1325 3425 0    50   ~ 0
-MCU_RESET_N
-Text Label 2825 3425 0    50   ~ 0
-POR_BUTTON
-Wire Wire Line
-	2775 3425 3425 3425
-Wire Wire Line
 	7450 4500 8050 4500

Commit message: Imported all hierarchical labels on top sheet
Connections:
- wire segments 213 -> 207
Changed lines of the file:
@@
 EESchema Schematic File Version 4
+LIBS:haathi_schematic-cache
 EELAYER 26 0
 EELAYER END
 $Descr A4 11693 8268
 encoding utf-8
-Sheet 1 1
+Sheet 2 9
 Title "haathi_cam"
 Date "2018-03-11"
@@
 Wire Wire Line
 	2000 1850 2000 2150
-Wire Wire Line
-	2000 2150 2100 2150
 Connection ~ 2400 2150
 Wire Wire Line
@@
 Connection ~ 6800 1250
 Wire Wire Line
-	6800 1250 6650 1250
-Wire Wire Line
 	6950 1900 6800 1900
 Wire Wire Line
@@
 	-1   0    0    1
 $EndComp
-Connection ~ 6650 1250
 Text HLabel 7700 1250 2    50   Input ~ 0
 DCDC_IN
@@
 	3450 7200 3800 7200
 Connection ~ 3800 7200
-Wire Wire Line
-	3800 7200 4000 7200
 Connection ~ 4200 7200
 Wire Wire Line
@@
 	1    0    0    -1
 $EndComp
-Connection ~ 4000 7200
-Wire Wire Line
-	4000 7200 4200 7200
 Text HLabel 8050 4500 2    50   Input ~ 0
 5V_USB_OTG
@@
 	1    0    0    1
 $EndComp
-Connection ~ 2100 2150
-Wire Wire Line
-	2100 2150 2400 2150
 Wire Wire Line
 	1550 1800 1550 2150
@@
 Wire Wire Line
 	10250 2350 10250 2500
-Connection ~ 10250 2500
 $Comp
 L power:GND #PWR?
@@
 	6450 1100 6450 1250
 Connection ~ 6450 1250
-Wire Wire Line
-	6450 1250 6650 1250
 $Comp
 L haathi_mayank:Conn_01x02 J?
@@
 VCC_3V3
 Wire Wire Line
-	5800 1100 5650 1100
-Connection ~ 5650 1100
-Wire Wire Line
-	5650 1100 5350 1100
-Wire Wire Line
-	1150 1500 1050 1500
-Connection ~ 1050 1500
-Wire Wire Line
-	1050 1500 950  1500
-Wire Wire Line
 	2000 1500 1550 1500
 $Comp
@@
 Text Label 9825 1100 0    50   ~ 0
 VDD_SNVS_IN
-Connection ~ 10400 1100
-Wire Wire Line
-	10400 1100 10450 1100
-Wire Wire Line
-	9750 1100 10400 1100
 $Comp
 L power:+3V3 #PWR?
@@
 Text Notes 10050 1450 0    50   ~ 0
 Add silk note warning\nto not put coin cell other\nway around
+Wire Wire Line
+	2000 2150 2400 2150
+Wire Wire Line
+	6450 1250 6800 1250
+Wire Wire Line
+	3800 7200 4200 7200
+Wire Wire Line
+	5350 1100 5800 1100
+Wire Wire Line
+	950  1500 1150 1500
+Wire Wire Line
+	9750 1100 10450 1100
 $EndSCHEMATC

Commit message: NVCC_SD0 and NVCC_SD1 are not from 3V3. Flag and GND connected properly.
Parts:
- removed R? (x2): 0E, symbol haathi_mayank:R
Changed lines of the file:
@@
 EESchema Schematic File Version 4
-LIBS:haathi_schematic-cache
+LIBS:haathi_power-cache
 EELAYER 26 0
 EELAYER END
 $Descr A4 11693 8268
 encoding utf-8
-Sheet 2 9
+Sheet 1 1
 Title "haathi_cam"
 Date "2018-03-11"
@@
 $Comp
 L haathi_mayank:R R?
-U 1 1 5A6ED45D
+U 1 1 5A6ED4CD
 P 7100 1600
 F 0 "R?" H 7170 1646 50  0000 L CNN
@@
 $Comp
 L haathi_mayank:R R?
-U 1 1 5A6ED497
+U 1 1 5A6ED6D7
 P 7100 1900
 F 0 "R?" H 7170 1946 50  0000 L CNN
@@
 $Comp
 L haathi_mayank:R R?
-U 1 1 5A6ED4CD
+U 1 1 5A6ED735
 P 7100 2200
 F 0 "R?" H 7170 2246 50  0000 L CNN
@@
 $Comp
 L haathi_mayank:R R?
-U 1 1 5A6ED6D7
-P 7100 2500
-F 0 "R?" H 7170 2546 50  0000 L CNN
-F 1 "0E" H 7170 2455 50  0000 L CNN
-F 2 "" V 7030 2500 30  0000 C CNN
-F 3 "" H 7100 2500 30  0000 C CNN
-	1    7100 2500
+U 1 1 5A6ED769
+P 7100 2450
+F 0 "R?" H 7170 2496 50  0000 L CNN
+F 1 "0E" H 7170 2405 50  0000 L CNN
+F 2 "" V 7030 2450 30  0000 C CNN
+F 3 "" H 7100 2450 30  0000 C CNN
+	1    7100 2450
 	0    1    1    0
 $EndComp
-$Comp
-L haathi_mayank:R R?
-U 1 1 5A6ED735
-P 7100 2800
-F 0 "R?" H 7170 2846 50  0000 L CNN
-F 1 "0E" H 7170 2755 50  0000 L CNN
-F 2 "" V 7030 2800 30  0000 C CNN
-F 3 "" H 7100 2800 30  0000 C CNN
-	1    7100 2800
-	0    1    1    0
-$EndComp
-$Comp
-L haathi_mayank:R R?
-U 1 1 5A6ED769
-P 7100 3050
-F 0 "R?" H 7170 3096 50  0000 L CNN
-F 1 "0E" H 7170 3005 50  0000 L CNN
-F 2 "" V 7030 3050 30  0000 C CNN
-F 3 "" H 7100 3050 30  0000 C CNN
-	1    7100 3050
-	0    1    1    0
-$EndComp
 Wire Wire Line
 	6950 1250 6800 1250
+Connection ~ 6800 1250
 Wire Wire Line
 	6950 1600 6800 1600
-Wire Wire Line
-	6800 1600 6800 1250
-Connection ~ 6800 1250
 Wire Wire Line
 	6950 1900 6800 1900
@@
 Connection ~ 6800 1900
 Wire Wire Line
-	6950 2500 6800 2500
-Wire Wire Line
-	6800 2500 6800 2200
+	6950 2450 6800 2450
+Wire Wire Line
+	6800 2450 6800 2200
 Connection ~ 6800 2200
-Wire Wire Line
-	6950 2800 6800 2800
-Wire Wire Line
-	6800 2800 6800 2500
-Connection ~ 6800 2500
-Wire Wire Line
-	6950 3050 6800 3050
-Wire Wire Line
-	6800 3050 6800 2800
-Connection ~ 6800 2800
 $Comp
 L power:PWR_FLAG #FLG?
@@
 DCDC_IN
 Text HLabel 7700 1600 2    50   Input ~ 0
-NVCC_SD0
+NVCC_EMC
 Text HLabel 7700 1900 2    50   Input ~ 0
-NVCC_SD1
-Text HLabel 7700 2200 2    50   Input ~ 0
-NVCC_EMC
-Text HLabel 7700 2500 2    50   Input ~ 0
 NVCC_GPIO
-Text HLabel 7875 2800 2    50   Input ~ 0
+Text HLabel 7875 2200 2    50   Input ~ 0
 VDDA_ADC_3P3
-Text HLabel 7875 3050 2    50   Input ~ 0
+Text HLabel 7875 2450 2    50   Input ~ 0
 VDD_HIGH_IN
 Text HLabel 1300 4600 0    50   Input ~ 0
@@
 Wire Wire Line
 	7250 1900 7700 1900
-Wire Wire Line
-	7250 2200 7700 2200
-Wire Wire Line
-	7250 2500 7700 2500
 Text Label 7325 1250 0    50   ~ 0
 DCDC_IN
-Text Label 7300 1600 0    50   ~ 0
-NVCC_SD0
-Text Label 7300 1900 0    50   ~ 0
-NVCC_SD1
-Text Label 7275 2200 0    50   ~ 0
+Text Label 7275 1600 0    50   ~ 0
 NVCC_EMC
-Text Label 7275 2500 0    50   ~ 0
+Text Label 7275 1900 0    50   ~ 0
 NVCC_GPIO
-Text Label 7250 2800 0    50   ~ 0
+Text Label 7250 2200 0    50   ~ 0
 VDDA_ADC_3P3
-Text Label 7275 3050 0    50   ~ 0
+Text Label 7275 2450 0    50   ~ 0
 VDD_HIGH_IN
 Wire Wire Line
-	7250 2800 7875 2800
-Wire Wire Line
-	7250 3050 7875 3050
+	7250 2200 7875 2200
+Wire Wire Line
+	7250 2450 7875 2450
 Wire Wire Line
 	4500 4600 5000 4600
@@
 Add silk note warning\nto not put coin cell other\nway around
 Wire Wire Line
-	2000 2150 2400 2150
-Wire Wire Line
-	6450 1250 6800 1250
-Wire Wire Line
-	3800 7200 4200 7200
-Wire Wire Line
-	5350 1100 5800 1100
-Wire Wire Line
-	950  1500 1150 1500
-Wire Wire Line
-	9750 1100 10450 1100
+	2000 2150 2100 2150
+Wire Wire Line
+	6450 1250 6650 1250
+Wire Wire Line
+	3800 7200 4000 7200
+Wire Wire Line
+	5350 1100 5650 1100
+Wire Wire Line
+	950  1500 1050 1500
+Wire Wire Line
+	9750 1100 10400 1100
+Connection ~ 10400 1100
+Wire Wire Line
+	10400 1100 10450 1100
+Connection ~ 1050 1500
+Wire Wire Line
+	1050 1500 1150 1500
+Connection ~ 2100 2150
+Wire Wire Line
+	2100 2150 2400 2150
+Connection ~ 5650 1100
+Wire Wire Line
+	5650 1100 5800 1100
+Connection ~ 6650 1250
+Wire Wire Line
+	6650 1250 6800 1250
+Connection ~ 4000 7200
+Wire Wire Line
+	4000 7200 4200 7200
+Wire Wire Line
+	6800 1250 6800 1600
 $EndSCHEMATC

Commit message: Annotated schematic
Parts:
- gave numbers to parts that had none: 67

Commit message: ERC pass 1: Check and resolve the errors
Signed-off-by: Kumar Abhishek <abhishek@theembeddedkitchen.net>
Connections:
- wire segments 207 -> 204
Changed lines of the file:
@@
 EESchema Schematic File Version 4
-LIBS:haathi_schematic-cache
+LIBS:haathi-cache
 EELAYER 26 0
 EELAYER END
 $Descr A4 11693 8268
 encoding utf-8
-Sheet 1 9
+Sheet 4 11
 Title "haathi_cam"
 Date "2018-03-11"
@@
 F 3 "" H 1050 1500 50  0001 C CNN
 	1    1050 1500
-	1    0    0    1
-$EndComp
-$Comp
-L power:PWR_FLAG #FLG03
-U 1 1 5A6E843F
-P 5650 1100
-F 0 "#FLG03" H 5650 1175 50  0001 C CNN
-F 1 "PWR_FLAG" H 5650 1274 50  0000 C CNN
-F 2 "" H 5650 1100 50  0001 C CNN
-F 3 "" H 5650 1100 50  0001 C CNN
-	1    5650 1100
 	1    0    0    1
 $EndComp
@@
 	6800 2450 6800 2200
 Connection ~ 6800 2200
-$Comp
-L power:PWR_FLAG #FLG04
-U 1 1 5A6FEDB5
-P 6650 1250
-F 0 "#FLG04" H 6650 1325 50  0001 C CNN
-F 1 "PWR_FLAG" H 6650 1423 50  0000 C CNN
-F 2 "" H 6650 1250 50  0001 C CNN
-F 3 "" H 6650 1250 50  0001 C CNN
-	1    6650 1250
-	-1   0    0    1
-$EndComp
 Text HLabel 7700 1250 2    50   Input ~ 0
 DCDC_IN
@@
 $EndComp
 Connection ~ 1550 1500
-$Comp
-L power:PWR_FLAG #FLG02
-U 1 1 5A75C5FD
-P 2100 2150
-F 0 "#FLG02" H 2100 2225 50  0001 C CNN
-F 1 "PWR_FLAG" H 2100 2324 50  0000 C CNN
-F 2 "" H 2100 2150 50  0001 C CNN
-F 3 "" H 2100 2150 50  0001 C CNN
-	1    2100 2150
-	1    0    0    1
-$EndComp
 Wire Wire Line
 	1550 1800 1550 2150
@@
 Add silk note warning\nto not put coin cell other\nway around
 Wire Wire Line
-	2000 2150 2100 2150
-Wire Wire Line
-	6450 1250 6650 1250
-Wire Wire Line
 	3800 7200 4000 7200
-Wire Wire Line
-	5350 1100 5650 1100
 Wire Wire Line
 	950  1500 1050 1500
@@
 Wire Wire Line
 	1050 1500 1150 1500
-Connection ~ 2100 2150
-Wire Wire Line
-	2100 2150 2400 2150
-Connection ~ 5650 1100
-Wire Wire Line
-	5650 1100 5800 1100
-Connection ~ 6650 1250
-Wire Wire Line
-	6650 1250 6800 1250
 Connection ~ 4000 7200
 Wire Wire Line
@@
 Wire Wire Line
 	6800 1250 6800 1600
+Wire Wire Line
+	5350 1100 5800 1100
+Wire Wire Line
+	6450 1250 6800 1250
+Wire Wire Line
+	2000 2150 2400 2150
+$Comp
+L power:PWR_FLAG #FLG0104
+U 1 1 5B2F54AB
+P 4200 6900
+F 0 "#FLG0104" H 4200 6975 50  0001 C CNN
+F 1 "PWR_FLAG" H 4200 7074 50  0000 C CNN
+F 2 "" H 4200 6900 50  0001 C CNN
+F 3 "~" H 4200 6900 50  0001 C CNN
+	1    4200 6900
+	1    0    0    -1
+$EndComp
+$Comp
+L power:PWR_FLAG #FLG0105
+U 1 1 5B310DC9
+P 3650 6150
+F 0 "#FLG0105" H 3650 6225 50  0001 C CNN
+F 1 "PWR_FLAG" H 3900 6225 50  0000 C CNN
+F 2 "" H 3650 6150 50  0001 C CNN
+F 3 "~" H 3650 6150 50  0001 C CNN
+	1    3650 6150
+	1    0    0    -1
+$EndComp
+$Comp
+L power:PWR_FLAG #FLG0106
+U 1 1 5B311192
+P 3350 5400
+F 0 "#FLG0106" H 3350 5475 50  0001 C CNN
+F 1 "PWR_FLAG" H 3600 5475 50  0000 C CNN
+F 2 "" H 3350 5400 50  0001 C CNN
+F 3 "~" H 3350 5400 50  0001 C CNN
+	1    3350 5400
+	1    0    0    -1
+$EndComp
+$Comp
+L power:PWR_FLAG #FLG0107
+U 1 1 5B31C81B
+P 1600 5400
+F 0 "#FLG0107" H 1600 5475 50  0001 C CNN
+F 1 "PWR_FLAG" H 1600 5550 50  0000 C CNN
+F 2 "" H 1600 5400 50  0001 C CNN
+F 3 "~" H 1600 5400 50  0001 C CNN
+	1    1600 5400
+	1    0    0    -1
+$EndComp
+$Comp
+L power:PWR_FLAG #FLG0108
+U 1 1 5B31C97F
+P 1550 6150
+F 0 "#FLG0108" H 1550 6225 50  0001 C CNN
+F 1 "PWR_FLAG" H 1550 6300 50  0000 C CNN
+F 2 "" H 1550 6150 50  0001 C CNN
+F 3 "~" H 1550 6150 50  0001 C CNN
+	1    1550 6150
+	1    0    0    -1
+$EndComp
+$Comp
+L power:PWR_FLAG #FLG0109
+U 1 1 5B31CA53
+P 1600 6850
+F 0 "#FLG0109" H 1600 6925 50  0001 C CNN
+F 1 "PWR_FLAG" H 1600 7000 50  0000 C CNN
+F 2 "" H 1600 6850 50  0001 C CNN
+F 3 "~" H 1600 6850 50  0001 C CNN
+	1    1600 6850
+	1    0    0    -1
+$EndComp
+$Comp
+L power:PWR_FLAG #FLG0110
+U 1 1 5B31F65C
+P 5000 4600
+F 0 "#FLG0110" H 5000 4675 50  0001 C CNN
+F 1 "PWR_FLAG" H 5000 4750 50  0000 C CNN
+F 2 "" H 5000 4600 50  0001 C CNN
+F 3 "~" H 5000 4600 50  0001 C CNN
+	1    5000 4600
+	1    0    0    -1
+$EndComp
+$Comp
+L power:PWR_FLAG #FLG0111
+U 1 1 5B31F905
+P 5000 5450
+F 0 "#FLG0111" H 5000 5525 50  0001 C CNN
+F 1 "PWR_FLAG" H 5000 5600 50  0000 C CNN
+F 2 "" H 5000 5450 50  0001 C CNN
+F 3 "~" H 5000 5450 50  0001 C CNN
+	1    5000 5450
+	1    0    0    -1
+$EndComp
+$Comp
+L power:PWR_FLAG #FLG0112
+U 1 1 5B31F996
+P 5000 6100
+F 0 "#FLG0112" H 5000 6175 50  0001 C CNN
+F 1 "PWR_FLAG" H 5000 6250 50  0000 C CNN
+F 2 "" H 5000 6100 50  0001 C CNN
+F 3 "~" H 5000 6100 50  0001 C CNN
+	1    5000 6100
+	1    0    0    -1
+$EndComp
 $EndSCHEMATC

Commit message: Changes OFF to mid pin in SP3T switch
Changes dual schottky diode to a single package.
Parts:
- removed D3, D4: D_Schottky, symbol haathi_mayank:D_Schottky
- added D?: PMEG3020CPA, symbol Device:D_Schottky_x2_KCom_AAK
- D2: value D_TVS -> SMBJ16D-M3/H
Changed lines of the file:
@@
 $Descr A4 11693 8268
 encoding utf-8
-Sheet 4 9
+Sheet 1 9
 Title "haathi_cam"
 Date "2018-03-11"
@@
 Text Label 950  1500 2    50   ~ 0
 VIN
-Text Label 7750 4600 0    50   ~ 0
-V_BATT
-Text Label 10850 2050 0    50   ~ 0
+Text Label 7750 4700 0    50   ~ 0
 V_BATT
 Text Notes 6950 4250 0    50   ~ 0
@@
 Text Notes 6950 950  0    50   ~ 0
 Supply Nets
-Text Notes 9500 1900 0    50   ~ 0
+Text Notes 9125 1925 0    50   ~ 0
 Battery
 $Comp
@@
 L haathi_mayank:Barrel_Jack J5
 U 1 1 5A7907B4
-P 9600 3100
-F 0 "J5" H 9678 3425 50  0000 C CNN
-F 1 "Barrel_Jack" H 9678 3334 50  0000 C CNN
-F 2 "" H 9650 3060 50  0001 C CNN
-F 3 "~" H 9650 3060 50  0001 C CNN
-	1    9600 3100
+P 9225 3125
+F 0 "J5" H 9303 3450 50  0000 C CNN
+F 1 "Barrel_Jack" H 9303 3359 50  0000 C CNN
+F 2 "" H 9275 3085 50  0001 C CNN
+F 3 "~" H 9275 3085 50  0001 C CNN
+	1    9225 3125
 	1    0    0    -1
 $EndComp
@@
 L haathi_mayank:Conn_01x02 J4
 U 1 1 5A790B17
-P 9550 2150
-F 0 "J4" H 9630 2142 50  0000 L CNN
-F 1 "Conn12_BAT" H 9630 2051 50  0000 L CNN
-F 2 "" H 9550 2150 50  0001 C CNN
-F 3 "~" H 9550 2150 50  0001 C CNN
-	1    9550 2150
+P 9175 2175
+F 0 "J4" H 9255 2167 50  0000 L CNN
+F 1 "Conn12_BAT" H 9255 2076 50  0000 L CNN
+F 2 "" H 9175 2175 50  0001 C CNN
+F 3 "~" H 9175 2175 50  0001 C CNN
+	1    9175 2175
 	-1   0    0    1
 $EndComp
@@
 L power:GND #PWR031
 U 1 1 5A7C72A6
-P 10250 2500
-F 0 "#PWR031" H 10250 2250 50  0001 C CNN
-F 1 "GND" H 10255 2327 50  0000 C CNN
-F 2 "" H 10250 2500 50  0001 C CNN
-F 3 "" H 10250 2500 50  0001 C CNN
-	1    10250 2500
+P 9575 2550
+F 0 "#PWR031" H 9575 2300 50  0001 C CNN
+F 1 "GND" H 9580 2377 50  0000 C CNN
+F 2 "" H 9575 2550 50  0001 C CNN
+F 3 "" H 9575 2550 50  0001 C CNN
+	1    9575 2550
 	1    0    0    -1
 $EndComp
@@
 L haathi_mayank:C_NP C45
 U 1 1 5A7C7321
-P 10250 2200
-F 0 "C45" H 10353 2238 40  0000 L CNN
-F 1 "0.1uF" H 10353 2162 40  0000 L CNN
-F 2 "" H 10250 2200 60  0000 C CNN
-F 3 "" H 10250 2200 60  0000 C CNN
-	1    10250 2200
-	1    0    0    -1
-$EndComp
-Wire Wire Line
-	9750 2150 9950 2150
-Wire Wire Line
-	9750 2050 10250 2050
-Connection ~ 10250 2050
-Wire Wire Line
-	10250 2050 10450 2050
-Wire Wire Line
-	9950 2500 10250 2500
-Wire Wire Line
-	9950 2150 9950 2500
-Wire Wire Line
-	10250 2350 10250 2500
+P 10775 2825
+F 0 "C45" H 10878 2863 40  0000 L CNN
+F 1 "0.1uF" H 10878 2787 40  0000 L CNN
+F 2 "" H 10775 2825 60  0000 C CNN
+F 3 "" H 10775 2825 60  0000 C CNN
+	1    10775 2825
+	1    0    0    -1
+$EndComp
+Wire Wire Line
+	9375 2175 9575 2175
 $Comp
 L power:GND #PWR030
 U 1 1 5A7FB66D
-P 10150 3350
-F 0 "#PWR030" H 10150 3100 50  0001 C CNN
-F 1 "GND" H 10155 3177 50  0000 C CNN
-F 2 "" H 10150 3350 50  0001 C CNN
-F 3 "" H 10150 3350 50  0001 C CNN
-	1    10150 3350
+P 9525 3425
+F 0 "#PWR030" H 9525 3175 50  0001 C CNN
+F 1 "GND" H 9530 3252 50  0000 C CNN
+F 2 "" H 9525 3425 50  0001 C CNN
+F 3 "" H 9525 3425 50  0001 C CNN
+	1    9525 3425
 	1    0    0    -1
 $EndComp
@@
 L haathi_mayank:C_NP C44
 U 1 1 5A7FB89E
-P 10150 3100
-F 0 "C44" H 10253 3138 40  0000 L CNN
-F 1 "22uF" H 10253 3062 40  0000 L CNN
-F 2 "" H 10150 3100 60  0000 C CNN
-F 3 "" H 10150 3100 60  0000 C CNN
-	1    10150 3100
-	1    0    0    -1
-$EndComp
-Wire Wire Line
-	9900 3100 9900 3200
-Wire Wire Line
-	9900 3200 9900 3300
-Wire Wire Line
-	9900 3300 10150 3300
-Connection ~ 9900 3200
-Wire Wire Line
-	9900 3000 9900 2950
-Wire Wire Line
-	9900 2950 10150 2950
-Wire Wire Line
-	10150 3250 10150 3300
-Wire Wire Line
-	10150 3300 10150 3350
-Connection ~ 10150 3300
-Text Label 10800 2950 0    50   ~ 0
+P 10375 2825
+F 0 "C44" H 10478 2863 40  0000 L CNN
+F 1 "22uF" H 10478 2787 40  0000 L CNN
+F 2 "" H 10375 2825 60  0000 C CNN
+F 3 "" H 10375 2825 60  0000 C CNN
+	1    10375 2825
+	1    0    0    -1
+$EndComp
+Wire Wire Line
+	9525 3125 9525 3225
+Connection ~ 9525 3225
+Wire Wire Line
+	9525 3025 9525 2975
+Text Label 10850 2550 0    50   ~ 0
 V_BATT
-$Comp
-L haathi_mayank:D_Schottky D4
-U 1 1 5A8309CA
-P 10600 2050
-F 0 "D4" H 10600 1834 50  0000 C CNN
-F 1 "D_Schottky" H 10600 1925 50  0000 C CNN
-F 2 "" H 10600 2050 50  0001 C CNN
-F 3 "" H 10600 2050 50  0001 C CNN
-	1    10600 2050
-	-1   0    0    1
-$EndComp
-$Comp
-L haathi_mayank:D_Schottky D3
-U 1 1 5A83100D
-P 10500 2950
-F 0 "D3" H 10500 2734 50  0000 C CNN
-F 1 "D_Schottky" H 10500 2825 50  0000 C CNN
-F 2 "" H 10500 2950 50  0001 C CNN
-F 3 "" H 10500 2950 50  0001 C CNN
-	1    10500 2950
-	-1   0    0    1
-$EndComp
-Wire Wire Line
-	10150 2950 10350 2950
-Connection ~ 10150 2950
-Wire Wire Line
-	10650 2950 10800 2950
-Wire Wire Line
-	10750 2050 10850 2050
+Wire Wire Line
+	10125 2550 10375 2550
 $Comp
 L haathi_mayank:SW_SP3T SW1
@@
 $EndComp
 Wire Wire Line
-	7450 4600 7750 4600
+	7450 4700 7750 4700
 Wire Wire Line
 	7050 4600 6950 4600
-NoConn ~ 7450 4700
-Text Notes 7550 4750 0    50   ~ 0
+NoConn ~ 7450 4600
+Text Notes 7500 4625 0    50   ~ 0
 OFF
 Text Label 6950 4600 2    50   ~ 0
@@
 P 7000 5400
 F 0 "D2" V 6954 5479 50  0000 L CNN
-F 1 "D_TVS" V 7045 5479 50  0000 L CNN
+F 1 "SMBJ16D-M3/H" V 7050 4725 50  0000 L CNN
 F 2 "" H 7000 5400 50  0001 C CNN
 F 3 "~" H 7000 5400 50  0001 C CNN
@@
 	1    0    0    -1
 $EndComp
+$Comp
+L Device:D_Schottky_x2_KCom_AAK D?
+U 1 1 5B013789
+P 9925 2550
+F 0 "D?" V 9971 2628 50  0000 L CNN
+F 1 "PMEG3020CPA" V 10050 1950 50  0000 L CNN
+F 2 "" H 9925 2550 50  0001 C CNN
+F 3 "~" H 9925 2550 50  0001 C CNN
+	1    9925 2550
+	0    -1   -1   0
+$EndComp
+Wire Wire Line
+	9925 2075 9925 2250
+Wire Wire Line
+	9925 2975 9925 2850
+Wire Wire Line
+	9375 2075 9925 2075
+Wire Wire Line
+	9525 2975 9925 2975
+Wire Wire Line
+	9575 2175 9575 2550
+Wire Wire Line
+	9525 3225 9525 3425
+$Comp
+L power:GND #PWR?
+U 1 1 5B071E70
+P 10375 3050
+F 0 "#PWR?" H 10375 2800 50  0001 C CNN
+F 1 "GND" H 10380 2877 50  0000 C CNN
+F 2 "" H 10375 3050 50  0001 C CNN
+F 3 "" H 10375 3050 50  0001 C CNN
+	1    10375 3050
+	1    0    0    -1
+$EndComp
+$Comp
+L power:GND #PWR?
+U 1 1 5B071EFF
+P 10775 3050
+F 0 "#PWR?" H 10775 2800 50  0001 C CNN
+F 1 "GND" H 10780 2877 50  0000 C CNN
+F 2 "" H 10775 3050 50  0001 C CNN
+F 3 "" H 10775 3050 50  0001 C CNN
+	1    10775 3050
+	1    0    0    -1
+$EndComp
+Wire Wire Line
+	10375 2975 10375 3050
+Wire Wire Line
+	10775 3050 10775 2975
+Wire Wire Line
+	10375 2675 10375 2550
+Connection ~ 10375 2550
+Wire Wire Line
+	10375 2550 10775 2550
+Wire Wire Line
+	10775 2675 10775 2550
+Connection ~ 10775 2550
+Wire Wire Line
+	10775 2550 10850 2550
 $EndSCHEMATC
