File: kicad/haathi_camera.sch (KiCad schematic (older format))
At the start: 0 parts

Commit message: Mayank, reverse polarity protection and test points
Parts:
- added J?: Conn_02x08_Odd_Even, symbol haathi_mayank:Conn_02x08_Odd_Even
Changed lines of the file:
@@
 Comment4 ""
 $EndDescr
+$Comp
+L haathi_mayank:Conn_02x08_Odd_Even J?
+U 1 1 5A760D6D
+P 3400 2000
+F 0 "J?" H 3450 2517 50  0000 C CNN
+F 1 "Conn_02x08_Odd_Even" H 3450 2426 50  0000 C CNN
+F 2 "" H 3400 2000 50  0001 C CNN
+F 3 "~" H 3400 2000 50  0001 C CNN
+	1    3400 2000
+	1    0    0    -1
+$EndComp
 $EndSCHEMATC

Commit message: Mayank, Camera sheet done with Arducam and FRC header
Parts:
- removed J?: Conn_02x08_Odd_Even, symbol haathi_mayank:Conn_02x08_Odd_Even
- added D?: D_Schottky, symbol haathi_mayank:D_Schottky
- added J?: Conn_01x20, symbol haathi_mayank:Conn_01x20
- added J?: Conn_02x10_Odd_Even, symbol haathi_mayank:Conn_02x10_Odd_Even
- added R? (x3): 10k, symbol haathi_mayank:R
- added R? (x19): 0E, symbol haathi_mayank:R
- added R?: 10k_DNP, symbol haathi_mayank:R
Connections:
- net labels added: CSI_D0, CSI_D1, CSI_D2, CSI_D3, CSI_D4, CSI_D5, CSI_D6, CSI_D7, CSI_D8, CSI_D9, CSI_GIO_0, CSI_GIO_1, CSI_GIO_2, CSI_GIO_3, CSI_HSYNC, CSI_I2C_SCL, CSI_I2C_SDA, CSI_PCLK, CSI_PWDN, CSI_RESET, CSI_VSYNC, CSI_XCLK, GND, GPIO_AD_B1_04, GPIO_AD_B1_05, GPIO_AD_B1_06, GPIO_AD_B1_07, GPIO_AD_B1_08, GPIO_AD_B1_09, GPIO_AD_B1_10, GPIO_AD_B1_11, GPIO_AD_B1_12, GPIO_AD_B1_13, GPIO_AD_B1_14, GPIO_AD_B1_15, GPIO_B1_06, GPIO_B1_07, GPIO_B1_08, GPIO_B1_09, GPIO_B1_10, GPIO_B1_11, I2C1_SCL, I2C1_SDA, VCC
- wire segments 0 -> 100
Other:
- note added: "Arducam Camera Connector"
- note added: "CSI Pin Mappings\n"
- note added: "CSI_DATA_10..13 (Table 4-1 Ref Manual)\n"
- note added: "Camera FRC Connector"

Commit message: Camera modified FRC connector and D9 to D0 on Box header
Parts:
- removed D?: D_Schottky, symbol haathi_mayank:D_Schottky
- removed J?: Conn_01x20, symbol haathi_mayank:Conn_01x20
- removed R?: 10k_DNP, symbol haathi_mayank:R
- added J?: Conn_01x30, symbol haathi_mayank:Conn_01x30
- added R? (x3): 0E, symbol haathi_mayank:R
- added R?: 10k, symbol haathi_mayank:R
Connections:
- net labels added: CSI_D10, CSI_D11, CSI_FLASH, CSI_STANDBY, CSI_TRIG, GPIO_EMC_30, GPIO_EMC_31, GPIO_EMC_32, GPIO_EMC_33
- net labels removed: CSI_PWDN, GPIO_B1_06, GPIO_B1_07
- wire segments 100 -> 122
Other:
- note added: "CSI_DATA_20..23 (Table 4-1 Ref Manual)\n"
- note removed: "CSI_DATA_10..13 (Table 4-1 Ref Manual)\n"

Commit message: Mayank, Camera: Renamed arducam connectors
Parts:
- J?: value Conn_02x10_Odd_Even -> Conn2x10_ArduCAM_Box
- J?: value Conn_01x30 -> Conn_01x30_ArduCAM_FRC
Changed lines of the file:
@@
 EESchema Schematic File Version 4
-LIBS:haathi-cache
 EELAYER 26 0
 EELAYER END
 $Descr A4 11693 8268
 encoding utf-8
-Sheet 11 12
+Sheet 1 1
 Title ""
 Date ""
@@
 P 5850 2300
 F 0 "J?" H 5900 2917 50  0000 C CNN
-F 1 "Conn_02x10_Odd_Even" H 5900 2826 50  0000 C CNN
+F 1 "Conn2x10_ArduCAM_Box" H 5900 2826 50  0000 C CNN
 F 2 "" H 5850 2300 50  0001 C CNN
 F 3 "~" H 5850 2300 50  0001 C CNN
@@
 P 3100 2750
 F 0 "J?" H 3180 2742 50  0000 L CNN
-F 1 "Conn_01x30" H 3180 2651 50  0000 L CNN
+F 1 "Conn_01x30_ArduCAM_FRC" H 3180 2651 50  0000 L CNN
 F 2 "" H 3100 2750 50  0001 C CNN
 F 3 "~" H 3100 2750 50  0001 C CNN

Commit message: Mayank, Camera, replaced VCC with +3V3 Flags
Connections:
- net labels added: +3V3
- net labels removed: VCC
Changed lines of the file:
@@
 EESchema Schematic File Version 4
+LIBS:haathi_camera-cache
 EELAYER 26 0
 EELAYER END
@@
 Wire Wire Line
 	6150 2600 6400 2600
-$Comp
-L power:VCC #PWR?
-U 1 1 5A86619C
-P 5150 1650
-F 0 "#PWR?" H 5150 1500 50  0001 C CNN
-F 1 "VCC" H 5167 1823 50  0000 C CNN
-F 2 "" H 5150 1650 50  0001 C CNN
-F 3 "" H 5150 1650 50  0001 C CNN
-	1    5150 1650
-	1    0    0    -1
-$EndComp
 $Comp
 L power:PWR_FLAG #FLG?
@@
 $EndComp
 $Comp
-L power:VCC #PWR?
-U 1 1 5A86712D
-P 5850 3200
-F 0 "#PWR?" H 5850 3050 50  0001 C CNN
-F 1 "VCC" H 5867 3373 50  0000 C CNN
-F 2 "" H 5850 3200 50  0001 C CNN
-F 3 "" H 5850 3200 50  0001 C CNN
-	1    5850 3200
-	1    0    0    -1
-$EndComp
-$Comp
 L haathi_mayank:R R?
 U 1 1 5A867A89
@@
 	1    5850 4100
 	0    1    1    0
-$EndComp
-$Comp
-L power:VCC #PWR?
-U 1 1 5A868A8E
-P 5850 4050
-F 0 "#PWR?" H 5850 3900 50  0001 C CNN
-F 1 "VCC" H 5867 4223 50  0000 C CNN
-F 2 "" H 5850 4050 50  0001 C CNN
-F 3 "" H 5850 4050 50  0001 C CNN
-	1    5850 4050
-	1    0    0    -1
 $EndComp
 $Comp
@@
 	2400 5800 2750 5800
 $Comp
-L power:VCC #PWR?
-U 1 1 5A8B8794
-P 2400 5400
-F 0 "#PWR?" H 2400 5250 50  0001 C CNN
-F 1 "VCC" H 2417 5573 50  0000 C CNN
-F 2 "" H 2400 5400 50  0001 C CNN
-F 3 "" H 2400 5400 50  0001 C CNN
-	1    2400 5400
-	1    0    0    -1
-$EndComp
-$Comp
 L power:PWR_FLAG #FLG?
 U 1 1 5A8B87D3
@@
 Wire Wire Line
 	1050 3900 1050 3750
-$Comp
-L power:VCC #PWR?
-U 1 1 5A915145
-P 1050 3750
-F 0 "#PWR?" H 1050 3600 50  0001 C CNN
-F 1 "VCC" H 1067 3923 50  0000 C CNN
-F 2 "" H 1050 3750 50  0001 C CNN
-F 3 "" H 1050 3750 50  0001 C CNN
-	1    1050 3750
-	1    0    0    -1
-$EndComp
 Wire Wire Line
 	1950 3650 2900 3650
@@
 Wire Wire Line
 	2400 6300 2400 6350
+$Comp
+L power:+3V3 #PWR?
+U 1 1 5AA2E81A
+P 5150 1650
+F 0 "#PWR?" H 5150 1500 50  0001 C CNN
+F 1 "+3V3" H 5165 1823 50  0000 C CNN
+F 2 "" H 5150 1650 50  0001 C CNN
+F 3 "" H 5150 1650 50  0001 C CNN
+	1    5150 1650
+	1    0    0    -1
+$EndComp
+$Comp
+L power:+3V3 #PWR?
+U 1 1 5AA2E864
+P 5850 3200
+F 0 "#PWR?" H 5850 3050 50  0001 C CNN
+F 1 "+3V3" H 5865 3373 50  0000 C CNN
+F 2 "" H 5850 3200 50  0001 C CNN
+F 3 "" H 5850 3200 50  0001 C CNN
+	1    5850 3200
+	1    0    0    -1
+$EndComp
+$Comp
+L power:+3V3 #PWR?
+U 1 1 5AA2EA1E
+P 5850 4050
+F 0 "#PWR?" H 5850 3900 50  0001 C CNN
+F 1 "+3V3" H 5865 4223 50  0000 C CNN
+F 2 "" H 5850 4050 50  0001 C CNN
+F 3 "" H 5850 4050 50  0001 C CNN
+	1    5850 4050
+	1    0    0    -1
+$EndComp
+$Comp
+L power:+3V3 #PWR?
+U 1 1 5AA2EB30
+P 1050 3750
+F 0 "#PWR?" H 1050 3600 50  0001 C CNN
+F 1 "+3V3" H 1065 3923 50  0000 C CNN
+F 2 "" H 1050 3750 50  0001 C CNN
+F 3 "" H 1050 3750 50  0001 C CNN
+	1    1050 3750
+	1    0    0    -1
+$EndComp
+$Comp
+L power:+3V3 #PWR?
+U 1 1 5AA2EE72
+P 2400 5400
+F 0 "#PWR?" H 2400 5250 50  0001 C CNN
+F 1 "+3V3" H 2415 5573 50  0000 C CNN
+F 2 "" H 2400 5400 50  0001 C CNN
+F 3 "" H 2400 5400 50  0001 C CNN
+	1    2400 5400
+	1    0    0    -1
+$EndComp
 $EndSCHEMATC
