File: kicad/haathi_camera.sch (KiCad schematic (older format))
At the start: 28 parts

Commit message: Make the internal camera signals local not hierarchical
Connections:
- wire segments 122 -> 120

Commit message: Annotated schematic
Parts:
- gave numbers to parts that had none: 28

Commit message: ERC pass 1: Check and resolve the errors
Signed-off-by: Kumar Abhishek <abhishek@theembeddedkitchen.net>
Connections:
- wire segments 120 -> 114
Changed lines of the file:
@@
 EESchema Schematic File Version 4
-LIBS:haathi_schematic-cache
+LIBS:haathi-cache
 EELAYER 26 0
 EELAYER END
 $Descr A4 11693 8268
 encoding utf-8
-Sheet 1 9
+Sheet 10 11
 Title "haathi_cam"
 Date "2018-03-11"
@@
 $EndComp
 $Comp
-L power:PWR_FLAG #FLG017
-U 1 1 5A866259
-P 5150 1700
-F 0 "#FLG017" H 5150 1775 50  0001 C CNN
-F 1 "PWR_FLAG" V 5150 1828 50  0000 L CNN
-F 2 "" H 5150 1700 50  0001 C CNN
-F 3 "" H 5150 1700 50  0001 C CNN
-	1    5150 1700
-	0    -1   -1   0
-$EndComp
-$Comp
 L power:GND #PWR0105
 U 1 1 5A86664D
@@
 Wire Wire Line
 	5650 1900 5150 1900
-Wire Wire Line
-	5150 1900 5150 1700
-Connection ~ 5150 1700
-Wire Wire Line
-	5150 1700 5150 1650
 Text HLabel 6250 3650 2    50   Input ~ 0
 I2C1_SCL
-$Comp
-L power:PWR_FLAG #FLG018
-U 1 1 5A86711E
-P 5850 3250
-F 0 "#FLG018" H 5850 3325 50  0001 C CNN
-F 1 "PWR_FLAG" V 5850 3378 50  0000 L CNN
-F 2 "" H 5850 3250 50  0001 C CNN
-F 3 "" H 5850 3250 50  0001 C CNN
-	1    5850 3250
-	0    1    1    0
-$EndComp
 $Comp
 L haathi_mayank:R R89
@@
 Wire Wire Line
 	5850 3650 6250 3650
-Wire Wire Line
-	5850 3200 5850 3250
-Connection ~ 5850 3250
-Wire Wire Line
-	5850 3250 5850 3350
 Connection ~ 5850 3650
 Text HLabel 6250 4500 2    50   Input ~ 0
 I2C1_SDA
-$Comp
-L power:PWR_FLAG #FLG019
-U 1 1 5A868A88
-P 5850 4100
-F 0 "#FLG019" H 5850 4175 50  0001 C CNN
-F 1 "PWR_FLAG" V 5850 4228 50  0000 L CNN
-F 2 "" H 5850 4100 50  0001 C CNN
-F 3 "" H 5850 4100 50  0001 C CNN
-	1    5850 4100
-	0    1    1    0
-$EndComp
 $Comp
 L haathi_mayank:R R90
@@
 Wire Wire Line
 	5850 4500 6250 4500
-Wire Wire Line
-	5850 4050 5850 4100
-Connection ~ 5850 4100
-Wire Wire Line
-	5850 4100 5850 4200
 Connection ~ 5850 4500
 $Comp
@@
 	2400 5800 2750 5800
 $Comp
-L power:PWR_FLAG #FLG016
-U 1 1 5A8B87D3
-P 2350 5450
-F 0 "#FLG016" H 2350 5525 50  0001 C CNN
-F 1 "PWR_FLAG" V 2350 5578 50  0000 L CNN
-F 2 "" H 2350 5450 50  0001 C CNN
-F 3 "" H 2350 5450 50  0001 C CNN
-	1    2350 5450
-	0    -1   -1   0
-$EndComp
-Wire Wire Line
-	2400 5400 2400 5450
-Wire Wire Line
-	2350 5450 2400 5450
-Connection ~ 2400 5450
-Wire Wire Line
-	2400 5450 2400 5500
-$Comp
 L haathi_mayank:Conn_01x30 J11
 U 1 1 5A8A94B7
@@
 Wire Wire Line
 	2550 3950 1050 3950
-Wire Wire Line
-	1050 3950 1050 3900
 Connection ~ 2550 3950
-$Comp
-L power:PWR_FLAG #FLG015
-U 1 1 5A915050
-P 1050 3900
-F 0 "#FLG015" H 1050 3975 50  0001 C CNN
-F 1 "PWR_FLAG" V 1050 4028 50  0000 L CNN
-F 2 "" H 1050 3900 50  0001 C CNN
-F 3 "" H 1050 3900 50  0001 C CNN
-	1    1050 3900
-	0    -1   -1   0
-$EndComp
-Connection ~ 1050 3900
-Wire Wire Line
-	1050 3900 1050 3750
 Wire Wire Line
 	1950 3650 2900 3650
@@
 Text Label 2350 3850 0    50   ~ 0
 CSI_STANDBY
+Wire Wire Line
+	5850 3200 5850 3350
+Wire Wire Line
+	5850 4050 5850 4200
+Wire Wire Line
+	2400 5400 2400 5500
+Wire Wire Line
+	1050 3750 1050 3950
+Wire Wire Line
+	5150 1650 5150 1900
 $EndSCHEMATC

Commit message: Updated the pin numbers to the camera as per the format of the new pin mapping.
Connections:
- net labels added: GPIO_AD_B0_04, GPIO_AD_B0_05, GPIO_AD_B0_15, GPIO_AD_B1_00, GPIO_AD_B1_01, GPIO_B1_13, GPIO_EMC_39, GPIO_EMC_41, GPIO_SD_B1_04, GPIO_SD_B1_05
- net labels removed: GPIO_AD_B1_06, GPIO_AD_B1_07, GPIO_AD_B1_08, GPIO_AD_B1_09, GPIO_EMC_30, GPIO_EMC_31, GPIO_EMC_32, GPIO_EMC_33, I2C1_SCL, I2C1_SDA
Changed lines of the file:
@@
 EESchema Schematic File Version 4
-LIBS:haathi-cache
+LIBS:haathi_camera-cache
 EELAYER 26 0
 EELAYER END
 $Descr A4 11693 8268
 encoding utf-8
-Sheet 10 11
+Sheet 1 1
 Title "haathi_cam"
 Date "2018-03-11"
@@
 	5650 1900 5150 1900
 Text HLabel 6250 3650 2    50   Input ~ 0
-I2C1_SCL
+GPIO_AD_B1_00
 $Comp
 L haathi_mayank:R R89
@@
 Connection ~ 5850 3650
 Text HLabel 6250 4500 2    50   Input ~ 0
-I2C1_SDA
+GPIO_AD_B1_01
 $Comp
 L haathi_mayank:R R90
@@
 GPIO_AD_B1_05
 Text HLabel 9100 1550 2    50   Input ~ 0
-GPIO_AD_B1_06
+GPIO_B1_13
 Text HLabel 9100 1650 2    50   Input ~ 0
-GPIO_AD_B1_07
+GPIO_AD_B0_15
 Text HLabel 9150 2400 2    50   Input ~ 0
 GPIO_AD_B1_10
@@
 	8750 2300 9150 2300
 Text HLabel 9150 2300 2    50   Input ~ 0
-GPIO_AD_B1_09
+GPIO_AD_B0_05
 Text HLabel 9150 2200 2    50   Input ~ 0
-GPIO_AD_B1_08
+GPIO_AD_B0_04
 Text Notes 7750 4150 0    50   ~ 0
 CSI_DATA_20..23 (Table 4-1 Ref Manual)\n
@@
 GPIO_B1_08
 Text HLabel 9150 3500 2    50   Input ~ 0
-GPIO_EMC_33
+GPIO_EMC_41
 Text HLabel 9150 3600 2    50   Input ~ 0
-GPIO_EMC_32
+GPIO_EMC_39
 Text HLabel 9150 3800 2    50   Input ~ 0
-GPIO_EMC_31
+GPIO_SD_B1_04
 Text HLabel 9150 3900 2    50   Input ~ 0
-GPIO_EMC_30
+GPIO_SD_B1_05
 $Comp
 L haathi_mayank:R R96
