File: kicad/haathi_sdram.sch (KiCad schematic (older format))
At the start: 0 parts

Commit message: Anool, updated SD-RAM schematic
Parts:
- added C? (x7): 100nF, 0603, symbol haathi:C_NP
- added C?: 22uF,6.3V, 0603, symbol haathi:C_NP
- added C?: 4.7uF,6.3V, 0603, symbol haathi:C_NP
- added R? (x2): 0E, symbol haathi:R
- added U?: MT48LC16M16A2B4, symbol haathi:MT48LC16M16A2B4
Connections:
- net labels added: DCDC_IN, E2, GND, SDRAM_CLK, SD_RAM_3V3, SEMC_A0, SEMC_A1, SEMC_A10, SEMC_A11, SEMC_A12, SEMC_A2, SEMC_A3, SEMC_A4, SEMC_A5, SEMC_A6, SEMC_A7, SEMC_A8, SEMC_A9, SEMC_A[0..12], SEMC_BA0, SEMC_BA1, SEMC_CAS, SEMC_CKE, SEMC_CLK, SEMC_CS0, SEMC_D0, SEMC_D1, SEMC_D10, SEMC_D11, SEMC_D12, SEMC_D13, SEMC_D14, SEMC_D15, SEMC_D2, SEMC_D3, SEMC_D4, SEMC_D5, SEMC_D6, SEMC_D7, SEMC_D8, SEMC_D9, SEMC_DM0, SEMC_DM1, SEMC_D[0..7], SEMC_D[8..15], SEMC_RAS, SEMC_WE
- wire segments 0 -> 91
- no-connect marks 0 -> 1
Other:
- note added: "150mA @ 3V3"
- note added: "One Capacitor for each\npower pin pair"
