File: kicad/haathi_memory.sch (KiCad schematic (older format))
At the start: 0 parts

Commit message: Anool, Memory schematic WIP
Parts:
- added C10, C9: 18pF, symbol haathi:C_NP
- added C6: 22uF,6.3V, symbol haathi:C_NP
- added C7: 4.7uF,6.3V, symbol haathi:C_NP
- added C8: 100nF, symbol haathi:C_NP
- added Q1: BC817, Package_TO_SOT_SMD:SOT-23, symbol haathi:BC817
- added R10, R11, R7: 0E, symbol haathi:R
- added R12, R13, R8, R9: 10k, symbol haathi:R
- added SD1: SD_CARD_Micro, symbol haathi:SD_CARD_Micro
Connections:
- net labels added: GND, GPIO_SD_B0_01_B, SD_CD_SW, SD_CLK, SD_CMD, SD_D0, SD_D1, SD_D2, SD_D3, VSD_3V3
- wire segments 0 -> 76
Other:
- note added: "FOR SD BOOT, ROM NEED SD_CD_SW PIN KEPT LOW\n===========================================\nCARD INSERT\nCD1&CD2 FLOAT-->Q14 ON-->SD_CD_SW LOW\n\nCARD OFF\nCD1&CD2 GND-->Q14 OFF-->SD_CD_SW HIGH"

Commit message: Mayank, SD card: Removed Transistor on Card Detect pin
Parts:
- removed Q1: BC817, Package_TO_SOT_SMD:SOT-23, symbol haathi:BC817
- removed R10: 0E, symbol haathi:R
- removed R12, R9: 10k, symbol haathi:R
Connections:
- wire segments 76 -> 62
Other:
- note removed: "FOR SD BOOT, ROM NEED SD_CD_SW PIN KEPT LOW\n===========================================\nCARD INSERT\nCD1&CD2 FLOAT-->Q14 ON-->SD_CD_SW LOW\n\nCARD OFF\nCD1&CD2 GND-->Q14 OFF-->SD_CD_SW HIGH"
Changed lines of the file:
@@
 EESchema Schematic File Version 4
-LIBS:haathi-cache
+LIBS:haathi_memory-cache
 EELAYER 26 0
 EELAYER END
 $Descr A4 11693 8268
 encoding utf-8
-Sheet 7 12
+Sheet 1 1
 Title ""
 Date ""
@@
 $EndComp
 $Comp
-L haathi:R R12
-U 1 1 5A6E3401
-P 5975 3100
-F 0 "R12" H 6000 3250 50  0000 L CNN
-F 1 "10k" V 5975 3025 50  0000 L CNN
-F 2 "" V 5905 3100 30  0000 C CNN
-F 3 "" H 5975 3100 30  0000 C CNN
-	1    5975 3100
-	1    0    0    -1
-$EndComp
-$Comp
-L haathi:R R9
-U 1 1 5A6E3455
-P 6350 2300
-F 0 "R9" H 6375 2450 50  0000 L CNN
-F 1 "10k" V 6350 2225 50  0000 L CNN
-F 2 "" V 6280 2300 30  0000 C CNN
-F 3 "" H 6350 2300 30  0000 C CNN
-	1    6350 2300
-	1    0    0    -1
-$EndComp
-$Comp
-L haathi:R R10
-U 1 1 5A6E34C9
-P 6875 2475
-F 0 "R10" V 6775 2475 50  0000 C CNN
-F 1 "0E" V 6875 2475 50  0000 C CNN
-F 2 "" V 6805 2475 30  0000 C CNN
-F 3 "" H 6875 2475 30  0000 C CNN
-	1    6875 2475
-	0    1    1    0
-$EndComp
-$Comp
 L haathi:R R7
 U 1 1 5A6E355E
-P 6875 1850
-F 0 "R7" V 6775 1850 50  0000 C CNN
-F 1 "0E" V 6875 1850 50  0000 C CNN
-F 2 "" V 6805 1850 30  0000 C CNN
-F 3 "" H 6875 1850 30  0000 C CNN
-	1    6875 1850
+P 6350 2700
+F 0 "R7" V 6250 2700 50  0000 C CNN
+F 1 "0E" V 6350 2700 50  0000 C CNN
+F 2 "" V 6280 2700 30  0000 C CNN
+F 3 "" H 6350 2700 30  0000 C CNN
+	1    6350 2700
 	0    1    1    0
-$EndComp
-$Comp
-L haathi:BC817 Q1
-U 1 1 5A6E58D8
-P 6250 2700
-F 0 "Q1" H 6475 2775 50  0000 L CNN
-F 1 "BC817" H 6475 2700 50  0000 L CNN
-F 2 "Package_TO_SOT_SMD:SOT-23" H 6450 2625 50  0001 L CIN
-F 3 "http://www.fairchildsemi.com/ds/BC/BC817.pdf" H 6250 2700 50  0001 L CNN
-	1    6250 2700
-	1    0    0    -1
 $EndComp
 Wire Wire Line
@@
 	5975 2450 5975 2700
 Wire Wire Line
-	6100 2700 5975 2700
-Connection ~ 5975 2700
-Wire Wire Line
-	5975 2700 5975 2950
-Wire Wire Line
 	5350 2700 5475 2700
 Wire Wire Line
@@
 Connection ~ 5475 2700
 Wire Wire Line
-	6350 2500 6350 2475
-Wire Wire Line
-	6725 2475 6350 2475
-Connection ~ 6350 2475
-Wire Wire Line
-	6350 2475 6350 2450
-Wire Wire Line
-	6350 2900 6350 3300
-Wire Wire Line
-	6350 3300 5975 3300
-Connection ~ 5200 3300
-Wire Wire Line
-	5975 3250 5975 3300
-Connection ~ 5975 3300
-Wire Wire Line
-	5975 3300 5200 3300
-Wire Wire Line
-	7025 2475 7125 2475
-Wire Wire Line
-	7125 2475 7125 1850
-Wire Wire Line
-	7125 1850 7025 1850
-Wire Wire Line
-	6725 1850 5475 1850
-Wire Wire Line
-	5475 1850 5475 2700
-Wire Wire Line
 	5975 2150 5975 1700
 Wire Wire Line
-	5975 1700 6350 1700
-Wire Wire Line
-	6350 1700 6350 2150
-Wire Wire Line
-	7125 1850 7125 1300
-Wire Wire Line
 	7125 1300 2300 1300
 Wire Wire Line
@@
 Wire Wire Line
 	2300 2400 1700 2400
-Connection ~ 7125 1850
 Wire Wire Line
 	2800 1700 1700 1700
@@
 	4225 1700 5975 1700
 Connection ~ 4225 1700
-Connection ~ 5975 1700
 Text Label 1700 1700 0    50   ~ 0
 VSD_3V3
@@
 Text Label 1700 2800 0    50   ~ 0
 GPIO_SD_B0_01_B
-Text Notes 6475 3325 0    40   ~ 0
-FOR SD BOOT, ROM NEED SD_CD_SW PIN KEPT LOW\n===========================================\nCARD INSERT\nCD1&CD2 FLOAT-->Q14 ON-->SD_CD_SW LOW\n\nCARD OFF\nCD1&CD2 GND-->Q14 OFF-->SD_CD_SW HIGH
+Wire Wire Line
+	5975 2700 6200 2700
+Connection ~ 5975 2700
+Wire Wire Line
+	6500 2700 7125 2700
+Wire Wire Line
+	7125 1300 7125 2700
 $EndSCHEMATC

Commit message: Mayank, added QSPI Flash symbol and connections
Parts:
- added C?: 0.1uF, symbol haathi_mayank:C_NP
- added C?: 1uF, symbol haathi_mayank:C_NP
- added U?: IS25WP080D, symbol haathi_mayank:IS25WP080D
Connections:
- net labels added: +1V8, FlexSPI_CLK, FlexSPI_D0_A, FlexSPI_D1_A, FlexSPI_D2_A, FlexSPI_D3_A, FlexSPI_SS0
- wire segments 62 -> 75
Changed lines of the file:
@@
 Wire Wire Line
 	7125 1300 7125 2700
+$Comp
+L haathi_mayank:IS25WP080D U?
+U 1 1 5AA454AE
+P 4800 5125
+F 0 "U?" H 4350 5450 50  0000 C CNN
+F 1 "IS25WP080D" H 5125 4625 50  0000 C CNN
+F 2 "" H 4350 4975 50  0001 C CNN
+F 3 "" H 4350 4975 50  0001 C CNN
+	1    4800 5125
+	1    0    0    -1
+$EndComp
+Wire Wire Line
+	4200 5075 3850 5075
+Wire Wire Line
+	4200 5175 3850 5175
+Wire Wire Line
+	4200 5275 3850 5275
+Wire Wire Line
+	4200 5375 3850 5375
+$Comp
+L power:+1V8 #PWR?
+U 1 1 5AA46B0D
+P 5675 4400
+F 0 "#PWR?" H 5675 4250 50  0001 C CNN
+F 1 "+1V8" H 5690 4573 50  0000 C CNN
+F 2 "" H 5675 4400 50  0001 C CNN
+F 3 "" H 5675 4400 50  0001 C CNN
+	1    5675 4400
+	1    0    0    -1
+$EndComp
+Wire Wire Line
+	5125 4400 4800 4400
+Wire Wire Line
+	4800 4400 4800 4775
+$Comp
+L power:GND #PWR?
+U 1 1 5AA47F6E
+P 4800 5775
+F 0 "#PWR?" H 4800 5525 50  0001 C CNN
+F 1 "GND" H 4900 5775 50  0000 C CNN
+F 2 "" H 4800 5775 50  0001 C CNN
+F 3 "" H 4800 5775 50  0001 C CNN
+	1    4800 5775
+	1    0    0    -1
+$EndComp
+Wire Wire Line
+	4800 5675 4800 5775
+Wire Wire Line
+	5450 5075 5925 5075
+Wire Wire Line
+	5450 5275 5925 5275
+$Comp
+L haathi_mayank:C_NP C?
+U 1 1 5AA4AEFD
+P 5125 4550
+F 0 "C?" H 5228 4588 40  0000 L CNN
+F 1 "0.1uF" H 5228 4512 40  0000 L CNN
+F 2 "" H 5125 4550 60  0000 C CNN
+F 3 "" H 5125 4550 60  0000 C CNN
+	1    5125 4550
+	1    0    0    -1
+$EndComp
+$Comp
+L haathi_mayank:C_NP C?
+U 1 1 5AA4AF9F
+P 5500 4550
+F 0 "C?" H 5603 4588 40  0000 L CNN
+F 1 "1uF" H 5603 4512 40  0000 L CNN
+F 2 "" H 5500 4550 60  0000 C CNN
+F 3 "" H 5500 4550 60  0000 C CNN
+	1    5500 4550
+	1    0    0    -1
+$EndComp
+Wire Wire Line
+	5125 4400 5500 4400
+Connection ~ 5125 4400
+$Comp
+L power:GND #PWR?
+U 1 1 5AA4C96A
+P 5250 4700
+F 0 "#PWR?" H 5250 4450 50  0001 C CNN
+F 1 "GND" H 5375 4625 50  0000 C CNN
+F 2 "" H 5250 4700 50  0001 C CNN
+F 3 "" H 5250 4700 50  0001 C CNN
+	1    5250 4700
+	1    0    0    -1
+$EndComp
+Wire Wire Line
+	5125 4700 5250 4700
+Connection ~ 5250 4700
+Wire Wire Line
+	5250 4700 5500 4700
+Wire Wire Line
+	5500 4400 5675 4400
+Connection ~ 5500 4400
+Text HLabel 3850 5275 0    50   Input ~ 0
+FlexSPI_D0_A
+Text HLabel 3850 5175 0    50   Input ~ 0
+FlexSPI_D1_A
+Text HLabel 5925 5075 2    50   Input ~ 0
+FlexSPI_D2_A
+Text HLabel 5925 5275 2    50   Input ~ 0
+FlexSPI_D3_A
+Text HLabel 3850 5075 0    50   Input ~ 0
+FlexSPI_SS0
+Text HLabel 3850 5375 0    50   Input ~ 0
+FlexSPI_CLK
 $EndSCHEMATC

Commit message: Mayank, added TLV70218 LDO for Flash
Parts:
- added C? (x2): 1uF, symbol haathi_mayank:C_NP
- added U?: TLV70218, symbol haathi_mayank:TLV70218
Connections:
- net labels added: +3V3, SD1_CLK, SD1_CMD, SD1_D0, SD1_D1, SD1_D2, SD1_D3
- wire segments 75 -> 88

Commit message: Mayank, added SD Card variable voltage regulator ckt and changed supply to NVCC_SD0
Parts:
- added C? (x2): 0.1uF, symbol haathi_mayank:C_NP
- added Q?: Q_NMOS_GSD, symbol haathi_mayank:Q_NMOS_GSD
- added R?: 47K, symbol haathi_mayank:R
- added R?: 93.1K, symbol haathi_mayank:R
- added R?: 37.4K, symbol haathi_mayank:R
- added R?: 100K, symbol haathi_mayank:R
- added TP?: TP_1V8, symbol haathi_mayank:Test_Point_Probe
- added TP?: TP_NVCC_SD0, symbol haathi_mayank:Test_Point_Probe
- added U?: TPS73101, symbol haathi_mayank:TPS73101
Connections:
- net labels added: NVCC_SD0, SD0_VSELECT
- wire segments 88 -> 119

Commit message: Edited NVCC_SD0 label on memory sheet TPS73101 output
Connections:
- net labels removed: VSD_3V3
Changed lines of the file:
@@
 EESchema Schematic File Version 4
-LIBS:haathi-cache
 EELAYER 26 0
 EELAYER END
 $Descr A4 11693 8268
 encoding utf-8
-Sheet 1 11
+Sheet 1 1
 Title "haathi_cam"
 Date "2018-03-11"
@@
 Text HLabel 10150 2225 2    50   Input ~ 0
 NVCC_SD0
-Text Label 9650 2225 0    50   ~ 0
-VSD_3V3
 $Comp
 L haathi_mayank:R R?
@@
 Wire Wire Line
 	10100 2225 10150 2225
+Text Label 9525 2225 0    50   ~ 0
+NVCC_SD0
 $EndSCHEMATC

Commit message: Memory sheet, changed supply of SD to 3V3 and removed extra GPIO tap to SD_CLK
Connections:
- net labels removed: GPIO_SD_B0_01_B
- wire segments 119 -> 118
Changed lines of the file:
@@
 $EndComp
-Wire Wire Line
-	3400 2800 1700 2800
-Connection ~ 3400 2800
 Wire Wire Line
 	2200 2650 2200 2600
@@
 	4225 1700 5975 1700
 Connection ~ 4225 1700
-Text Label 1700 1700 0    50   ~ 0
-NVCC_SD0
 Text Label 1700 2400 0    50   ~ 0
 SD_CD_SW
@@
 Text Label 1700 3100 0    50   ~ 0
 SD_CLK
-Text Label 1700 2800 0    50   ~ 0
-GPIO_SD_B0_01_B
 Wire Wire Line
 	5975 2700 6200 2700
@@
 Text HLabel 1700 2400 0    50   Input ~ 0
 SD_CD_SW
-Text HLabel 1700 1700 0    50   Input ~ 0
-NVCC_SD0
 $Comp
 L haathi_mayank:TLV70218 U?
@@
 L power:+3V3 #PWR?
 U 1 1 5AA68EC5
-P 7900 2200
-F 0 "#PWR?" H 7900 2050 50  0001 C CNN
-F 1 "+3V3" H 7915 2373 50  0000 C CNN
-F 2 "" H 7900 2200 50  0001 C CNN
-F 3 "" H 7900 2200 50  0001 C CNN
-	1    7900 2200
+P 1700 1700
+F 0 "#PWR?" H 1700 1550 50  0001 C CNN
+F 1 "+3V3" H 1715 1873 50  0000 C CNN
+F 2 "" H 1700 1700 50  0001 C CNN
+F 3 "" H 1700 1700 50  0001 C CNN
+	1    1700 1700
 	1    0    0    -1
 $EndComp
@@
 Text Label 9525 2225 0    50   ~ 0
 NVCC_SD0
+$Comp
+L power:+3V3 #PWR?
+U 1 1 5AA6DC7F
+P 7900 2200
+F 0 "#PWR?" H 7900 2050 50  0001 C CNN
+F 1 "+3V3" H 7915 2373 50  0000 C CNN
+F 2 "" H 7900 2200 50  0001 C CNN
+F 3 "" H 7900 2200 50  0001 C CNN
+	1    7900 2200
+	1    0    0    -1
+$EndComp
 $EndSCHEMATC
