File: kicad/haathi_interfaces.sch (KiCad schematic (older format))
At the start: 0 parts

Commit message: Mayank, GPIO and Interfaces: Added JTAG, RGB LED, Buttons and GPIO blank headers
Parts:
- added D?: LED_ARGB, symbol haathi_mayank:LED_ARGB
- added J? (x2): Conn_02x20_Odd_Even, symbol haathi_mayank:Conn_02x20_Odd_Even
- added J?: Conn_ARM_JTAG_SWD_10, Connector_PinHeader_1.27mm:PinHeader_2x05_P1.27mm_Vertical_SMD, symbol haathi_mayank:Conn_ARM_JTAG_SWD_10
- added R? (x5): 0E, symbol haathi_mayank:R
- added R?: 430, symbol haathi_mayank:R
- added R? (x2): 80, symbol haathi_mayank:R
- added S? (x2): SW-SPST-M, symbol haathi_mayank:SW-SPST-M
Connections:
- net labels added: GND, JTAG_TCK, JTAG_TDI, JTAG_TDO, JTAG_TMS, JTAG_nTRST, LED_B, LED_G, LED_R, USER_SW_0, USER_SW_1, VCC
- wire segments 0 -> 41
Other:
- note added: "GPIO Breakout\n"
- note added: "JTAG\n"
- note added: "Raspberry Pi compatible Header\n"
- note added: "User Buttons and RGB LED\n"

Commit message: Interfaces, added USB External signals
Connections:
- net labels added: 5V_USB_HS_EXTERN, USB_GND_EXTERN, USB_OTG2_D+_EXTERN, USB_OTG2_D-_EXTERN, USB_OTG2_ID_EXTERN
- wire segments 41 -> 54
Changed lines of the file:
@@
 Wire Wire Line
 	1600 3800 1850 3800
+Wire Wire Line
+	6500 3450 6150 3450
+Wire Wire Line
+	7000 3450 7350 3450
+Text HLabel 6150 3450 0    50   Input ~ 0
+5V_USB_HS_EXTERN
+Wire Wire Line
+	6500 3550 6150 3550
+Wire Wire Line
+	6500 3650 6150 3650
+Wire Wire Line
+	6500 3750 6150 3750
+Wire Wire Line
+	6500 3850 6150 3850
+Wire Wire Line
+	6500 3950 6150 3950
+Wire Wire Line
+	6500 4050 6150 4050
+Wire Wire Line
+	6500 4150 6150 4150
+Wire Wire Line
+	6500 4250 6150 4250
+Wire Wire Line
+	6500 4350 6150 4350
+Wire Wire Line
+	6500 4450 6150 4450
+Wire Wire Line
+	6500 4550 6150 4550
+Text HLabel 6150 3550 0    50   Input ~ 0
+USB_OTG2_D-_EXTERN
+Text HLabel 6150 3650 0    50   Input ~ 0
+USB_OTG2_D+_EXTERN
+Text HLabel 6150 3750 0    50   Input ~ 0
+USB_OTG2_ID_EXTERN
+Text HLabel 6150 3850 0    50   Input ~ 0
+USB_GND_EXTERN
 $EndSCHEMATC

Commit message: Mayank, added RPi3 interfaces and haathi periph
Connections:
- net labels added: +3V3, 5V_USB_OTG, AUD_INT, BACKLIGHT_CTL, CAN2_RX, CAN2_TX, ENET_CRS_DV, ENET_RXD0, ENET_RXD1, ENET_RXER, ENET_TXD0, ENET_TXD1, ENET_TXEN, ENET_TX_CLK, FlexSPI_CLK_B, FlexSPI_D0_B, FlexSPI_D1_B, FlexSPI_SS_B, I2C1_SCL, I2C1_SDA, LCDIF_CLK, LCDIF_D0, LCDIF_D1, LCDIF_D10, LCDIF_D11, LCDIF_D12, LCDIF_D13, LCDIF_D14, LCDIF_D15, LCDIF_D2, LCDIF_D3, LCDIF_D4, LCDIF_D5, LCDIF_D6, LCDIF_D7, LCDIF_D8, LCDIF_D9, LCDIF_D[15:0], LCDIF_ENABLE, LCDIF_HSYNC, LCDIF_VSYNC, ONOFF, SAI1_MCLK, SAI1_RXD, SAI1_RX_BCLK, SAI1_RX_SYNC, SAI1_TXD, SAI1_TX_BCLK, SAI1_TX_SYNC, UART1_RXD, UART1_TXD, WAKEUP_BUTTON
- wire segments 54 -> 134

Commit message: Mayank, corrected bus labels in interfaces and cpu
Connections:
- net labels added: LCDIF_D[0..15]
- net labels removed: LCDIF_D[15:0]
Changed lines of the file:
@@
 	8100 3700 8100 5300
 Text HLabel 8250 3700 2    50   Input ~ 0
-LCDIF_D[15:0]
+LCDIF_D[0..15]
 Text Label 7050 3850 0    50   ~ 0
 LCDIF_D0

Commit message: interfaces, cpu: I2C1 w/o pull-ups and I2C2 w/ pull-ups added, ADC pins broken out to RasPi header
Connections:
- net labels added: GPIO_AD_B0_00, GPIO_AD_B0_01, GPIO_AD_B1_04, GPIO_AD_B1_05, GPIO_AD_B1_06, GPIO_AD_B1_07, I2C2_SCL, I2C2_SDA, SPDIF_IN, SPDIF_OUT
- wire segments 134 -> 135
Changed lines of the file:
@@
 	3700 5300 4050 5300
-Wire Wire Line
-	3700 5400 4050 5400
 Wire Wire Line
 	3200 3600 2850 3600
@@
 Wire Bus Line
 	8100 3700 8250 3700
-Wire Bus Line
-	8100 3700 8100 5300
 Text HLabel 8250 3700 2    50   Input ~ 0
 LCDIF_D[0..15]
@@
 Text HLabel 2850 5200 0    50   Input ~ 0
 ENET_RXER
+Text HLabel 4050 4200 2    50   Input ~ 0
+I2C2_SCL
+Text HLabel 4050 4300 2    50   Input ~ 0
+I2C2_SDA
+Text HLabel 4050 4000 2    50   Input ~ 0
+GPIO_AD_B0_00
+Text HLabel 4050 4500 2    50   Input ~ 0
+GPIO_AD_B0_01
+Text HLabel 4050 4700 2    50   Input ~ 0
+GPIO_AD_B1_04
+Text HLabel 4050 4800 2    50   Input ~ 0
+GPIO_AD_B1_05
+Text HLabel 4050 5000 2    50   Input ~ 0
+GPIO_AD_B1_06
+Text HLabel 4050 5200 2    50   Input ~ 0
+GPIO_AD_B1_07
+Text HLabel 2850 5300 0    50   Input ~ 0
+SPDIF_IN
+Text HLabel 4050 5300 2    50   Input ~ 0
+SPDIF_OUT
+$Comp
+L power:+3V3 #PWR?
+U 1 1 5AB7B7C5
+P 4200 3350
+F 0 "#PWR?" H 4200 3200 50  0001 C CNN
+F 1 "+3V3" H 4215 3523 50  0000 C CNN
+F 2 "" H 4200 3350 50  0001 C CNN
+F 3 "" H 4200 3350 50  0001 C CNN
+	1    4200 3350
+	1    0    0    -1
+$EndComp
+Wire Wire Line
+	4200 3350 4200 5400
+Wire Wire Line
+	3700 5400 4200 5400
+Wire Bus Line
+	8100 3700 8100 5300
 $EndSCHEMATC

Commit message: interfaces: conencted RGB LED and Switches to GPIO pins
Connections:
- net labels added: FlexSPI_D2_B, FlexSPI_D3_B
Changed lines of the file:
@@
 Text Notes 2850 5650 0    50   ~ 0
 Raspberry Pi compatible Header\n
-Text HLabel 1000 3100 0    50   Input ~ 0
+Text HLabel 4800 1600 0    50   Input ~ 0
 LED_R
-Text HLabel 1000 3300 0    50   Input ~ 0
+Text HLabel 4800 1800 0    50   Input ~ 0
 LED_G
-Text HLabel 1000 3500 0    50   Input ~ 0
+Text HLabel 4800 2000 0    50   Input ~ 0
 LED_B
 Wire Wire Line
-	1000 3100 1300 3100
-Wire Wire Line
-	1000 3300 1300 3300
-Wire Wire Line
-	1000 3500 1300 3500
+	4800 1600 5100 1600
+Wire Wire Line
+	4800 1800 5100 1800
+Wire Wire Line
+	4800 2000 5100 2000
 $Comp
 L haathi_mayank:R R?
 U 1 1 5A85A90F
-P 1450 3100
-F 0 "R?" V 1400 3200 50  0000 L CNN
-F 1 "0E" V 1450 3050 50  0000 L CNN
-F 2 "" V 1380 3100 30  0000 C CNN
-F 3 "" H 1450 3100 30  0000 C CNN
-	1    1450 3100
+P 5250 1600
+F 0 "R?" V 5200 1700 50  0000 L CNN
+F 1 "0E" V 5250 1550 50  0000 L CNN
+F 2 "" V 5180 1600 30  0000 C CNN
+F 3 "" H 5250 1600 30  0000 C CNN
+	1    5250 1600
 	0    1    1    0
 $EndComp
 Wire Wire Line
-	1600 3100 1850 3100
+	5400 1600 5650 1600
 $Comp
 L haathi_mayank:R R?
 U 1 1 5A85AEF0
-P 1450 3300
-F 0 "R?" V 1400 3400 50  0000 L CNN
-F 1 "0E" V 1450 3250 50  0000 L CNN
-F 2 "" V 1380 3300 30  0000 C CNN
-F 3 "" H 1450 3300 30  0000 C CNN
-	1    1450 3300
+P 5250 1800
+F 0 "R?" V 5200 1900 50  0000 L CNN
+F 1 "0E" V 5250 1750 50  0000 L CNN
+F 2 "" V 5180 1800 30  0000 C CNN
+F 3 "" H 5250 1800 30  0000 C CNN
+	1    5250 1800
 	0    1    1    0
 $EndComp
@@
 L haathi_mayank:R R?
 U 1 1 5A85AF1E
-P 1450 3500
-F 0 "R?" V 1400 3600 50  0000 L CNN
-F 1 "0E" V 1450 3450 50  0000 L CNN
-F 2 "" V 1380 3500 30  0000 C CNN
-F 3 "" H 1450 3500 30  0000 C CNN
-	1    1450 3500
+P 5250 2000
+F 0 "R?" V 5200 2100 50  0000 L CNN
+F 1 "0E" V 5250 1950 50  0000 L CNN
+F 2 "" V 5180 2000 30  0000 C CNN
+F 3 "" H 5250 2000 30  0000 C CNN
+	1    5250 2000
 	0    1    1    0
 $EndComp
 Wire Wire Line
-	1600 3300 1850 3300
-Wire Wire Line
-	1600 3500 1850 3500
-Text HLabel 1000 3800 0    50   Input ~ 0
+	5400 1800 5650 1800
+Wire Wire Line
+	5400 2000 5650 2000
+Text HLabel 4800 2300 0    50   Input ~ 0
 USER_SW_1
-Text HLabel 1000 3700 0    50   Input ~ 0
+Text HLabel 4800 2200 0    50   Input ~ 0
 USER_SW_0
 Wire Wire Line
-	1000 3700 1300 3700
-Wire Wire Line
-	1000 3800 1300 3800
+	4800 2200 5100 2200
+Wire Wire Line
+	4800 2300 5100 2300
 $Comp
 L haathi_mayank:R R?
 U 1 1 5A85C0CC
-P 1450 3700
-F 0 "R?" V 1400 3800 50  0000 L CNN
-F 1 "0E" V 1450 3650 50  0000 L CNN
-F 2 "" V 1380 3700 30  0000 C CNN
-F 3 "" H 1450 3700 30  0000 C CNN
-	1    1450 3700
+P 5250 2200
+F 0 "R?" V 5200 2300 50  0000 L CNN
+F 1 "0E" V 5250 2150 50  0000 L CNN
+F 2 "" V 5180 2200 30  0000 C CNN
+F 3 "" H 5250 2200 30  0000 C CNN
+	1    5250 2200
 	0    1    1    0
 $EndComp
@@
 L haathi_mayank:R R?
 U 1 1 5A85C0FA
-P 1450 3800
-F 0 "R?" V 1400 3900 50  0000 L CNN
-F 1 "0E" V 1450 3750 50  0000 L CNN
-F 2 "" V 1380 3800 30  0000 C CNN
-F 3 "" H 1450 3800 30  0000 C CNN
-	1    1450 3800
+P 5250 2300
+F 0 "R?" V 5200 2400 50  0000 L CNN
+F 1 "0E" V 5250 2250 50  0000 L CNN
+F 2 "" V 5180 2300 30  0000 C CNN
+F 3 "" H 5250 2300 30  0000 C CNN
+	1    5250 2300
 	0    1    1    0
 $EndComp
 Wire Wire Line
-	1600 3700 1850 3700
-Wire Wire Line
-	1600 3800 1850 3800
+	5400 2200 5650 2200
+Wire Wire Line
+	5400 2300 5650 2300
 Wire Wire Line
 	6500 3450 6150 3450
@@
 Wire Wire Line
 	3700 5400 4200 5400
+Text HLabel 5650 1600 2    50   Input ~ 0
+FlexSPI_D0_B
+Text HLabel 5650 1800 2    50   Input ~ 0
+FlexSPI_D1_B
+Text HLabel 5650 2000 2    50   Input ~ 0
+FlexSPI_D2_B
+Text HLabel 5650 2200 2    50   Input ~ 0
+FlexSPI_D3_B
+Text HLabel 5650 2300 2    50   Input ~ 0
+FlexSPI_CLK_B
 Wire Bus Line
 	8100 3700 8100 5300
