File: kicad/haathi_interfaces.sch (KiCad schematic (older format))
At the start: 16 parts

Commit message: Rearrange buttons and LED pin connections
LED pins go to PWM pins
Switches go to previously SPDIF_IN and OUT pins
FlexSPI 2 pins freed up

Signed-off-by: Kumar Abhishek <abhishek@theembeddedkitchen.net>
Connections:
- net labels added: GPIO_AD_B1_03, GPIO_B1_15, SA1_MCLK
- net labels removed: FlexSPI_D2_B, FlexSPI_D3_B, SPDIF_IN, SPDIF_OUT
Changed lines of the file:
@@
 EESchema Schematic File Version 4
-LIBS:haathi_schematic-cache
+LIBS:haathi-cache
 EELAYER 26 0
 EELAYER END
 $Descr A4 11693 8268
 encoding utf-8
-Sheet 6 9
+Sheet 8 11
 Title "haathi_cam"
 Date "2018-03-11"
@@
 	3700 5400 4200 5400
 Text HLabel 5650 2000 2    50   Input ~ 0
-FlexSPI_D2_B
-Text HLabel 5650 2200 2    50   Input ~ 0
-FlexSPI_D3_B
-Text HLabel 5650 2300 2    50   Input ~ 0
-FlexSPI_CLK_B
+GPIO_B1_15
 $Comp
 L power:+3V3 #PWR?
@@
 Wire Wire Line
 	2600 4200 2600 3500
-Text HLabel 5650 1600 2    50   Input ~ 0
-SPDIF_IN
-Text HLabel 5650 1800 2    50   Input ~ 0
-SPDIF_OUT
+Text HLabel 5650 2300 2    50   Input ~ 0
+GPIO_AD_B1_03
 Text Label 4800 1600 0    50   ~ 0
 LED_R
@@
 Wire Wire Line
 	4350 4000 4600 4000
+Text Label 5650 1600 0    50   ~ 0
+SA1_MCLK
+Text Label 5650 1800 0    50   ~ 0
+AUD_INT
 Wire Bus Line
 	8100 3700 8100 5300
+Text HLabel 5650 2200 2    50   Input ~ 0
+GPIO_AD_B1_05
 $EndSCHEMATC

Commit message: Added MCU_RESET_N to interfaces
Connections:
- net labels added: MCU_RESET_N
- net labels removed: GPIO_AD_B1_07
Changed lines of the file:
@@
 EESchema Schematic File Version 4
-LIBS:haathi-cache
+LIBS:haathi_schematic-cache
 EELAYER 26 0
 EELAYER END
 $Descr A4 11693 8268
 encoding utf-8
-Sheet 8 11
+Sheet 1 9
 Title "haathi_cam"
 Date "2018-03-11"
@@
 Text HLabel 4050 5000 2    50   Input ~ 0
 GPIO_AD_B1_06
-Text HLabel 4050 5200 2    50   Input ~ 0
-GPIO_AD_B1_07
 $Comp
 L power:+3V3 #PWR?
@@
 Text Label 5650 1800 0    50   ~ 0
 AUD_INT
+Text HLabel 5650 2200 2    50   Input ~ 0
+GPIO_AD_B1_05
 Wire Bus Line
 	8100 3700 8100 5300
-Text HLabel 5650 2200 2    50   Input ~ 0
-GPIO_AD_B1_05
+Text HLabel 4050 5200 2    50   Input ~ 0
+MCU_RESET_N
 $EndSCHEMATC

Commit message: Annotated schematic
Parts:
- gave numbers to parts that had none: 16
Changed lines of the file:
@@
 GPIO Breakout\n
 $Comp
-L haathi_mayank:Conn_02x20_Odd_Even J?
+L haathi_mayank:Conn_02x20_Odd_Even J8
 U 1 1 5A868BCC
 P 3400 4400
-F 0 "J?" H 3450 5517 50  0000 C CNN
+F 0 "J8" H 3450 5517 50  0000 C CNN
 F 1 "Conn_02x20_Odd_Even" H 3450 5426 50  0000 C CNN
 F 2 "" H 3400 4400 50  0001 C CNN
@@
 $EndComp
 $Comp
-L haathi_mayank:Conn_02x20_Odd_Even J?
+L haathi_mayank:Conn_02x20_Odd_Even J9
 U 1 1 5A86901A
 P 6700 4350
-F 0 "J?" H 6750 5467 50  0000 C CNN
+F 0 "J9" H 6750 5467 50  0000 C CNN
 F 1 "Conn_02x20_Odd_Even" H 6750 5376 50  0000 C CNN
 F 2 "" H 6700 4350 50  0001 C CNN
@@
 $EndComp
 $Comp
-L haathi_mayank:Conn_ARM_JTAG_SWD_10 J?
+L haathi_mayank:Conn_ARM_JTAG_SWD_10 J10
 U 1 1 5A8692F2
 P 8450 1800
-F 0 "J?" H 8010 1846 50  0000 R CNN
+F 0 "J10" H 8010 1846 50  0000 R CNN
 F 1 "Conn_ARM_JTAG_SWD_10" H 8010 1755 50  0000 R CNN
 F 2 "Connector_PinHeader_1.27mm:PinHeader_2x05_P1.27mm_Vertical_SMD" H 8500 1250 50  0001 L TNN
@@
 $EndComp
 $Comp
-L haathi_mayank:LED_ARGB D?
+L haathi_mayank:LED_ARGB D8
 U 1 1 5A86C6F9
 P 1550 1750
-F 0 "D?" V 1596 1420 50  0000 R CNN
+F 0 "D8" V 1596 1420 50  0000 R CNN
 F 1 "LED_ARGB" V 1505 1420 50  0000 R CNN
 F 2 "" H 1550 1700 50  0001 C CNN
@@
 $EndComp
 $Comp
-L haathi_mayank:R R?
+L haathi_mayank:R R73
 U 1 1 5A86CADB
 P 1350 2200
-F 0 "R?" V 1300 2300 50  0000 L CNN
+F 0 "R73" V 1300 2300 50  0000 L CNN
 F 1 "430" V 1350 2150 50  0000 L CNN
 F 2 "" V 1280 2200 30  0000 C CNN
@@
 	1350 2050 1350 1950
 $Comp
-L haathi_mayank:R R?
+L haathi_mayank:R R74
 U 1 1 5A86CC47
 P 1550 2200
-F 0 "R?" V 1500 2300 50  0000 L CNN
+F 0 "R74" V 1500 2300 50  0000 L CNN
 F 1 "80" V 1550 2150 50  0000 L CNN
 F 2 "" V 1480 2200 30  0000 C CNN
@@
 $EndComp
 $Comp
-L haathi_mayank:R R?
+L haathi_mayank:R R75
 U 1 1 5A86CC67
 P 1750 2200
-F 0 "R?" V 1700 2300 50  0000 L CNN
+F 0 "R75" V 1700 2300 50  0000 L CNN
 F 1 "80" V 1750 2150 50  0000 L CNN
 F 2 "" V 1680 2200 30  0000 C CNN
@@
 	1550 1550 1550 1500
 $Comp
-L power:VCC #PWR?
+L power:VCC #PWR084
 U 1 1 5A86CEAC
 P 1550 1450
-F 0 "#PWR?" H 1550 1300 50  0001 C CNN
+F 0 "#PWR084" H 1550 1300 50  0001 C CNN
 F 1 "VCC" H 1567 1623 50  0000 C CNN
 F 2 "" H 1550 1450 50  0001 C CNN
@@
 $EndComp
 $Comp
-L power:PWR_FLAG #FLG?
+L power:PWR_FLAG #FLG012
 U 1 1 5A86CF68
 P 1550 1500
-F 0 "#FLG?" H 1550 1575 50  0001 C CNN
+F 0 "#FLG012" H 1550 1575 50  0001 C CNN
 F 1 "PWR_FLAG" V 1550 1628 50  0000 L CNN
 F 2 "" H 1550 1500 50  0001 C CNN
@@
 	1550 1500 1550 1450
 $Comp
-L haathi_mayank:SW-SPST-M S?
+L haathi_mayank:SW-SPST-M S4
 U 1 1 5A86D4EB
 P 3100 1700
-F 0 "S?" H 3100 2002 40  0000 C CNB
+F 0 "S4" H 3100 2002 40  0000 C CNB
 F 1 "SW-SPST-M" H 3100 1926 40  0000 C CNB
 F 2 "" H 3100 1700 60  0000 C CNN
@@
 $EndComp
 $Comp
-L haathi_mayank:SW-SPST-M S?
+L haathi_mayank:SW-SPST-M S5
 U 1 1 5A86D57B
 P 3100 2200
-F 0 "S?" H 3100 2502 40  0000 C CNB
+F 0 "S5" H 3100 2502 40  0000 C CNB
 F 1 "SW-SPST-M" H 3100 2426 40  0000 C CNB
 F 2 "" H 3100 2200 60  0000 C CNN
@@
 	2700 2200 2700 2400
 $Comp
-L power:GND #PWR?
+L power:GND #PWR087
 U 1 1 5A86DF4F
 P 2700 2400
-F 0 "#PWR?" H 2700 2150 50  0001 C CNN
+F 0 "#PWR087" H 2700 2150 50  0001 C CNN
 F 1 "GND" H 2705 2227 50  0000 C CNN
 F 2 "" H 2700 2400 50  0001 C CNN
@@
 JTAG_TDI
 $Comp
-L power:GND #PWR?
+L power:GND #PWR093
 U 1 1 5A86E5EB
 P 8450 2600
-F 0 "#PWR?" H 8450 2350 50  0001 C CNN
+F 0 "#PWR093" H 8450 2350 50  0001 C CNN
 F 1 "GND" H 8455 2427 50  0000 C CNN
 F 2 "" H 8450 2600 50  0001 C CNN
@@
 Connection ~ 8450 2400
 $Comp
-L power:VCC #PWR?
+L power:VCC #PWR092
 U 1 1 5A86EC70
 P 8450 1050
-F 0 "#PWR?" H 8450 900 50  0001 C CNN
+F 0 "#PWR092" H 8450 900 50  0001 C CNN
 F 1 "VCC" H 8467 1223 50  0000 C CNN
 F 2 "" H 8450 1050 50  0001 C CNN
@@
 	8450 1050 8450 1100
 $Comp
-L power:PWR_FLAG #FLG?
+L power:PWR_FLAG #FLG014
 U 1 1 5A86F0A0
 P 8450 2550
-F 0 "#FLG?" H 8450 2625 50  0001 C CNN
+F 0 "#FLG014" H 8450 2625 50  0001 C CNN
 F 1 "PWR_FLAG" V 8450 2678 50  0000 L CNN
 F 2 "" H 8450 2550 50  0001 C CNN
@@
 	8450 2550 8450 2600
 $Comp
-L power:PWR_FLAG #FLG?
+L power:PWR_FLAG #FLG013
 U 1 1 5A86F1E8
 P 8450 1100
-F 0 "#FLG?" H 8450 1175 50  0001 C CNN
+F 0 "#FLG013" H 8450 1175 50  0001 C CNN
 F 1 "PWR_FLAG" V 8450 1228 50  0000 L CNN
 F 2 "" H 8450 1100 50  0001 C CNN
@@
 	4800 2000 5100 2000
 $Comp
-L haathi_mayank:R R?
+L haathi_mayank:R R78
 U 1 1 5A85A90F
 P 5250 1600
-F 0 "R?" V 5200 1700 50  0000 L CNN
+F 0 "R78" V 5200 1700 50  0000 L CNN
 F 1 "0E" V 5250 1550 50  0000 L CNN
 F 2 "" V 5180 1600 30  0000 C CNN
@@
 	5400 1600 5650 1600
 $Comp
-L haathi_mayank:R R?
+L haathi_mayank:R R79
 U 1 1 5A85AEF0
 P 5250 1800
-F 0 "R?" V 5200 1900 50  0000 L CNN
+F 0 "R79" V 5200 1900 50  0000 L CNN
 F 1 "0E" V 5250 1750 50  0000 L CNN
 F 2 "" V 5180 1800 30  0000 C CNN
@@
 $EndComp
 $Comp
-L haathi_mayank:R R?
+L haathi_mayank:R R80
 U 1 1 5A85AF1E
 P 5250 2000
-F 0 "R?" V 5200 2100 50  0000 L CNN
+F 0 "R80" V 5200 2100 50  0000 L CNN
 F 1 "0E" V 5250 1950 50  0000 L CNN
 F 2 "" V 5180 2000 30  0000 C CNN
@@
 	5400 2000 5650 2000
 $Comp
-L haathi_mayank:R R?
+L haathi_mayank:R R81
 U 1 1 5A85C0CC
 P 5250 2200
-F 0 "R?" V 5200 2300 50  0000 L CNN
+F 0 "R81" V 5200 2300 50  0000 L CNN
 F 1 "0E" V 5250 2150 50  0000 L CNN
 F 2 "" V 5180 2200 30  0000 C CNN
@@
 $EndComp
 $Comp
-L haathi_mayank:R R?
+L haathi_mayank:R R82
 U 1 1 5A85C0FA
 P 5250 2300
-F 0 "R?" V 5200 2400 50  0000 L CNN
+F 0 "R82" V 5200 2400 50  0000 L CNN
 F 1 "0E" V 5250 2250 50  0000 L CNN
 F 2 "" V 5180 2300 30  0000 C CNN
@@
 WAKEUP_BUTTON
 $Comp
-L power:+3V3 #PWR?
+L power:+3V3 #PWR086
 U 1 1 5AA63850
 P 2600 3350
-F 0 "#PWR?" H 2600 3200 50  0001 C CNN
+F 0 "#PWR086" H 2600 3200 50  0001 C CNN
 F 1 "+3V3" H 2615 3523 50  0000 C CNN
 F 2 "" H 2600 3350 50  0001 C CNN
@@
 5V_USB_OTG
 $Comp
-L power:GND #PWR?
+L power:GND #PWR085
 U 1 1 5AA639C2
 P 2400 5550
-F 0 "#PWR?" H 2400 5300 50  0001 C CNN
+F 0 "#PWR085" H 2400 5300 50  0001 C CNN
 F 1 "GND" H 2405 5377 50  0000 C CNN
 F 2 "" H 2400 5550 50  0001 C CNN
@@
 Connection ~ 2600 3500
 $Comp
-L power:GND #PWR?
+L power:GND #PWR089
 U 1 1 5AA892A4
 P 4400 5550
-F 0 "#PWR?" H 4400 5300 50  0001 C CNN
+F 0 "#PWR089" H 4400 5300 50  0001 C CNN
 F 1 "GND" H 4405 5377 50  0000 C CNN
 F 2 "" H 4400 5550 50  0001 C CNN
@@
 FlexSPI_SS_B
 $Comp
-L power:GND #PWR?
+L power:GND #PWR090
 U 1 1 5AAA953A
 P 5750 5450
-F 0 "#PWR?" H 5750 5200 50  0001 C CNN
+F 0 "#PWR090" H 5750 5200 50  0001 C CNN
 F 1 "GND" H 5755 5277 50  0000 C CNN
 F 2 "" H 5750 5450 50  0001 C CNN
@@
 GPIO_AD_B1_06
 $Comp
-L power:+3V3 #PWR?
+L power:+3V3 #PWR088
 U 1 1 5AB7B7C5
 P 4200 3350
-F 0 "#PWR?" H 4200 3200 50  0001 C CNN
+F 0 "#PWR088" H 4200 3200 50  0001 C CNN
 F 1 "+3V3" H 4215 3523 50  0000 C CNN
 F 2 "" H 4200 3350 50  0001 C CNN
@@
 GPIO_B1_15
 $Comp
-L power:+3V3 #PWR?
+L power:+3V3 #PWR091
 U 1 1 5AB7D289
 P 7775 3325
-F 0 "#PWR?" H 7775 3175 50  0001 C CNN
+F 0 "#PWR091" H 7775 3175 50  0001 C CNN
 F 1 "+3V3" H 7790 3498 50  0000 C CNN
 F 2 "" H 7775 3325 50  0001 C CNN
@@
 LED_B
 $Comp
-L haathi_mayank:R R?
+L haathi_mayank:R R76
 U 1 1 5B03D6DC
 P 4200 4000
-F 0 "R?" V 4150 4100 50  0000 L CNN
+F 0 "R76" V 4150 4100 50  0000 L CNN
 F 1 "0E" V 4200 3950 50  0000 L CNN
 F 2 "" V 4130 4000 30  0000 C CNN
@@
 $EndComp
 $Comp
-L haathi_mayank:R R?
+L haathi_mayank:R R77
 U 1 1 5B04A370
 P 4200 4500
-F 0 "R?" V 4150 4600 50  0000 L CNN
+F 0 "R77" V 4150 4600 50  0000 L CNN
 F 1 "0E" V 4200 4450 50  0000 L CNN
 F 2 "" V 4130 4500 30  0000 C CNN

Commit message: ERC pass 1: Check and resolve the errors
Signed-off-by: Kumar Abhishek <abhishek@theembeddedkitchen.net>
Connections:
- net labels removed: SA1_MCLK
- wire segments 139 -> 137
Changed lines of the file:
@@
 EESchema Schematic File Version 4
-LIBS:haathi_schematic-cache
+LIBS:haathi-cache
 EELAYER 26 0
 EELAYER END
 $Descr A4 11693 8268
 encoding utf-8
-Sheet 1 9
+Sheet 1 11
 Title "haathi_cam"
 Date "2018-03-11"
@@
 Wire Wire Line
 	1750 2650 1000 2650
-Wire Wire Line
-	1550 1550 1550 1500
-$Comp
-L power:VCC #PWR084
-U 1 1 5A86CEAC
-P 1550 1450
-F 0 "#PWR084" H 1550 1300 50  0001 C CNN
-F 1 "VCC" H 1567 1623 50  0000 C CNN
-F 2 "" H 1550 1450 50  0001 C CNN
-F 3 "" H 1550 1450 50  0001 C CNN
-	1    1550 1450
-	1    0    0    -1
-$EndComp
-$Comp
-L power:PWR_FLAG #FLG012
-U 1 1 5A86CF68
-P 1550 1500
-F 0 "#FLG012" H 1550 1575 50  0001 C CNN
-F 1 "PWR_FLAG" V 1550 1628 50  0000 L CNN
-F 2 "" H 1550 1500 50  0001 C CNN
-F 3 "" H 1550 1500 50  0001 C CNN
-	1    1550 1500
-	0    1    1    0
-$EndComp
-Connection ~ 1550 1500
-Wire Wire Line
-	1550 1500 1550 1450
 $Comp
 L haathi_mayank:SW-SPST-M S4
@@
 Wire Wire Line
 	8350 2400 8450 2400
-Wire Wire Line
-	8450 2400 8450 2550
 Connection ~ 8450 2400
 $Comp
@@
 Wire Wire Line
 	8450 1050 8450 1100
-$Comp
-L power:PWR_FLAG #FLG014
-U 1 1 5A86F0A0
-P 8450 2550
-F 0 "#FLG014" H 8450 2625 50  0001 C CNN
-F 1 "PWR_FLAG" V 8450 2678 50  0000 L CNN
-F 2 "" H 8450 2550 50  0001 C CNN
-F 3 "" H 8450 2550 50  0001 C CNN
-	1    8450 2550
-	0    1    1    0
-$EndComp
-Connection ~ 8450 2550
-Wire Wire Line
-	8450 2550 8450 2600
 $Comp
 L power:PWR_FLAG #FLG013
@@
 Wire Wire Line
 	4350 4000 4600 4000
-Text Label 5650 1600 0    50   ~ 0
-SA1_MCLK
-Text Label 5650 1800 0    50   ~ 0
-AUD_INT
 Text HLabel 5650 2200 2    50   Input ~ 0
 GPIO_AD_B1_05
@@
 Text HLabel 4050 5200 2    50   Input ~ 0
 MCU_RESET_N
+Wire Wire Line
+	8450 2400 8450 2600
+$Comp
+L power:+3V3 #PWR0107
+U 1 1 5B336EAD
+P 1550 1450
+F 0 "#PWR0107" H 1550 1300 50  0001 C CNN
+F 1 "+3V3" H 1565 1623 50  0000 C CNN
+F 2 "" H 1550 1450 50  0001 C CNN
+F 3 "" H 1550 1450 50  0001 C CNN
+	1    1550 1450
+	1    0    0    -1
+$EndComp
+Wire Wire Line
+	1550 1450 1550 1550
+Text HLabel 5650 1600 2    50   Input ~ 0
+SAI1_MCLK
+Text HLabel 5650 1800 2    50   Input ~ 0
+AUD_INT
 $EndSCHEMATC
