File: kicad/haathi_interfaces.sch (KiCad schematic (older format))
At the start: 16 parts, among them J10 Conn_ARM_JTAG_SWD_10, J8 Conn_02x20_Odd_Even, J9 Conn_02x20_Odd_Even

Commit message: Interfaces, reconnected I2C, RGB LED, CAN
Connections:
- net labels added: CAN1_RX, CAN1_TX, GPIO_AD_B1_00, GPIO_AD_B1_01, GPIO_AD_B1_07, GPIO_AD_B1_08, GPIO_SD_B1_00, GPIO_SD_B1_02, GPIO_SD_B1_03, I2C3_SCL, I2C3_SDA
- net labels removed: CAN2_RX, CAN2_TX, ENET_RXD1, ENET_RXER, ENET_TXD1, ENET_TXEN, ENET_TX_CLK, I2C2_SCL, I2C2_SDA
- wire segments 137 -> 143
Changed lines of the file:
@@
 EESchema Schematic File Version 4
-LIBS:haathi-cache
+LIBS:haathi_interfaces-cache
 EELAYER 26 0
 EELAYER END
 $Descr A4 11693 8268
 encoding utf-8
-Sheet 8 11
+Sheet 1 1
 Title "haathi_cam"
 Date "2018-03-11"
@@
 Wire Wire Line
 	4400 4900 4400 5100
-Text HLabel 2850 3700 0    50   Input ~ 0
-I2C1_SCL
-Text HLabel 2850 3600 0    50   Input ~ 0
-I2C1_SDA
 Text HLabel 4050 3800 2    50   Input ~ 0
 UART1_TXD
@@
 Text HLabel 2850 4600 0    50   Input ~ 0
 FlexSPI_CLK_B
-Text HLabel 4050 4600 2    50   Input ~ 0
-FlexSPI_SS_B
 $Comp
 L power:GND #PWR090
@@
 Wire Wire Line
 	5750 5350 5750 5450
-Text HLabel 4050 5300 2    50   Input ~ 0
-CAN2_TX
-Text HLabel 2850 5300 0    50   Input ~ 0
-CAN2_RX
 Wire Wire Line
 	5750 4750 5750 5350
@@
 Text HLabel 7350 3750 2    50   Input ~ 0
 BACKLIGHT_CTL
-Text HLabel 2850 4800 0    50   Input ~ 0
-ENET_RXD1
-Text HLabel 2850 4900 0    50   Input ~ 0
-ENET_TXD1
-Text HLabel 2850 5000 0    50   Input ~ 0
-ENET_TXEN
-Text HLabel 2850 5100 0    50   Input ~ 0
-ENET_TX_CLK
-Text HLabel 2850 5200 0    50   Input ~ 0
-ENET_RXER
-Text HLabel 4050 4200 2    50   Input ~ 0
-I2C2_SCL
-Text HLabel 4050 4300 2    50   Input ~ 0
-I2C2_SDA
 Text HLabel 4600 4000 2    50   Input ~ 0
 GPIO_AD_B0_00
@@
 Wire Wire Line
 	3700 5400 4200 5400
-Text HLabel 5650 2000 2    50   Input ~ 0
-GPIO_B1_15
 $Comp
 L power:+3V3 #PWR091
@@
 Text HLabel 5650 2200 2    50   Input ~ 0
 GPIO_AD_B1_05
-Wire Bus Line
-	8100 3700 8100 5300
 Text HLabel 4050 5200 2    50   Input ~ 0
 MCU_RESET_N
@@
 Wire Wire Line
 	1550 1450 1550 1550
+Text Label 2850 3600 0    50   ~ 0
+I2C1_SDA
+Text Label 2850 3700 0    50   ~ 0
+I2C1_SCL
+Wire Wire Line
+	2450 6100 2850 6100
+Text Label 2850 6100 2    50   ~ 0
+I2C1_SDA
+Text Label 2850 6200 2    50   ~ 0
+I2C1_SCL
+Wire Wire Line
+	2450 6200 2850 6200
+Text HLabel 2450 6100 0    50   Input ~ 0
+GPIO_AD_B1_01
+Text HLabel 2450 6200 0    50   Input ~ 0
+GPIO_AD_B1_00
+Text HLabel 2450 6400 0    50   Input ~ 0
+GPIO_AD_B1_06
+Text HLabel 2450 6500 0    50   Input ~ 0
+GPIO_AD_B1_07
+Wire Wire Line
+	2450 6400 2850 6400
+Wire Wire Line
+	2450 6500 2850 6500
+Text Label 2850 6400 2    50   ~ 0
+I2C3_SDA
+Text Label 2850 6500 2    50   ~ 0
+I2C3_SCL
+Text Label 4050 4200 2    50   ~ 0
+I2C3_SCL
+Text Label 4050 4300 2    50   ~ 0
+I2C3_SDA
 Text HLabel 5650 1600 2    50   Input ~ 0
-SAI1_MCLK
+GPIO_SD_B1_00
 Text HLabel 5650 1800 2    50   Input ~ 0
-AUD_INT
+GPIO_SD_B1_02
+Text HLabel 5650 2000 2    50   Input ~ 0
+GPIO_AD_B0_01
+Text HLabel 4050 4600 2    50   Input ~ 0
+FlexSPI_SS_B
+Text HLabel 2850 4800 0    50   Input ~ 0
+GPIO_B1_15
+Text Label 2850 5300 0    50   ~ 0
+CAN1_RX
+Text Label 4050 5300 2    50   ~ 0
+CAN1_TX
+Text Label 2800 6700 2    50   ~ 0
+CAN1_RX
+Text Label 2800 6800 2    50   ~ 0
+CAN1_TX
+Wire Wire Line
+	2800 6700 2400 6700
+Wire Wire Line
+	2800 6800 2400 6800
+Wire Bus Line
+	8100 3700 8100 5300
+Text HLabel 2400 6700 0    50   Input ~ 0
+GPIO_SD_B1_03
+Text HLabel 2400 6800 0    50   Input ~ 0
+GPIO_AD_B1_08
 $EndSCHEMATC

Commit message: Interfaces, re-connected SPI, ADC, Switch GPIO
Connections:
- net labels added: ADC1, GPIO_AD_B0_12, GPIO_AD_B0_13, GPIO_B1_04, GPIO_B1_05, GPIO_B1_06, GPIO_B1_07, LPSPI4_PCS0, LPSPI4_SCK, LPSPI4_SDI, LPSPI4_SDO, PMIC_ON_REQ, PMIC_STBY_REQ
- net labels removed: FlexSPI_CLK_B, FlexSPI_D0_B, FlexSPI_D1_B, FlexSPI_SS_B, GPIO_AD_B1_04
- wire segments 143 -> 150
Changed lines of the file:
@@
 	3700 3600 4050 3600
 Wire Wire Line
-	3700 3800 4050 3800
-Wire Wire Line
-	3700 3900 4050 3900
-Wire Wire Line
 	3700 4000 4050 4000
 Wire Wire Line
@@
 	3700 4500 4050 4500
 Wire Wire Line
-	3700 4600 4050 4600
-Wire Wire Line
 	3700 4700 4050 4700
 Wire Wire Line
@@
 Wire Wire Line
 	3200 4100 2850 4100
-Wire Wire Line
-	3200 4400 2850 4400
-Wire Wire Line
-	3200 4500 2850 4500
-Wire Wire Line
-	3200 4600 2850 4600
 Wire Wire Line
 	3200 4800 2850 4800
@@
 Wire Wire Line
 	4400 4900 4400 5100
-Text HLabel 4050 3800 2    50   Input ~ 0
-UART1_TXD
-Text HLabel 4050 3900 2    50   Input ~ 0
-UART1_RXD
-Text HLabel 2850 4400 0    50   Input ~ 0
-FlexSPI_D0_B
-Text HLabel 2850 4500 0    50   Input ~ 0
-FlexSPI_D1_B
-Text HLabel 2850 4600 0    50   Input ~ 0
-FlexSPI_CLK_B
 $Comp
 L power:GND #PWR090
@@
 Text HLabel 6150 5250 0    50   Input ~ 0
 LCDIF_VSYNC
-Text HLabel 2850 3800 0    50   Input ~ 0
-ENET_CRS_DV
-Text HLabel 2850 4000 0    50   Input ~ 0
-ENET_RXD0
-Text HLabel 2850 4100 0    50   Input ~ 0
-ENET_TXD0
 Text HLabel 7350 3750 2    50   Input ~ 0
 BACKLIGHT_CTL
@@
 Text HLabel 4600 4500 2    50   Input ~ 0
 GPIO_AD_B0_01
-Text HLabel 4050 4700 2    50   Input ~ 0
-GPIO_AD_B1_04
+Text HLabel 2600 6050 0    50   Input ~ 0
+GPIO_AD_B1_03
 Text HLabel 4050 4800 2    50   Input ~ 0
 GPIO_AD_B1_05
@@
 Wire Wire Line
 	2600 4200 2600 3500
-Text HLabel 5650 2300 2    50   Input ~ 0
-GPIO_AD_B1_03
 Text Label 4800 1600 0    50   ~ 0
 LED_R
@@
 Wire Wire Line
 	4350 4000 4600 4000
-Text HLabel 5650 2200 2    50   Input ~ 0
-GPIO_AD_B1_05
 Text HLabel 4050 5200 2    50   Input ~ 0
 MCU_RESET_N
@@
 I2C1_SCL
 Wire Wire Line
-	2450 6100 2850 6100
-Text Label 2850 6100 2    50   ~ 0
+	1400 6050 1800 6050
+Text Label 1800 6050 2    50   ~ 0
 I2C1_SDA
-Text Label 2850 6200 2    50   ~ 0
+Text Label 1800 6150 2    50   ~ 0
 I2C1_SCL
 Wire Wire Line
-	2450 6200 2850 6200
-Text HLabel 2450 6100 0    50   Input ~ 0
+	1400 6150 1800 6150
+Text HLabel 1400 6050 0    50   Input ~ 0
 GPIO_AD_B1_01
-Text HLabel 2450 6200 0    50   Input ~ 0
+Text HLabel 1400 6150 0    50   Input ~ 0
 GPIO_AD_B1_00
-Text HLabel 2450 6400 0    50   Input ~ 0
+Text HLabel 1400 6350 0    50   Input ~ 0
 GPIO_AD_B1_06
-Text HLabel 2450 6500 0    50   Input ~ 0
+Text HLabel 1400 6450 0    50   Input ~ 0
 GPIO_AD_B1_07
 Wire Wire Line
-	2450 6400 2850 6400
-Wire Wire Line
-	2450 6500 2850 6500
-Text Label 2850 6400 2    50   ~ 0
+	1400 6350 1800 6350
+Wire Wire Line
+	1400 6450 1800 6450
+Text Label 1800 6350 2    50   ~ 0
 I2C3_SDA
-Text Label 2850 6500 2    50   ~ 0
+Text Label 1800 6450 2    50   ~ 0
 I2C3_SCL
 Text Label 4050 4200 2    50   ~ 0
@@
 Text HLabel 5650 2000 2    50   Input ~ 0
 GPIO_AD_B0_01
-Text HLabel 4050 4600 2    50   Input ~ 0
-FlexSPI_SS_B
 Text HLabel 2850 4800 0    50   Input ~ 0
 GPIO_B1_15
@@
 Text Label 4050 5300 2    50   ~ 0
 CAN1_TX
-Text Label 2800 6700 2    50   ~ 0
+Text Label 1750 6650 2    50   ~ 0
 CAN1_RX
-Text Label 2800 6800 2    50   ~ 0
+Text Label 1750 6750 2    50   ~ 0
 CAN1_TX
 Wire Wire Line
-	2800 6700 2400 6700
-Wire Wire Line
-	2800 6800 2400 6800
+	1750 6650 1350 6650
+Wire Wire Line
+	1750 6750 1350 6750
+Text HLabel 1350 6650 0    50   Input ~ 0
+GPIO_SD_B1_03
+Text HLabel 1350 6750 0    50   Input ~ 0
+GPIO_AD_B1_08
+Text HLabel 1350 6900 0    50   Input ~ 0
+GPIO_AD_B0_12
+Text Label 4150 3800 2    50   ~ 0
+UART1_TXD
+Text Label 1800 6900 2    50   ~ 0
+UART1_TXD
+Text HLabel 1350 7000 0    50   Input ~ 0
+GPIO_AD_B0_13
+Text Label 1800 7000 2    50   ~ 0
+UART1_RXD
+Text Label 4150 3900 2    50   ~ 0
+UART1_RXD
+Wire Wire Line
+	3700 3800 4150 3800
+Wire Wire Line
+	3700 3900 4150 3900
+Wire Wire Line
+	1350 7000 1800 7000
+Wire Wire Line
+	1350 6900 1800 6900
+Text HLabel 1350 7150 0    50   Input ~ 0
+GPIO_B1_07
+Text Label 1850 7150 2    50   ~ 0
+LPSPI4_SCK
+Text HLabel 1350 7250 0    50   Input ~ 0
+GPIO_B1_06
+Wire Wire Line
+	1350 7250 1850 7250
+Wire Wire Line
+	1350 7150 1850 7150
+Text Label 1850 7250 2    50   ~ 0
+LPSPI4_SDO
+Text HLabel 1350 7350 0    50   Input ~ 0
+GPIO_B1_05
+Text HLabel 1350 7450 0    50   Input ~ 0
+GPIO_B1_04
+Wire Wire Line
+	1350 7350 1850 7350
+Wire Wire Line
+	1350 7450 1850 7450
+Text Label 1850 7350 2    50   ~ 0
+LPSPI4_SDI
+Text Label 1850 7450 2    50   ~ 0
+LPSPI4_PCS0
+Text Label 2700 4400 0    50   ~ 0
+LPSPI4_SDO
+Text Label 2700 4500 0    50   ~ 0
+LPSPI4_SDI
+Text Label 2700 4600 0    50   ~ 0
+LPSPI4_SCK
+Text Label 4250 4600 2    50   ~ 0
+LPSPI4_PCS0
+Wire Wire Line
+	2700 4400 3200 4400
+Wire Wire Line
+	2700 4500 3200 4500
+Wire Wire Line
+	2700 4600 3200 4600
+Text HLabel 2850 4100 0    50   Input ~ 0
+ENET_TXD0
+Text HLabel 2850 4000 0    50   Input ~ 0
+ENET_RXD0
+Text HLabel 2850 3800 0    50   Input ~ 0
+ENET_CRS_DV
+Wire Wire Line
+	3700 4600 4250 4600
+Wire Wire Line
+	2600 6050 3050 6050
 Wire Bus Line
 	8100 3700 8100 5300
-Text HLabel 2400 6700 0    50   Input ~ 0
-GPIO_SD_B1_03
-Text HLabel 2400 6800 0    50   Input ~ 0
-GPIO_AD_B1_08
+Text Label 3050 6050 2    50   ~ 0
+ADC1
+Text Label 4050 4700 2    50   ~ 0
+ADC1
+Text HLabel 5650 2200 2    50   Input ~ 0
+PMIC_STBY_REQ
+Text HLabel 5650 2300 2    50   Input ~ 0
+PMIC_ON_REQ
 $EndSCHEMATC

Commit message: Re-wired CSI/SAI interface pins to headers
Parts:
- removed R76, R77: 0E, symbol haathi_mayank:R
- added R?: 0E, symbol haathi_mayank:R
- added RN?: R_Pack08_0E_DNP, symbol haathi_mayank:R_Pack08
- added RN?: R_Pack04_0E_DNP, symbol haathi_mayank:R_Pack04
Connections:
- net labels added: CAN2_RX, CAN_STBY, ENC1_HOME, ENC1_PHASEA, ENC1_PHASEB, ENET_RXER, ENET_TX_CLK, GPIO_AD_B0_02, GPIO_AD_B0_03, GPIO_AD_B0_04, GPIO_AD_B0_05, GPIO_AD_B0_14, GPIO_AD_B0_15, GPIO_AD_B1_04, GPIO_AD_B1_09, GPIO_AD_B1_10, GPIO_AD_B1_11, GPIO_AD_B1_12, GPIO_AD_B1_13, GPIO_AD_B1_14, GPIO_AD_B1_15, GPIO_B1_10, GPIO_B1_11, GPIO_EMC_40, OTG2_ID, OTG2_OC, PWM4, SAI_MCLK, SPDIF_OUT, SPDIF_SR_CLK
- net labels removed: ENET_CRS_DV, ENET_RXD0, ENET_TXD0
- wire segments 150 -> 182
Other:
- note added: "Note: Muxed with CSI !\n\n"

Commit message: Interfaces, added 4.7k DNP pull ups to I2C3 bus
Parts:
- added R? (x2): 4.7k_DNP, symbol haathi_mayank:R
Connections:
- wire segments 182 -> 188
Changed lines of the file:
@@
 Text HLabel 1250 6150 0    50   Input ~ 0
 GPIO_AD_B1_00
-Text HLabel 1250 6350 0    50   Input ~ 0
+Text HLabel 1250 7500 0    50   Input ~ 0
 GPIO_AD_B1_06
-Text HLabel 1250 6450 0    50   Input ~ 0
+Text HLabel 1250 7600 0    50   Input ~ 0
 GPIO_AD_B1_07
 Wire Wire Line
-	1250 6350 1650 6350
-Wire Wire Line
-	1250 6450 1650 6450
-Text Label 1650 6350 2    50   ~ 0
+	1250 7500 1400 7500
+Wire Wire Line
+	1250 7600 1550 7600
+Text Label 1650 7500 2    50   ~ 0
 I2C3_SDA
-Text Label 1650 6450 2    50   ~ 0
+Text Label 1650 7600 2    50   ~ 0
 I2C3_SCL
 Text Label 4050 4200 2    50   ~ 0
@@
 Text Label 4050 5300 2    50   ~ 0
 CAN1_TX
-Text Label 1600 6650 2    50   ~ 0
+Text Label 1650 6350 2    50   ~ 0
 CAN1_RX
-Text Label 1600 6750 2    50   ~ 0
+Text Label 1650 6450 2    50   ~ 0
 CAN1_TX
 Wire Wire Line
-	1600 6650 1200 6650
-Wire Wire Line
-	1600 6750 1200 6750
-Text HLabel 1200 6650 0    50   Input ~ 0
+	1650 6350 1250 6350
+Wire Wire Line
+	1650 6450 1250 6450
+Text HLabel 1250 6350 0    50   Input ~ 0
 GPIO_SD_B1_03
-Text HLabel 1200 6750 0    50   Input ~ 0
+Text HLabel 1250 6450 0    50   Input ~ 0
 GPIO_AD_B1_08
-Text HLabel 1200 6900 0    50   Input ~ 0
+Text HLabel 1250 6600 0    50   Input ~ 0
 GPIO_AD_B0_12
 Text Label 4150 3800 2    50   ~ 0
 UART1_TXD
-Text Label 1650 6900 2    50   ~ 0
+Text Label 1700 6600 2    50   ~ 0
 UART1_TXD
-Text HLabel 1200 7000 0    50   Input ~ 0
+Text HLabel 1250 6700 0    50   Input ~ 0
 GPIO_AD_B0_13
-Text Label 1650 7000 2    50   ~ 0
+Text Label 1700 6700 2    50   ~ 0
 UART1_RXD
 Text Label 4150 3900 2    50   ~ 0
@@
 	3700 3900 4150 3900
 Wire Wire Line
-	1200 7000 1650 7000
-Wire Wire Line
-	1200 6900 1650 6900
+	1250 6700 1700 6700
+Wire Wire Line
+	1250 6600 1700 6600
 Text HLabel 2400 6050 0    50   Input ~ 0
 GPIO_B1_07
@@
 Wire Notes Line
 	5500 5900 5500 7500
+$Comp
+L haathi_mayank:R R?
+U 1 1 5B465F1F
+P 1550 7200
+F 0 "R?" H 1400 7150 50  0000 L CNN
+F 1 "4.7k_DNP" H 1150 7250 50  0000 L CNN
+F 2 "" V 1480 7200 30  0000 C CNN
+F 3 "" H 1550 7200 30  0000 C CNN
+	1    1550 7200
+	-1   0    0    1
+$EndComp
+$Comp
+L haathi_mayank:R R?
+U 1 1 5B46616D
+P 1400 7200
+F 0 "R?" H 1500 7150 50  0000 L CNN
+F 1 "4.7k_DNP" H 1500 7250 50  0000 L CNN
+F 2 "" V 1330 7200 30  0000 C CNN
+F 3 "" H 1400 7200 30  0000 C CNN
+	1    1400 7200
+	-1   0    0    1
+$EndComp
+Wire Wire Line
+	1400 7350 1400 7500
+Connection ~ 1400 7500
+Wire Wire Line
+	1400 7500 1650 7500
+Wire Wire Line
+	1550 7350 1550 7600
+Connection ~ 1550 7600
+Wire Wire Line
+	1550 7600 1650 7600
+$Comp
+L power:+3V3 #PWR?
+U 1 1 5B48CD9A
+P 1550 6950
+F 0 "#PWR?" H 1550 6800 50  0001 C CNN
+F 1 "+3V3" H 1565 7123 50  0000 C CNN
+F 2 "" H 1550 6950 50  0001 C CNN
+F 3 "" H 1550 6950 50  0001 C CNN
+	1    1550 6950
+	1    0    0    -1
+$EndComp
+Wire Wire Line
+	1550 7050 1550 6950
+Wire Wire Line
+	1400 7050 1550 7050
 Wire Bus Line
 	8100 3700 8100 5300
+Connection ~ 1550 7050
 $EndSCHEMATC

Commit message: Switch RGB LED from GPIO_AD_B0_01 to GPIO_SD_B1_02
GPIO_AD_B0_01 was already used for LED backlight

Signed-off-by: Kumar Abhishek <abhishek@theembeddedkitchen.net>
Connections:
- net labels added: GPIO_SD_B1_01
Changed lines of the file:
@@
 EESchema Schematic File Version 4
-LIBS:haathi_interfaces-cache
+LIBS:haathi_schematic-cache
 EELAYER 26 0
 EELAYER END
 $Descr A4 11693 8268
 encoding utf-8
-Sheet 1 1
+Sheet 6 9
 Title "haathi_cam"
 Date "2018-03-11"
@@
 GPIO_SD_B1_02
 Text HLabel 5650 2000 2    50   Input ~ 0
-GPIO_AD_B0_01
+GPIO_SD_B1_01
 Text Label 2850 5300 0    50   ~ 0
 CAN1_RX
@@
 Wire Wire Line
 	1400 7050 1550 7050
+Connection ~ 1550 7050
 Wire Bus Line
 	8100 3700 8100 5300
-Connection ~ 1550 7050
 $EndSCHEMATC

Commit message: Updates the USB OTG connections for OTG2 on the shield
Connections:
- net labels added: GPIO_EMC_41, OTG2_PWR
- net labels removed: GPIO_AD_B0_00, OTG2_ID
Other:
- note added: "Note: EMC_41 is muxed with CSI page pin!\n\n"
Changed lines of the file:
@@
 $Descr A4 11693 8268
 encoding utf-8
-Sheet 6 9
+Sheet 1 9
 Title "haathi_cam"
 Date "2018-03-11"
@@
 Text HLabel 6150 3650 0    50   Input ~ 0
 USB_OTG2_D+_EXTERN
-Text HLabel 6150 3750 0    50   Input ~ 0
-USB_OTG2_ID_EXTERN
 Text HLabel 6150 3850 0    50   Input ~ 0
 USB_GND_EXTERN
@@
 Wire Wire Line
 	3200 5300 2850 5300
-Text HLabel 7350 3450 2    50   Input ~ 0
+Text HLabel 4050 4000 2    50   Input ~ 0
 ONOFF
-Text HLabel 7350 3550 2    50   Input ~ 0
+Text HLabel 4050 4500 2    50   Input ~ 0
 WAKEUP_BUTTON
 $Comp
@@
 Wire Wire Line
 	2650 4100 3200 4100
-Text HLabel 2400 6750 0    50   Input ~ 0
-GPIO_AD_B0_00
-Wire Wire Line
-	2400 6750 3000 6750
 Wire Wire Line
 	2400 6850 3000 6850
 Text HLabel 2400 6850 0    50   Input ~ 0
 GPIO_EMC_40
-Text Label 3000 6750 2    50   ~ 0
-OTG2_ID
 Text Label 3000 6850 2    50   ~ 0
-OTG2_OC
-Text Label 4050 4000 2    50   ~ 0
-OTG2_ID
-Text Label 4050 4500 2    50   ~ 0
 OTG2_OC
 Text Label 5950 4050 0    50   ~ 0
@@
 	1400 7050 1550 7050
 Connection ~ 1550 7050
+Wire Wire Line
+	2400 6950 3000 6950
+Text HLabel 2400 6950 0    50   Input ~ 0
+GPIO_EMC_41
+Text Label 3000 6950 2    50   ~ 0
+OTG2_PWR
+Text Label 7350 3550 2    50   ~ 0
+OTG2_OC
+Text Label 7350 3450 2    50   ~ 0
+OTG2_PWR
+Text Notes 2425 7125 0    50   ~ 0
+Note: EMC_41 is muxed with CSI page pin!\n\n
 Wire Bus Line
 	8100 3700 8100 5300
+Text HLabel 6150 3750 0    50   Input ~ 0
+USB_OTG2_ID_EXTERN
 $EndSCHEMATC
